Commit message: update collision files for two robots

File: mecademic_description/urdf/meca_500_r3_capsule.urdf.xacro (robot description, xacro)
@@ -1,14 +1,14 @@
-<?xml version="1.0" ?>
-<robot name="meca_500_r3" version="1.0">
+<robot name="meca_500_r3" xmlns:xacro="http://ros.org/wiki/xacro">
   <link name="world"/>
-  <joint name="world" type="fixed">
+  <joint name="world_A" type="fixed">
     <parent link="world"/>
-    <child link="meca_base_link"/>
-  </joint>
-  <link name="meca_base_link">
-    <visual>
-      <origin rpy="0.0 0.0 0.0" xyz="0.0 0.0 0.0"/>
-      <geometry>
-        <mesh filename="package://mecademic_description/meshes/meca_500_r3_base.dae"/>
+    <child link="meca_base_link_A"/>
+  </joint>
+  <!-- Base link is the center of the robot's bottom plate -->
+  <link name="meca_base_link_A">
+    <visual>
+      <origin xyz="0 0 0" rpy="0 0 0" />
+      <geometry>
+        <mesh filename="package://mecademic_description/meshes/meca_500_r3_base.dae" />
       </geometry>
     </visual>
@@ -36,9 +36,23 @@
     </inertial>
   </link>
-  <link name="meca_axis_1_link">
-    <visual>
-      <origin rpy="0.0 0.0 0.0" xyz="0.0 0.0 0.0"/>
-      <geometry>
-        <mesh filename="package://mecademic_description/meshes/meca_500_r3_j1.dae"/>
+  <gazebo>
+      <plugin filename="libxbot2_gz_joint_server.so" name="xbot2_gz_joint_server">
+         <pid>
+            <pid name="meca_axis_1_joint_A" profile="small_mot"/>
+            <pid name="meca_axis_2_joint_A" profile="small_mot"/>
+            <pid name="meca_axis_3_joint_A" profile="small_mot"/>
+            <pid name="meca_axis_4_joint_A" profile="small_mot"/>
+            <pid name="meca_axis_5_joint_A" profile="small_mot"/>
+            <pid name="meca_axis_6_joint_A" profile="small_mot"/>
+         </pid>
+         <gain d="5" name="small_mot" p="100"/>
+      </plugin>
+   </gazebo>
+  <!-- Joint 1 -->
+  <link name="meca_axis_1_link_A">
+    <visual>
+      <origin xyz="0 0 0" rpy="0 0 0" />
+      <geometry>
+        <mesh filename="package://mecademic_description/meshes/meca_500_r3_j1.dae" />
       </geometry>
     </visual>
@@ -66,16 +80,17 @@
     </inertial>
   </link>
-  <joint name="meca_axis_1_joint" type="revolute">
-    <origin rpy="0.0 0.0 0.0" xyz="0.012498 0.0 0.091"/>
-    <axis xyz="0.0 0.0 1.0"/>
-    <parent link="meca_base_link"/>
-    <child link="meca_axis_1_link"/>
-    <limit effort="10.0" lower="-3.05433" upper="3.05433" velocity="2.61799"/>
-  </joint>
-  <link name="meca_axis_2_link">
-    <visual>
-      <origin rpy="0.0 0.0 0.0" xyz="0.0 0.0 0.0"/>
-      <geometry>
-        <mesh filename="package://mecademic_description/meshes/meca_500_r3_j2.dae"/>
+  <joint name="meca_axis_1_joint_A" type="revolute">
+    <origin xyz="0.012498 0 0.091" rpy="0 0 0" />
+    <parent link="meca_base_link_A" />
+    <child link="meca_axis_1_link_A" />
+    <axis xyz="0 0 1" />
+    <limit effort="10.0" velocity="2.61799" lower="-3.05433" upper="3.05433" />
+  </joint>
+  <!-- Joint 2 -->
+  <link name="meca_axis_2_link_A">
+    <visual>
+      <origin xyz="0 0 0" rpy="0 0 0" />
+      <geometry>
+        <mesh filename="package://mecademic_description/meshes/meca_500_r3_j2.dae" />
       </geometry>
     </visual>
@@ -103,16 +118,17 @@
     </inertial>
   </link>
-  <joint name="meca_axis_2_joint" type="revolute">
-    <origin rpy="0.0 0.0 0.0" xyz="0.0 0.0 0.044"/>
-    <axis xyz="0.0 1.0 0.0"/>
-    <parent link="meca_axis_1_link"/>
-    <child link="meca_axis_2_link"/>
-    <limit effort="10.0" lower="-1.22173048" upper="1.5708" velocity="2.61799"/>
-  </joint>
-  <link name="meca_axis_3_link">
-    <visual>
-      <origin rpy="0.0 0.0 0.0" xyz="0.0 0.0 0.0"/>
-      <geometry>
-        <mesh filename="package://mecademic_description/meshes/meca_500_r3_j3.dae"/>
+  <joint name="meca_axis_2_joint_A" type="revolute">
+    <origin xyz="0 0 0.044" rpy="0 0 0" />
+    <parent link="meca_axis_1_link_A" />
+    <child link="meca_axis_2_link_A" />
+    <axis xyz="0 1 0" />
+    <limit effort="10.0" velocity="2.61799" lower="-1.22173048" upper="1.5708" />
+  </joint>
+  <!-- Joint 3 -->
+  <link name="meca_axis_3_link_A">
+    <visual>
+      <origin xyz="0 0 0" rpy="0 0 0" />
+      <geometry>
+        <mesh filename="package://mecademic_description/meshes/meca_500_r3_j3.dae" />
       </geometry>
     </visual>
@@ -140,16 +156,17 @@
     </inertial>
   </link>
-  <joint name="meca_axis_3_joint" type="revolute">
-    <origin rpy="0.0 0.0 0.0" xyz="0.0 0.0 0.135"/>
-    <axis xyz="0.0 1.0 0.0"/>
-    <parent link="meca_axis_2_link"/>
-    <child link="meca_axis_3_link"/>
-    <limit effort="10.0" lower="-2.35619" upper="1.22173048" velocity="3.14159"/>
-  </joint>
-  <link name="meca_axis_4_link">
-    <visual>
-      <origin rpy="0.0 0.0 0.0" xyz="0.0 0.0 0.0"/>
-      <geometry>
-        <mesh filename="package://mecademic_description/meshes/meca_500_r3_j4.dae"/>
+  <joint name="meca_axis_3_joint_A" type="revolute">
+    <origin xyz="0 0 0.135" rpy="0 0 0" />
+    <parent link="meca_axis_2_link_A" />
+    <child link="meca_axis_3_link_A" />
+    <axis xyz="0 1 0" />
+    <limit effort="10.0" velocity="3.14159" lower="-2.35619" upper="1.22173048" />
+  </joint>
+  <!-- Joint 4 -->
+  <link name="meca_axis_4_link_A">
+    <visual>
+      <origin xyz="0 0 0" rpy="0 0 0" />
+      <geometry>
+        <mesh filename="package://mecademic_description/meshes/meca_500_r3_j4.dae" />
       </geometry>
     </visual>
@@ -177,16 +194,17 @@
     </inertial>
   </link>
-  <joint name="meca_axis_4_joint" type="revolute">
-    <origin rpy="0.0 0.0 0.0" xyz="0.0 0.0 0.038"/>
-    <axis xyz="1.0 0.0 0.0"/>
-    <parent link="meca_axis_3_link"/>
-    <child link="meca_axis_4_link"/>
-    <limit effort="10.0" lower="-2.96706" upper="2.96706" velocity="5.23599"/>
-  </joint>
-  <link name="meca_axis_5_link">
-    <visual>
-      <origin rpy="0.0 0.0 0.0" xyz="0.0 0.0 0.0"/>
-      <geometry>
-        <mesh filename="package://mecademic_description/meshes/meca_500_r3_j5.dae"/>
+  <joint name="meca_axis_4_joint_A" type="revolute">
+    <origin xyz="0 0 0.038" rpy="0 0 0" />
+    <parent link="meca_axis_3_link_A" />
+    <child link="meca_axis_4_link_A" />
+    <axis xyz="1 0 0" />
+    <limit effort="10.0" velocity="5.23599" lower="-2.96706" upper="2.96706" />
+  </joint>
+  <!-- Joint 5 -->
+  <link name="meca_axis_5_link_A">
+    <visual>
+      <origin xyz="0 0 0" rpy="0 0 0" />
+      <geometry>
+        <mesh filename="package://mecademic_description/meshes/meca_500_r3_j5.dae" />
       </geometry>
     </visual>
@@ -214,16 +232,17 @@
     </inertial>
   </link>
-  <joint name="meca_axis_5_joint" type="revolute">
-    <origin rpy="0.0 0.0 0.0" xyz="0.12 0.0 0.0"/>
-    <axis xyz="0.0 1.0 0.0"/>
-    <parent link="meca_axis_4_link"/>
-    <child link="meca_axis_5_link"/>
-    <limit effort="10.0" lower="-2.00713" upper="2.00713" velocity="5.23599"/>
-  </joint>
-  <link name="meca_axis_6_link">
-    <visual>
-      <origin rpy="0.0 0.0 0.0" xyz="0.0 0.0 0.0"/>
-      <geometry>
-        <mesh filename="package://mecademic_description/meshes/meca_500_r3_j6.dae"/>
+  <joint name="meca_axis_5_joint_A" type="revolute">
+    <origin xyz="0.12 0 0" rpy="0 0 0" />
+    <parent link="meca_axis_4_link_A" />
+    <child link="meca_axis_5_link_A" />
+    <axis xyz="0 1 0" />
+    <limit effort="10.0" velocity="5.23599" lower="-2.00713" upper="2.00713" />
+  </joint>
+  <!-- Joint 6 -->
+  <link name="meca_axis_6_link_A">
+    <visual>
+      <origin xyz="0 0 0" rpy="0 0 0" />
+      <geometry>
+        <mesh filename="package://mecademic_description/meshes/meca_500_r3_j6.dae" />
       </geometry>
     </visual>
@@ -251,10 +270,345 @@
     </inertial>
   </link>
-  <joint name="meca_axis_6_joint" type="revolute">
-    <origin rpy="0.0 0.0 0.0" xyz="0.07 0.0 0.0"/>
-    <axis xyz="1.0 0.0 0.0"/>
-    <parent link="meca_axis_5_link"/>
-    <child link="meca_axis_6_link"/>
-    <limit effort="10.0" lower="-3.14159" upper="3.14159" velocity="8.72665"/>
-  </joint>
+  <joint name="meca_axis_6_joint_A" type="revolute">
+    <origin xyz="0.07 0 0" rpy="0 0 0" />
+    <parent link="meca_axis_5_link_A" />
+    <child link="meca_axis_6_link_A" />
+    <axis xyz="1 0 0" />
+    <limit effort="10.0" velocity="8.72665" lower="-4.712" upper="4.712" />
+  </joint>
+<!-- 2nd ROBOT -->
+  <joint name="world_B" type="fixed">
+      <origin xyz="0.2 0.3 0" rpy="0 0 0"/>
+      <parent link="world"/>
+      <child link="meca_base_link_B"/>
+    </joint>
+    <!-- Base link is the center of the robot's bottom plate -->
+  <link name="meca_base_link_B">
+    <visual>
+      <origin xyz="0 0 0" rpy="0 0 0" />
+      <geometry>
+        <mesh filename="package://mecademic_description/meshes/meca_500_r3_base.dae" />
+      </geometry>
+    </visual>
+    <collision>
+      <origin rpy="-0.00464229562531 1.241639409 -0.00331992768483" xyz="0.002912665 2.5933825e-05 0.03195115"/>
+      <geometry>
+        <cylinder length="0.0247681427348" radius="0.069277"/>
+      </geometry>
+    </collision>
+    <collision>
+      <origin rpy="-0.00464229562531 1.241639409 -0.00331992768483" xyz="-0.008807 0.000007 0.027948"/>
+      <geometry>
+        <sphere radius="0.069277"/>
+      </geometry>
+    </collision>
+    <collision>
+      <origin rpy="-0.00464229562531 1.241639409 -0.00331992768483" xyz="0.014632 0.000045 0.035954"/>
+      <geometry>
+        <sphere radius="0.069277"/>
+      </geometry>
+    </collision>
+    <inertial>
+      <mass value="1"/>
+      <inertia ixx="0.01" ixy="0" ixz="0" iyy="0.01" iyz="0" izz="0.01"/>
+    </inertial>
+  </link>
+  <gazebo>
+      <plugin filename="libxbot2_gz_joint_server.so" name="xbot2_gz_joint_server">
+          <pid>
+            <pid name="meca_axis_1_joint_B" profile="small_mot"/>
+            <pid name="meca_axis_2_joint_B" profile="small_mot"/>
+            <pid name="meca_axis_3_joint_B" profile="small_mot"/>
+            <pid name="meca_axis_4_joint_B" profile="small_mot"/>
+            <pid name="meca_axis_5_joint_B" profile="small_mot"/>
+            <pid name="meca_axis_6_joint_B" profile="small_mot"/>
+          </pid>
+          <gain d="5" name="small_mot" p="100"/>
+      </plugin>
+    </gazebo>
+  <!-- Joint 1 -->
+  <link name="meca_axis_1_link_B">
+    <visual>
+      <origin xyz="0 0 0" rpy="0 0 0" />
+      <geometry>
+        <mesh filename="package://mecademic_description/meshes/meca_500_r3_j1.dae" />
+      </geometry>
+    </visual>
+    <collision>
+      <origin rpy="-1.5643390872 0.00108905813092 -0.00108204843032" xyz="1.404e-07 -0.00017605 0.03168225"/>
+      <geometry>
+        <cylinder length="0.0388249324419" radius="0.0530516"/>
+      </geometry>
+    </collision>
+    <collision>
+      <origin rpy="-1.5643390872 0.00108905813092 -0.00108204843032" xyz="-0.000021 -0.019588 0.031557"/>
+      <geometry>
+        <sphere radius="0.0530516"/>
+      </geometry>
+    </collision>
+    <collision>
+      <origin rpy="-1.5643390872 0.00108905813092 -0.00108204843032" xyz="0.000021 0.019236 0.031808"/>
+      <geometry>
+        <sphere radius="0.0530516"/>
+      </geometry>
+    </collision>
+    <inertial>
+      <mass value="1"/>
+      <inertia ixx="0.01" ixy="0" ixz="0" iyy="0.01" iyz="0" izz="0.01"/>
+    </inertial>
+  </link>
+  <joint name="meca_axis_1_joint_B" type="revolute">
+    <origin xyz="0.012498 0 0.091" rpy="0 0 0" />
+    <parent link="meca_base_link_B" />
+    <child link="meca_axis_1_link_B" />
+    <axis xyz="0 0 1" />
+    <limit effort="10.0" velocity="2.61799" lower="-3.05433" upper="3.05433" />
+  </joint>
+  <!-- Joint 2 -->
+  <link name="meca_axis_2_link_B">
+    <visual>
+      <origin xyz="0 0 0" rpy="0 0 0" />
+      <geometry>
+        <mesh filename="package://mecademic_description/meshes/meca_500_r3_j2.dae" />
+      </geometry>
+    </visual>
+    <collision>
+      <origin rpy="3.14150631803 -0.0666872950524 -3.13900434911" xyz="-0.007204205 2.561655e-06 0.07263715"/>
+      <geometry>
+        <cylinder length="0.121249210008" radius="0.0578403"/>
+      </geometry>
+    </collision>
+    <collision>
+      <origin rpy="3.14150631803 -0.0666872950524 -3.13900434911" xyz="-0.003164 0.000008 0.133127"/>
+      <geometry>
+        <sphere radius="0.0578403"/>
+      </geometry>
+    </collision>
+    <collision>
+      <origin rpy="3.14150631803 -0.0666872950524 -3.13900434911" xyz="-0.011244 -0.000003 0.012147"/>
+      <geometry>
+        <sphere radius="0.0578403"/>
+      </geometry>
+    </collision>
+    <inertial>
+      <mass value="1"/>
+      <inertia ixx="0.01" ixy="0" ixz="0" iyy="0.01" iyz="0" izz="0.01"/>
+    </inertial>
+  </link>
+  <joint name="meca_axis_2_joint_B" type="revolute">
+    <origin xyz="0 0 0.044" rpy="0 0 0" />
+    <parent link="meca_axis_1_link_B" />
+    <child link="meca_axis_2_link_B" />
+    <axis xyz="0 1 0" />
+    <limit effort="10.0" velocity="2.61799" lower="-1.22173048" upper="1.5708" />
+  </joint>
+  <!-- Joint 3 -->
+  <link name="meca_axis_3_link_B">
+    <visual>
+      <origin xyz="0 0 0" rpy="0 0 0" />
+      <geometry>
+        <mesh filename="package://mecademic_description/meshes/meca_500_r3_j3.dae" />
+      </geometry>
+    </visual>
+    <collision>
+      <origin rpy="-0.0775632999618 0.486298597709 -0.0192491912301" xyz="0.009983498 -0.000990284 0.020095595"/>
+      <geometry>
+        <cylinder length="0.0408120816515" radius="0.0503272"/>
+      </geometry>
+    </collision>
+    <collision>
+      <origin rpy="-0.0775632999618 0.486298597709 -0.0192491912301" xyz="0.000447 -0.002388 0.002109"/>
+      <geometry>
+        <sphere radius="0.0503272"/>
+      </geometry>
+    </collision>
+    <collision>
+      <origin rpy="-0.0775632999618 0.486298597709 -0.0192491912301" xyz="0.019520 0.000408 0.038082"/>
+      <geometry>
+        <sphere radius="0.0503272"/>
+      </geometry>
+    </collision>
+    <inertial>
+      <mass value="1"/>
+      <inertia ixx="0.01" ixy="0" ixz="0" iyy="0.01" iyz="0" izz="0.01"/>
+    </inertial>
+  </link>
+  <joint name="meca_axis_3_joint_B" type="revolute">
+    <origin xyz="0 0 0.135" rpy="0 0 0" />
+    <parent link="meca_axis_2_link_B" />
+    <child link="meca_axis_3_link_B" />
+    <axis xyz="0 1 0" />
+    <limit effort="10.0" velocity="3.14159" lower="-2.35619" upper="1.22173048" />
+  </joint>
+  <!-- Joint 4 -->
+  <link name="meca_axis_4_link_B">
+    <visual>
+      <origin xyz="0 0 0" rpy="0 0 0" />
+      <geometry>
+        <mesh filename="package://mecademic_description/meshes/meca_500_r3_j4.dae" />
+      </geometry>
+    </visual>
+    <collision>
+      <origin rpy="-1.61527511752 1.5509782436 -1.59546790677" xyz="0.1018437 -0.00037629375 0.0004856635"/>
+      <geometry>
+        <cylinder length="0.0362997282424" radius="0.0387182"/>
+      </geometry>
+    </collision>
+    <collision>
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