Commit message: update urdf and srdf with new capsules (rotary and linear)

File: mecademic_description/urdf/meca_500_r3_capsule.urdf.xacro (robot description, xacro)
@@ -1,107 +1,131 @@
-<robot name="meca_500_r3" xmlns:xacro="http://ros.org/wiki/xacro">
-<material name="blue">
-    <color rgba="0 0 0.8 1"/>
+<?xml version="1.0" ?>
+<robot name="meca_500_r3" version="1.0">
+  <material name="blue">
+    <color rgba="0.0 0.0 0.8 1.0"/>
   </material>
   <material name="black">
-    <color rgba="0 0 0 1"/>
+    <color rgba="0.0 0.0 0.0 1.0"/>
   </material>
   <material name="white">
-    <color rgba="1 1 1 1"/>
+    <color rgba="1.0 1.0 1.0 1.0"/>
   </material>
   <material name="grey">
-    <color rgba="0.5 0.5 0.5 1"/>
+    <color rgba="0.5 0.5 0.5 1.0"/>
   </material>
   <material name="red">
-    <color rgba="1 0 0 1"/>
+    <color rgba="1.0 0.0 0.0 1.0"/>
   </material>
   <material name="green">
-    <color rgba="0 1 0 1"/>
+    <color rgba="0.0 1.0 0.0 1.0"/>
   </material>
   <material name="yellow">
-    <color rgba="1 1 0 1"/>
+    <color rgba="1.0 1.0 0.0 1.0"/>
   </material>
   <material name="tree_green">
-    <color rgba="0.13 0.54 0.13 1"/>
+    <color rgba="0.13 0.54 0.13 1.0"/>
   </material>
   <link name="world"/>
-<!-- 1st ROBOT -->
   <joint name="world_to_base_A" type="fixed">
+    <origin rpy="0.0 0.0 0.0" xyz="0.6 0.153 0.05"/>
     <parent link="world"/>
     <child link="base_link_A"/>
-    <origin rpy="0 0 0" xyz="0.600 0.153 0.050"/>
   </joint>
   <gazebo>
-      <plugin filename="libxbot2_gz_joint_server.so" name="xbot2_gz_joint_server">
-          <pid>
-            <pid name="BL4104C_1" profile="medium_mot"/>
-            <pid name="meca_axis_1_joint_A" profile="small_mot"/>
-            <pid name="meca_axis_2_joint_A" profile="small_mot"/>
-            <pid name="meca_axis_3_joint_A" profile="small_mot"/>
-            <pid name="meca_axis_4_joint_A" profile="small_mot"/>
-            <pid name="meca_axis_5_joint_A" profile="small_mot"/>
-            <pid name="meca_axis_6_joint_A" profile="small_mot"/>
-          </pid>
-          <gain d="5" name="small_mot" p="100"/>
-      </plugin>
-    </gazebo>
+    <plugin filename="libxbot2_gz_joint_server.so" name="xbot2_gz_joint_server">
+      <pid>
+        <pid name="BL4104C_1" profile="medium_mot"/>
+        <pid name="meca_axis_1_joint_A" profile="small_mot"/>
+        <pid name="meca_axis_2_joint_A" profile="small_mot"/>
+        <pid name="meca_axis_3_joint_A" profile="small_mot"/>
+        <pid name="meca_axis_4_joint_A" profile="small_mot"/>
+        <pid name="meca_axis_5_joint_A" profile="small_mot"/>
+        <pid name="meca_axis_6_joint_A" profile="small_mot"/>
+      </pid>
+      <gain d="5" name="small_mot" p="100"/>
+    </plugin>
+  </gazebo>
   <link name="base_link_A">
     <inertial>
       <mass value="0.1"/>
-      <inertia ixx="1.0e-03" ixy="0.0" ixz="0.0" iyy="1.0e-03" iyz="0.0" izz="1.0e-03"/>
+      <inertia ixx="0.001" ixy="0.0" ixz="0.0" iyy="0.001" iyz="0.0" izz="0.001"/>
     </inertial>
   </link>
   <joint name="fixed_gear_box" type="fixed">
+    <origin rpy="0.0 0.0 1.571" xyz="0.431 0.0 0.05"/>
     <parent link="base_link_A"/>
     <child link="gear_box"/>
-    <origin xyz="0.431 0.0 0.05" rpy="0 0 1.571" />
   </joint>
   <link name="gear_box">
-    <visual>
-      <geometry>
-        <cylinder length="0.366" radius="0.12"/>
-      </geometry>
-      <material name="blue">
-        <color rgba="0 0 .8 1"/>
-      </material>
-      <origin xyz="0.183 0 0" rpy="0 1.571 0" />
-    </visual>
-    <collision>
-      <origin xyz="0.183 0 0" rpy="0 1.571 0" />
-      <geometry>
-        <cylinder length="0.366" radius="0.12" />
-      </geometry>
-    </collision>
-    <inertial>
-      <origin rpy="0 0 0" xyz="0.0 0.0 0.10614489"/>
+    <inertial>
+      <origin rpy="0.0 0.0 0.0" xyz="0.0 0.0 0.10614489"/>
       <mass value="2.0554934"/>
       <inertia ixx="0.01068855" ixy="-1.14168e-05" ixz="2.71689e-06" iyy="0.010584907" iyz="8.76312e-05" izz="0.0032026258"/>
     </inertial>
+    <visual>
+      <origin rpy="0.0 1.571 0.0" xyz="0.183 0.0 0.0"/>
+      <geometry>
+        <cylinder length="0.366" radius="0.12"/>
+      </geometry>
+      <material name="blue">
+        <color rgba="0.0 0.0 0.8 1.0"/>
+      </material>
+    </visual>
+    <collision>
+      <origin rpy="0.0 1.571 0.0" xyz="0.183 0.0 0.0"/>
+      <geometry>
+        <cylinder length="0.366" radius="0.12"/>
+      </geometry>
+    </collision>
+    <collision>
+      <origin rpy="0.0 1.571 0.0" xyz="0.000000 0.000000 0.000037"/>
+      <geometry>
+        <sphere radius="0.12"/>
+      </geometry>
+    </collision>
+    <collision>
+      <origin rpy="0.0 1.571 0.0" xyz="0.366000 0.000000 -0.000037"/>
+      <geometry>
+        <sphere radius="0.12"/>
+      </geometry>
+    </collision>
   </link>
   <joint name="fixed_linear_motor" type="fixed">
+    <origin rpy="0.0 0.0 0.0" xyz="0.0 0.0 0.05"/>
     <parent link="base_link_A"/>
     <child link="linear_motor_stator"/>
-    <origin xyz="0.0 0.0 0.05" rpy="0 0 0" />
   </joint>
   <link name="linear_motor_stator">
-    <visual>
-      <geometry>
-        <box size="0.98 0.12 0.1"/>
-      </geometry>
-      <material name="blue">
-        <color rgba="0 0 .8 1"/>
-      </material>
-      <origin xyz="0 0 0" rpy="0 0 0" />
-    </visual>
-    <collision>
-      <origin xyz="0 0 0.05" rpy="0 1.571 0" />
-      <geometry>
-        <cylinder length="0.98" radius="0.12" />
-      </geometry>
-    </collision>
-    <inertial>
-      <origin rpy="0 0 0" xyz="0.0 0.0 0.10614489"/>
+    <inertial>
+      <origin rpy="0.0 0.0 0.0" xyz="0.0 0.0 0.10614489"/>
       <mass value="2.0554934"/>
       <inertia ixx="0.01068855" ixy="-1.14168e-05" ixz="2.71689e-06" iyy="0.010584907" iyz="8.76312e-05" izz="0.0032026258"/>
     </inertial>
+    <visual>
+      <origin rpy="0.0 0.0 0.0" xyz="0.0 0.0 0.0"/>
+      <geometry>
+        <box size="0.98 0.12 0.1"/>
+      </geometry>
+      <material name="blue">
+        <color rgba="0.0 0.0 0.8 1.0"/>
+      </material>
+    </visual>
+    <collision>
+      <origin rpy="0.0 1.571 0.0" xyz="0.0 0.0 0.05"/>
+      <geometry>
+        <cylinder length="0.98" radius="0.12"/>
+      </geometry>
+    </collision>
+    <collision>
+      <origin rpy="0.0 1.571 0.0" xyz="-0.490000 0.000000 0.050100"/>
+      <geometry>
+        <sphere radius="0.12"/>
+      </geometry>
+    </collision>
+    <collision>
+      <origin rpy="0.0 1.571 0.0" xyz="0.490000 0.000000 0.049900"/>
+      <geometry>
+        <sphere radius="0.12"/>
+      </geometry>
+    </collision>
   </link>
   <gazebo reference="linear_motor_stator">
@@ -115,43 +139,46 @@
   </gazebo>
   <joint name="linear_motor" type="prismatic">
-    <axis xyz="1 0 0"/>
+    <origin rpy="0.0 0.0 0.0" xyz="-0.26 0.0 0.09"/>
+    <axis xyz="1.0 0.0 0.0"/>
     <parent link="linear_motor_stator"/>
     <child link="L_1_A"/>
-    <limit effort="100.0" lower="-0.002" upper="0.400" velocity="0.5"/>
-    <origin rpy="0 0 0" xyz="-0.26 0 0.09"/>
+    <limit effort="100.0" lower="-0.002" upper="0.4" velocity="0.5"/>
   </joint>
   <link name="L_1_A">
-    <visual>
-      <geometry>
-        <box size="0.2 0.2 0.04"/>
-      </geometry>
-      <material name="blue">
-        <color rgba="0 0 .8 1"/>
-      </material>
-      <origin xyz="0 0 -0.02" rpy="0 0 0" />
-    </visual>
-    <collision>
-      <origin xyz="0 0 -0.02" rpy="0 0 0" />
-      <geometry>
-        <box size="0.2 0.2 0.04"/>
-      </geometry>
-    </collision>
-    <inertial>
-      <origin rpy="0 0 0" xyz="0.0 0.0 -0.024438213"/>
+    <inertial>
+      <origin rpy="0.0 0.0 0.0" xyz="0.0 0.0 -0.024438213"/>
       <mass value="0.42322395"/>
       <inertia ixx="0.00063746146" ixy="1.1903424e-05" ixz="6.7230372e-07" iyy="0.00064218987" iyz="2.203073e-05" izz="0.001009674"/>
     </inertial>
+    <visual>
+      <origin rpy="0.0 0.0 0.0" xyz="0.0 0.0 -0.02"/>
+      <geometry>
+        <box size="0.2 0.2 0.04"/>
+      </geometry>
+      <material name="blue">
+        <color rgba="0.0 0.0 0.8 1.0"/>
+      </material>
+    </visual>
+    <collision>
+      <origin rpy="0.0 0.0 0.0" xyz="0.0 0.0 -0.02"/>
+      <geometry>
+        <box size="0.2 0.2 0.04"/>
+      </geometry>
+    </collision>
   </link>
   <joint name="L_1_A_to_meca_base_link_A" type="fixed">
+    <origin rpy="0.0 1.571 1.571" xyz="0.0 0.014 0.0744"/>
     <parent link="L_1_A"/>
     <child link="meca_base_link_A"/>
-    <origin rpy="0 1.571 1.571" xyz="0.0 0.014 0.0744"/>
-  </joint>
-    <!-- Base link is the center of the robot's bottom plate -->
+  </joint>
   <link name="meca_base_link_A">
-    <visual>
-      <origin xyz="0 0 0" rpy="0 0 0" />
-      <geometry>
-        <mesh filename="package://mecademic_description/meshes/meca_500_r3_base.dae" />
+    <inertial>
+      <mass value="1.0"/>
+      <inertia ixx="0.01" ixy="0.0" ixz="0.0" iyy="0.01" iyz="0.0" izz="0.01"/>
+    </inertial>
+    <visual>
+      <origin rpy="0.0 0.0 0.0" xyz="0.0 0.0 0.0"/>
+      <geometry>
+        <mesh filename="package://mecademic_description/meshes/meca_500_r3_base.dae"/>
       </geometry>
     </visual>
@@ -174,15 +201,14 @@
       </geometry>
     </collision>
-    <inertial>
-      <mass value="1"/>
-      <inertia ixx="0.01" ixy="0" ixz="0" iyy="0.01" iyz="0" izz="0.01"/>
-    </inertial>
-  </link>
-  <!-- Joint 1 -->
+  </link>
   <link name="meca_axis_1_link_A">
-    <visual>
-      <origin xyz="0 0 0" rpy="0 0 0" />
-      <geometry>
-        <mesh filename="package://mecademic_description/meshes/meca_500_r3_j1.dae" />
+    <inertial>
+      <mass value="1.0"/>
+      <inertia ixx="0.01" ixy="0.0" ixz="0.0" iyy="0.01" iyz="0.0" izz="0.01"/>
+    </inertial>
+    <visual>
+      <origin rpy="0.0 0.0 0.0" xyz="0.0 0.0 0.0"/>
+      <geometry>
+        <mesh filename="package://mecademic_description/meshes/meca_500_r3_j1.dae"/>
       </geometry>
     </visual>
@@ -205,22 +231,21 @@
       </geometry>
     </collision>
-    <inertial>
-      <mass value="1"/>
-      <inertia ixx="0.01" ixy="0" ixz="0" iyy="0.01" iyz="0" izz="0.01"/>
-    </inertial>
   </link>
   <joint name="meca_axis_1_joint_A" type="revolute">
-    <origin xyz="0.012498 0 0.091" rpy="0 0 0" />
-    <parent link="meca_base_link_A" />
-    <child link="meca_axis_1_link_A" />
-    <axis xyz="0 0 1" />
+    <origin rpy="0.0 0.0 0.0" xyz="0.012498 0.0 0.091"/>
+    <axis xyz="0.0 0.0 1.0"/>
+    <parent link="meca_base_link_A"/>
+    <child link="meca_axis_1_link_A"/>
     <limit effort="10.0" lower="-3.05" upper="3.05" velocity="2.61799"/>
   </joint>
-  <!-- Joint 2 -->
   <link name="meca_axis_2_link_A">
-    <visual>
-      <origin xyz="0 0 0" rpy="0 0 0" />
-      <geometry>
-        <mesh filename="package://mecademic_description/meshes/meca_500_r3_j2.dae" />
+    <inertial>
+      <mass value="1.0"/>
+      <inertia ixx="0.01" ixy="0.0" ixz="0.0" iyy="0.01" iyz="0.0" izz="0.01"/>
+    </inertial>
+    <visual>
+      <origin rpy="0.0 0.0 0.0" xyz="0.0 0.0 0.0"/>
+      <geometry>
+        <mesh filename="package://mecademic_description/meshes/meca_500_r3_j2.dae"/>
       </geometry>
     </visual>
@@ -243,22 +268,21 @@
       </geometry>
     </collision>
-    <inertial>
-      <mass value="1"/>
-      <inertia ixx="0.01" ixy="0" ixz="0" iyy="0.01" iyz="0" izz="0.01"/>
-    </inertial>
   </link>
   <joint name="meca_axis_2_joint_A" type="revolute">
-    <origin xyz="0 0 0.044" rpy="0 0 0" />
-    <parent link="meca_axis_1_link_A" />
-    <child link="meca_axis_2_link_A" />
-    <axis xyz="0 1 0" />
+    <origin rpy="0.0 0.0 0.0" xyz="0.0 0.0 0.044"/>
+    <axis xyz="0.0 1.0 0.0"/>
+    <parent link="meca_axis_1_link_A"/>
+    <child link="meca_axis_2_link_A"/>
     <limit effort="10.0" lower="-1.22" upper="1.57" velocity="2.61799"/>
   </joint>
-  <!-- Joint 3 -->
   <link name="meca_axis_3_link_A">
-    <visual>
-      <origin xyz="0 0 0" rpy="0 0 0" />
-      <geometry>
-        <mesh filename="package://mecademic_description/meshes/meca_500_r3_j3.dae" />
+    <inertial>
+      <mass value="1.0"/>
+      <inertia ixx="0.01" ixy="0.0" ixz="0.0" iyy="0.01" iyz="0.0" izz="0.01"/>
+    </inertial>
+    <visual>
+      <origin rpy="0.0 0.0 0.0" xyz="0.0 0.0 0.0"/>
+      <geometry>
+        <mesh filename="package://mecademic_description/meshes/meca_500_r3_j3.dae"/>
       </geometry>
     </visual>
@@ -281,22 +305,21 @@
       </geometry>
     </collision>
-    <inertial>
-      <mass value="1"/>
-      <inertia ixx="0.01" ixy="0" ixz="0" iyy="0.01" iyz="0" izz="0.01"/>
-    </inertial>
   </link>
   <joint name="meca_axis_3_joint_A" type="revolute">
-    <origin xyz="0 0 0.135" rpy="0 0 0" />
-    <parent link="meca_axis_2_link_A" />
-    <child link="meca_axis_3_link_A" />
-    <axis xyz="0 1 0" />
+    <origin rpy="0.0 0.0 0.0" xyz="0.0 0.0 0.135"/>
+    <axis xyz="0.0 1.0 0.0"/>
+    <parent link="meca_axis_2_link_A"/>
+    <child link="meca_axis_3_link_A"/>
     <limit effort="10.0" lower="-2.35" upper="1.22" velocity="3.14159"/>
   </joint>
-  <!-- Joint 4 -->
   <link name="meca_axis_4_link_A">
-    <visual>
-      <origin xyz="0 0 0" rpy="0 0 0" />
-      <geometry>
-        <mesh filename="package://mecademic_description/meshes/meca_500_r3_j4.dae" />
+    <inertial>
+      <mass value="1.0"/>
+      <inertia ixx="0.01" ixy="0.0" ixz="0.0" iyy="0.01" iyz="0.0" izz="0.01"/>
+    </inertial>
+    <visual>
+      <origin rpy="0.0 0.0 0.0" xyz="0.0 0.0 0.0"/>
+      <geometry>
+        <mesh filename="package://mecademic_description/meshes/meca_500_r3_j4.dae"/>
       </geometry>
     </visual>
@@ -319,22 +342,21 @@
       </geometry>
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
Commit message: reduce dimension of rotary table collision objects (it was exagerated)

File: mecademic_description/urdf/meca_500_r3_capsule.urdf.xacro (robot description, xacro)
@@ -516,5 +516,5 @@
       <origin rpy="0.0 0.0 0.0" xyz="0.0 0.0 0.105"/>
       <geometry>
-        <cylinder length="0.21" radius="0.16"/>
+        <cylinder length="0.21" radius="0.145"/>
       </geometry>
     </collision>
@@ -522,5 +522,5 @@
       <origin rpy="0.0 0.0 0.0" xyz="0.000000 0.000000 0.000000"/>
       <geometry>
-        <sphere radius="0.16"/>
+        <sphere radius="0.145"/>
       </geometry>
     </collision>
@@ -528,5 +528,5 @@
       <origin rpy="0.0 0.0 0.0" xyz="0.000000 0.000000 0.210000"/>
       <geometry>
-        <sphere radius="0.16"/>
+        <sphere radius="0.145"/>
       </geometry>
     </collision>

Commit message: update capsule urdf as well

File: mecademic_description/urdf/meca_500_r3_capsule.urdf.xacro (robot description, xacro)
@@ -938,5 +938,5 @@
   </joint>
   <joint name="world_to_buffer" type="fixed">
-     <origin xyz="0 0.585 0.2" rpy="0 0 0"/>
+    <origin xyz="0 0.650 0.075" rpy="0 0 0"/>
     <parent link="world"/>
     <child link="buffer_base_link"/>
@@ -944,5 +944,5 @@
   <link name="buffer_base_link">
     <visual>
-      <origin xyz="0 0.065 -0.075" rpy="1.57 0 -1.57" />
+      <origin xyz="0 0.0 0.0" rpy="1.57 0 -1.57" />
       <geometry>
         <mesh filename="package://mecademic_description/meshes/buffer_and_slide_support_v17.stl" scale="0.001 0.001 0.001"/>
@@ -950,5 +950,5 @@
     </visual>
     <collision>
-      <origin xyz="0 0.065 -0.075" rpy="1.57 0 -1.57" />
+      <origin xyz="0 0.0 0.0" rpy="1.57 0 -1.57" />
       <geometry>
         <mesh filename="package://mecademic_description/meshes/buffer_and_slide_support_v17.stl" scale="0.001 0.001 0.001"/>
@@ -961,5 +961,5 @@
   </link>
   <joint name="buffer_base_to_1" type="fixed">
-    <origin xyz="0.525 0 0" rpy="0 0 0"/>
+    <origin xyz="0.525 -0.065 0.03" rpy="0 0 0"/>
     <parent link="buffer_base_link"/>
     <child link="buffer_1"/>
@@ -967,5 +967,5 @@
   <link name="buffer_1"/>
   <joint name="buffer_base_to_2" type="fixed">
-        <origin xyz="0.650 0.0 0" rpy="0 0 0"/>
+        <origin xyz="0.650 -0.065 0.03" rpy="0 0 0"/>
         <parent link="buffer_base_link"/>
         <child link="buffer_2"/>
@@ -992,5 +992,5 @@
   <!-- SLIDERS -->
   <joint name="world_to_slider" type="fixed">
-    <origin rpy="0.0 0.0 0.0" xyz="0.0 0.585 0.0"/>
+    <origin xyz="0 0.650 0.0" rpy="0 0 0"/>
     <parent link="world"/>
     <child link="slider_base_link"/>
@@ -998,5 +998,5 @@
   <link name="slider_base_link"/>
   <joint name="slider_base_to_empty" type="fixed">
-    <origin rpy="0.0 0.1745 0.0" xyz="0.397 0.0 0.194"/>
+    <origin xyz="0.397 -0.065 0.194" rpy="0 0.1745 0"/>
     <parent link="slider_base_link"/>
     <child link="empty_container"/>
@@ -1004,5 +1004,5 @@
   <link name="empty_container"/>
   <joint name="sliders_base_to_lid" type="fixed">
-    <origin rpy="0.0 0.1745 0.0" xyz="0.322 0.0 0.319"/>
+    <origin xyz="0.322 -0.065 0.319" rpy="0 0.1745 0"/>
     <parent link="slider_base_link"/>
     <child link="lid"/>
@@ -1010,5 +1010,5 @@
   <link name="lid"/>
   <joint name="sliders_base_to_full" type="fixed">
-    <origin rpy="0.0 0.1745 0.0" xyz="0.809 0.0 0.295"/>
+    <origin xyz="0.809 -0.065 0.295" rpy="0 0.1745 0"/>
     <parent link="slider_base_link"/>
     <child link="full_container"/>
