Commit message: rbdl compatibility (add inertias and world frame)

File: mecademic_description/urdf/meca_500_r3.urdf.xacro (robot description, xacro)
@@ -1,3 +1,8 @@
 <robot name="meca_500_r3" xmlns:xacro="http://ros.org/wiki/xacro">
+  <link name="world"/>
+  <joint name="world" type="fixed">
+    <parent link="world"/>
+    <child link="meca_base_link"/>
+  </joint>
   <!-- Base link is the center of the robot's bottom plate -->
   <link name="meca_base_link">
@@ -14,4 +19,8 @@
       </geometry>
     </collision>
+    <inertial>
+      <mass value="1"/>
+      <inertia ixx="0.01" ixy="0" ixz="0" iyy="0.01" iyz="0" izz="0.01"/>
+    </inertial>
   </link>
   <!-- Joint 1 -->
@@ -29,4 +38,8 @@
       </geometry>
     </collision>
+    <inertial>
+      <mass value="1"/>
+      <inertia ixx="0.01" ixy="0" ixz="0" iyy="0.01" iyz="0" izz="0.01"/>
+    </inertial>
   </link>
   <joint name="meca_axis_1_joint" type="revolute">
@@ -51,4 +64,8 @@
       </geometry>
     </collision>
+    <inertial>
+      <mass value="1"/>
+      <inertia ixx="0.01" ixy="0" ixz="0" iyy="0.01" iyz="0" izz="0.01"/>
+    </inertial>
   </link>
   <joint name="meca_axis_2_joint" type="revolute">
@@ -73,4 +90,8 @@
       </geometry>
     </collision>
+    <inertial>
+      <mass value="1"/>
+      <inertia ixx="0.01" ixy="0" ixz="0" iyy="0.01" iyz="0" izz="0.01"/>
+    </inertial>
   </link>
   <joint name="meca_axis_3_joint" type="revolute">
@@ -95,4 +116,8 @@
       </geometry>
     </collision>
+    <inertial>
+      <mass value="1"/>
+      <inertia ixx="0.01" ixy="0" ixz="0" iyy="0.01" iyz="0" izz="0.01"/>
+    </inertial>
   </link>
   <joint name="meca_axis_4_joint" type="revolute">
@@ -117,4 +142,8 @@
       </geometry>
     </collision>
+    <inertial>
+      <mass value="1"/>
+      <inertia ixx="0.01" ixy="0" ixz="0" iyy="0.01" iyz="0" izz="0.01"/>
+    </inertial>
   </link>
   <joint name="meca_axis_5_joint" type="revolute">
@@ -139,4 +168,8 @@
       </geometry>
     </collision>
+    <inertial>
+      <mass value="1"/>
+      <inertia ixx="0.01" ixy="0" ixz="0" iyy="0.01" iyz="0" izz="0.01"/>
+    </inertial>
   </link>
   <joint name="meca_axis_6_joint" type="revolute">

Commit message: modify joint limits to be more conservative
this to avoid floating point representation issues.
the robot will go in error if it receives a value higher than the limit.

File: mecademic_description/urdf/meca_500_r3.urdf.xacro (robot description, xacro)
@@ -61,5 +61,5 @@
     <child link="meca_axis_1_link" />
     <axis xyz="0 0 1" />
-    <limit effort="10.0" velocity="2.61799" lower="-3.05433" upper="3.05433" />
+    <limit effort="10.0" velocity="2.61799" lower="-3.05" upper="3.05" />
   </joint>
   <!-- Joint 2 -->
@@ -87,5 +87,5 @@
     <child link="meca_axis_2_link" />
     <axis xyz="0 1 0" />
-    <limit effort="10.0" velocity="2.61799" lower="-1.22173048" upper="1.5708" />
+    <limit effort="10.0" velocity="2.61799" lower="-1.22" upper="1.57" />
   </joint>
   <!-- Joint 3 -->
@@ -113,5 +113,5 @@
     <child link="meca_axis_3_link" />
     <axis xyz="0 1 0" />
-    <limit effort="10.0" velocity="3.14159" lower="-2.35619" upper="1.22173048" />
+    <limit effort="10.0" velocity="3.14159" lower="-2.35" upper="1.22" />
   </joint>
   <!-- Joint 4 -->
@@ -139,5 +139,5 @@
     <child link="meca_axis_4_link" />
     <axis xyz="1 0 0" />
-    <limit effort="10.0" velocity="5.23599" lower="-2.96706" upper="2.96706" />
+    <limit effort="10.0" velocity="5.23599" lower="-2.96" upper="2.96" />
   </joint>
   <!-- Joint 5 -->
@@ -165,5 +165,5 @@
     <child link="meca_axis_5_link" />
     <axis xyz="0 1 0" />
-    <limit effort="10.0" velocity="5.23599" lower="-2.00713" upper="2.00713" />
+    <limit effort="10.0" velocity="5.23599" lower="-2.00" upper="2.00" />
   </joint>
   <!-- Joint 6 -->
@@ -191,5 +191,5 @@
     <child link="meca_axis_6_link" />
     <axis xyz="1 0 0" />
-    <limit effort="10.0" velocity="8.72665" lower="-3.14159" upper="3.14159" />
+    <limit effort="10.0" velocity="8.72665" lower="-3.14" upper="3.14" />
   </joint>
 </robot>

File: mecademic_description/urdf/meca_500_r3_capsule.urdf.xacro (robot description, xacro)
@@ -71,5 +71,5 @@
     <parent link="meca_base_link"/>
     <child link="meca_axis_1_link"/>
-    <limit effort="10.0" lower="-3.05433" upper="3.05433" velocity="2.61799"/>
+    <limit effort="10.0" lower="-3.05" upper="3.05" velocity="2.61799"/>
   </joint>
   <link name="meca_axis_2_link">
@@ -108,5 +108,5 @@
     <parent link="meca_axis_1_link"/>
     <child link="meca_axis_2_link"/>
-    <limit effort="10.0" lower="-1.22173048" upper="1.5708" velocity="2.61799"/>
+    <limit effort="10.0" lower="-1.22" upper="1.57" velocity="2.61799"/>
   </joint>
   <link name="meca_axis_3_link">
@@ -145,5 +145,5 @@
     <parent link="meca_axis_2_link"/>
     <child link="meca_axis_3_link"/>
-    <limit effort="10.0" lower="-2.35619" upper="1.22173048" velocity="3.14159"/>
+    <limit effort="10.0" lower="-2.35" upper="1.22" velocity="3.14159"/>
   </joint>
   <link name="meca_axis_4_link">
@@ -182,5 +182,5 @@
     <parent link="meca_axis_3_link"/>
     <child link="meca_axis_4_link"/>
-    <limit effort="10.0" lower="-2.96706" upper="2.96706" velocity="5.23599"/>
+    <limit effort="10.0" lower="-2.96" upper="2.96" velocity="5.23599"/>
   </joint>
   <link name="meca_axis_5_link">
@@ -219,5 +219,5 @@
     <parent link="meca_axis_4_link"/>
     <child link="meca_axis_5_link"/>
-    <limit effort="10.0" lower="-2.00713" upper="2.00713" velocity="5.23599"/>
+    <limit effort="10.0" lower="-2.00" upper="2.00" velocity="5.23599"/>
   </joint>
   <link name="meca_axis_6_link">
@@ -256,5 +256,5 @@
     <parent link="meca_axis_5_link"/>
     <child link="meca_axis_6_link"/>
-    <limit effort="10.0" lower="-3.14159" upper="3.14159" velocity="8.72665"/>
+    <limit effort="10.0" lower="-3.14" upper="3.14" velocity="8.72665"/>
   </joint>
 </robot>

Commit message: update problem and robot description: 2 meca and 2 buffers

File: mecademic_description/urdf/meca_500_r3.urdf.xacro (robot description, xacro)
@@ -1,10 +1,10 @@
 <robot name="meca_500_r3" xmlns:xacro="http://ros.org/wiki/xacro">
   <link name="world"/>
-  <joint name="world" type="fixed">
+  <joint name="world_A" type="fixed">
     <parent link="world"/>
-    <child link="meca_base_link"/>
+    <child link="meca_base_link_A"/>
   </joint>
   <!-- Base link is the center of the robot's bottom plate -->
-  <link name="meca_base_link">
+  <link name="meca_base_link_A">
     <visual>
       <origin xyz="0 0 0" rpy="0 0 0" />
@@ -27,10 +27,10 @@
       <plugin filename="libxbot2_gz_joint_server.so" name="xbot2_gz_joint_server">
          <pid>
-            <pid name="meca_axis_1_joint" profile="small_mot"/>
-            <pid name="meca_axis_2_joint" profile="small_mot"/>
-            <pid name="meca_axis_3_joint" profile="small_mot"/>
-            <pid name="meca_axis_4_joint" profile="small_mot"/>
-            <pid name="meca_axis_5_joint" profile="small_mot"/>
-            <pid name="meca_axis_6_joint" profile="small_mot"/>
+            <pid name="meca_axis_1_joint_A" profile="small_mot"/>
+            <pid name="meca_axis_2_joint_A" profile="small_mot"/>
+            <pid name="meca_axis_3_joint_A" profile="small_mot"/>
+            <pid name="meca_axis_4_joint_A" profile="small_mot"/>
+            <pid name="meca_axis_5_joint_A" profile="small_mot"/>
+            <pid name="meca_axis_6_joint_A" profile="small_mot"/>
          </pid>
          <gain d="5" name="small_mot" p="100"/>
@@ -38,5 +38,5 @@
    </gazebo>
   <!-- Joint 1 -->
-  <link name="meca_axis_1_link">
+  <link name="meca_axis_1_link_A">
     <visual>
       <origin xyz="0 0 0" rpy="0 0 0" />
@@ -56,13 +56,13 @@
     </inertial>
   </link>
-  <joint name="meca_axis_1_joint" type="revolute">
+  <joint name="meca_axis_1_joint_A" type="revolute">
     <origin xyz="0.012498 0 0.091" rpy="0 0 0" />
-    <parent link="meca_base_link" />
-    <child link="meca_axis_1_link" />
+    <parent link="meca_base_link_A" />
+    <child link="meca_axis_1_link_A" />
     <axis xyz="0 0 1" />
     <limit effort="10.0" velocity="2.61799" lower="-3.05433" upper="3.05433" />
   </joint>
   <!-- Joint 2 -->
-  <link name="meca_axis_2_link">
+  <link name="meca_axis_2_link_A">
     <visual>
       <origin xyz="0 0 0" rpy="0 0 0" />
@@ -82,13 +82,13 @@
     </inertial>
   </link>
-  <joint name="meca_axis_2_joint" type="revolute">
+  <joint name="meca_axis_2_joint_A" type="revolute">
     <origin xyz="0 0 0.044" rpy="0 0 0" />
-    <parent link="meca_axis_1_link" />
-    <child link="meca_axis_2_link" />
+    <parent link="meca_axis_1_link_A" />
+    <child link="meca_axis_2_link_A" />
     <axis xyz="0 1 0" />
     <limit effort="10.0" velocity="2.61799" lower="-1.22173048" upper="1.5708" />
   </joint>
   <!-- Joint 3 -->
-  <link name="meca_axis_3_link">
+  <link name="meca_axis_3_link_A">
     <visual>
       <origin xyz="0 0 0" rpy="0 0 0" />
@@ -108,13 +108,13 @@
     </inertial>
   </link>
-  <joint name="meca_axis_3_joint" type="revolute">
+  <joint name="meca_axis_3_joint_A" type="revolute">
     <origin xyz="0 0 0.135" rpy="0 0 0" />
-    <parent link="meca_axis_2_link" />
-    <child link="meca_axis_3_link" />
+    <parent link="meca_axis_2_link_A" />
+    <child link="meca_axis_3_link_A" />
     <axis xyz="0 1 0" />
     <limit effort="10.0" velocity="3.14159" lower="-2.35619" upper="1.22173048" />
   </joint>
   <!-- Joint 4 -->
-  <link name="meca_axis_4_link">
+  <link name="meca_axis_4_link_A">
     <visual>
       <origin xyz="0 0 0" rpy="0 0 0" />
@@ -134,13 +134,13 @@
     </inertial>
   </link>
-  <joint name="meca_axis_4_joint" type="revolute">
+  <joint name="meca_axis_4_joint_A" type="revolute">
     <origin xyz="0 0 0.038" rpy="0 0 0" />
-    <parent link="meca_axis_3_link" />
-    <child link="meca_axis_4_link" />
+    <parent link="meca_axis_3_link_A" />
+    <child link="meca_axis_4_link_A" />
     <axis xyz="1 0 0" />
     <limit effort="10.0" velocity="5.23599" lower="-2.96706" upper="2.96706" />
   </joint>
   <!-- Joint 5 -->
-  <link name="meca_axis_5_link">
+  <link name="meca_axis_5_link_A">
     <visual>
       <origin xyz="0 0 0" rpy="0 0 0" />
@@ -160,13 +160,13 @@
     </inertial>
   </link>
-  <joint name="meca_axis_5_joint" type="revolute">
+  <joint name="meca_axis_5_joint_A" type="revolute">
     <origin xyz="0.12 0 0" rpy="0 0 0" />
-    <parent link="meca_axis_4_link" />
-    <child link="meca_axis_5_link" />
+    <parent link="meca_axis_4_link_A" />
+    <child link="meca_axis_5_link_A" />
     <axis xyz="0 1 0" />
     <limit effort="10.0" velocity="5.23599" lower="-2.00713" upper="2.00713" />
   </joint>
   <!-- Joint 6 -->
-  <link name="meca_axis_6_link">
+  <link name="meca_axis_6_link_A">
     <visual>
       <origin xyz="0 0 0" rpy="0 0 0" />
@@ -186,10 +186,223 @@
     </inertial>
   </link>
-  <joint name="meca_axis_6_joint" type="revolute">
+  <joint name="meca_axis_6_joint_A" type="revolute">
     <origin xyz="0.07 0 0" rpy="0 0 0" />
-    <parent link="meca_axis_5_link" />
-    <child link="meca_axis_6_link" />
+    <parent link="meca_axis_5_link_A" />
+    <child link="meca_axis_6_link_A" />
     <axis xyz="1 0 0" />
-    <limit effort="10.0" velocity="8.72665" lower="-3.14159" upper="3.14159" />
-  </joint>
+    <limit effort="10.0" velocity="8.72665" lower="-4.712" upper="4.712" />
+  </joint>
+<!-- 2nd ROBOT -->
+  <joint name="world_B" type="fixed">
+      <origin xyz="0.3 0.3 0" rpy="0 0 0"/>
+      <parent link="world"/>
+      <child link="meca_base_link_B"/>
+    </joint>
+    <!-- Base link is the center of the robot's bottom plate -->
+  <link name="meca_base_link_B">
+    <visual>
+      <origin xyz="0 0 0" rpy="0 0 0" />
+      <geometry>
+        <mesh filename="package://mecademic_description/meshes/meca_500_r3_base.dae" />
+      </geometry>
+    </visual>
+    <collision>
+      <origin xyz="0 0 0" rpy="0 0 0" />
+      <geometry>
+        <mesh filename="package://mecademic_description/meshes/meca_500_r3_base_collision.stl" />
+      </geometry>
+    </collision>
+    <inertial>
+      <mass value="1"/>
+      <inertia ixx="0.01" ixy="0" ixz="0" iyy="0.01" iyz="0" izz="0.01"/>
+    </inertial>
+  </link>
+  <gazebo>
+      <plugin filename="libxbot2_gz_joint_server.so" name="xbot2_gz_joint_server">
+          <pid>
+            <pid name="meca_axis_1_joint_B" profile="small_mot"/>
+            <pid name="meca_axis_2_joint_B" profile="small_mot"/>
+            <pid name="meca_axis_3_joint_B" profile="small_mot"/>
+            <pid name="meca_axis_4_joint_B" profile="small_mot"/>
+            <pid name="meca_axis_5_joint_B" profile="small_mot"/>
+            <pid name="meca_axis_6_joint_B" profile="small_mot"/>
+          </pid>
+          <gain d="5" name="small_mot" p="100"/>
+      </plugin>
+    </gazebo>
+  <!-- Joint 1 -->
+  <link name="meca_axis_1_link_B">
+    <visual>
+      <origin xyz="0 0 0" rpy="0 0 0" />
+      <geometry>
+        <mesh filename="package://mecademic_description/meshes/meca_500_r3_j1.dae" />
+      </geometry>
+    </visual>
+    <collision>
+      <origin xyz="0 0 0" rpy="0 0 0" />
+      <geometry>
+        <mesh filename="package://mecademic_description/meshes/meca_500_r3_j1_collision.stl" />
+      </geometry>
+    </collision>
+    <inertial>
+      <mass value="1"/>
+      <inertia ixx="0.01" ixy="0" ixz="0" iyy="0.01" iyz="0" izz="0.01"/>
+    </inertial>
+  </link>
+  <joint name="meca_axis_1_joint_B" type="revolute">
+    <origin xyz="0.012498 0 0.091" rpy="0 0 0" />
+    <parent link="meca_base_link_B" />
+    <child link="meca_axis_1_link_B" />
+    <axis xyz="0 0 1" />
+    <limit effort="10.0" velocity="2.61799" lower="-3.05433" upper="3.05433" />
+  </joint>
+  <!-- Joint 2 -->
+  <link name="meca_axis_2_link_B">
+    <visual>
+      <origin xyz="0 0 0" rpy="0 0 0" />
+      <geometry>
+        <mesh filename="package://mecademic_description/meshes/meca_500_r3_j2.dae" />
+      </geometry>
+    </visual>
+    <collision>
+      <origin xyz="0 0 0" rpy="0 0 0" />
+      <geometry>
+        <mesh filename="package://mecademic_description/meshes/meca_500_r3_j2_collision.stl" />
+      </geometry>
+    </collision>
+    <inertial>
+      <mass value="1"/>
+      <inertia ixx="0.01" ixy="0" ixz="0" iyy="0.01" iyz="0" izz="0.01"/>
+    </inertial>
+  </link>
+  <joint name="meca_axis_2_joint_B" type="revolute">
+    <origin xyz="0 0 0.044" rpy="0 0 0" />
+    <parent link="meca_axis_1_link_B" />
+    <child link="meca_axis_2_link_B" />
+    <axis xyz="0 1 0" />
+    <limit effort="10.0" velocity="2.61799" lower="-1.22173048" upper="1.5708" />
+  </joint>
+  <!-- Joint 3 -->
+  <link name="meca_axis_3_link_B">
+    <visual>
+      <origin xyz="0 0 0" rpy="0 0 0" />
+      <geometry>
+        <mesh filename="package://mecademic_description/meshes/meca_500_r3_j3.dae" />
+      </geometry>
+    </visual>
+    <collision>
+      <origin xyz="0 0 0" rpy="0 0 0" />
+      <geometry>
+        <mesh filename="package://mecademic_description/meshes/meca_500_r3_j3_collision.stl" />
+      </geometry>
+    </collision>
+    <inertial>
+      <mass value="1"/>
+      <inertia ixx="0.01" ixy="0" ixz="0" iyy="0.01" iyz="0" izz="0.01"/>
+    </inertial>
+  </link>
+  <joint name="meca_axis_3_joint_B" type="revolute">
+    <origin xyz="0 0 0.135" rpy="0 0 0" />
+    <parent link="meca_axis_2_link_B" />
+    <child link="meca_axis_3_link_B" />
+    <axis xyz="0 1 0" />
+    <limit effort="10.0" velocity="3.14159" lower="-2.35619" upper="1.22173048" />
+  </joint>
+  <!-- Joint 4 -->
+  <link name="meca_axis_4_link_B">
+    <visual>
+      <origin xyz="0 0 0" rpy="0 0 0" />
+      <geometry>
+        <mesh filename="package://mecademic_description/meshes/meca_500_r3_j4.dae" />
+      </geometry>
+    </visual>
+    <collision>
+      <origin xyz="0 0 0" rpy="0 0 0" />
+      <geometry>
+        <mesh filename="package://mecademic_description/meshes/meca_500_r3_j4_collision.stl" />
+      </geometry>
+    </collision>
+    <inertial>
+      <mass value="1"/>
+      <inertia ixx="0.01" ixy="0" ixz="0" iyy="0.01" iyz="0" izz="0.01"/>
+    </inertial>
+  </link>
+  <joint name="meca_axis_4_joint_B" type="revolute">
+    <origin xyz="0 0 0.038" rpy="0 0 0" />
+    <parent link="meca_axis_3_link_B" />
+    <child link="meca_axis_4_link_B" />
+    <axis xyz="1 0 0" />
+    <limit effort="10.0" velocity="5.23599" lower="-2.96706" upper="2.96706" />
+  </joint>
+  <!-- Joint 5 -->
+  <link name="meca_axis_5_link_B">
+    <visual>
+      <origin xyz="0 0 0" rpy="0 0 0" />
+      <geometry>
+        <mesh filename="package://mecademic_description/meshes/meca_500_r3_j5.dae" />
+      </geometry>
+    </visual>
+    <collision>
+      <origin xyz="0 0 0" rpy="0 0 0" />
+      <geometry>
+        <mesh filename="package://mecademic_description/meshes/meca_500_r3_j5_collision.stl" />
+      </geometry>
+    </collision>
+    <inertial>
+      <mass value="1"/>
+      <inertia ixx="0.01" ixy="0" ixz="0" iyy="0.01" iyz="0" izz="0.01"/>
+    </inertial>
+  </link>
+  <joint name="meca_axis_5_joint_B" type="revolute">
+    <origin xyz="0.12 0 0" rpy="0 0 0" />
+    <parent link="meca_axis_4_link_B" />
+    <child link="meca_axis_5_link_B" />
+    <axis xyz="0 1 0" />
+    <limit effort="10.0" velocity="5.23599" lower="-2.00713" upper="2.00713" />
+  </joint>
+  <!-- Joint 6 -->
+  <link name="meca_axis_6_link_B">
+    <visual>
+      <origin xyz="0 0 0" rpy="0 0 0" />
+      <geometry>
+        <mesh filename="package://mecademic_description/meshes/meca_500_r3_j6.dae" />
+      </geometry>
+    </visual>
+    <collision>
+      <origin xyz="0 0 0" rpy="0 0 0" />
+      <geometry>
+        <mesh filename="package://mecademic_description/meshes/meca_500_r3_j6_collision.stl" />
+      </geometry>
+    </collision>
+    <inertial>
+      <mass value="1"/>
+      <inertia ixx="0.01" ixy="0" ixz="0" iyy="0.01" iyz="0" izz="0.01"/>
+    </inertial>
+  </link>
+  <joint name="meca_axis_6_joint_B" type="revolute">
+    <origin xyz="0.07 0 0" rpy="0 0 0" />
+    <parent link="meca_axis_5_link_B" />
+    <child link="meca_axis_6_link_B" />
+    <axis xyz="1 0 0" />
+    <limit effort="10.0" velocity="8.72665" lower="-4.712" upper="4.712" />
+  </joint>
+  <!-- BUFFERS -->
+  <joint name="world_buffer" type="fixed">
+    <origin xyz="0.15 0.1 0.1" rpy="0 0 0"/>
+    <parent link="world"/>
+    <child link="buffer_base_link"/>
+  </joint>
+  <link name="buffer_base_link"/>
+  <joint name="buffer_base_to_1" type="fixed">
+    <origin xyz="0 0 0" rpy="0 0 0"/>
+    <parent link="buffer_base_link"/>
+    <child link="buffer_1"/>
+  </joint>
+  <link name="buffer_1"/>
+  <joint name="buffer_1_to_2" type="fixed">
+        <origin xyz="0.1 0.0 0" rpy="0 0 0"/>
+        <parent link="buffer_1"/>
+        <child link="buffer_2"/>
+      </joint>
+  <link name="buffer_2"/>
 </robot>

Commit message: update robot description: add sliders and mill

File: mecademic_description/urdf/meca_500_r3.urdf.xacro (robot description, xacro)
@@ -195,5 +195,5 @@
 <!-- 2nd ROBOT -->
   <joint name="world_B" type="fixed">
-      <origin xyz="0.3 0.3 0" rpy="0 0 0"/>
+      <origin xyz="0.2 0.25 0" rpy="0 0 0"/>
       <parent link="world"/>
       <child link="meca_base_link_B"/>
@@ -388,6 +388,6 @@
   </joint>
   <!-- BUFFERS -->
-  <joint name="world_buffer" type="fixed">
-    <origin xyz="0.15 0.1 0.1" rpy="0 0 0"/>
+  <joint name="world_to_buffer" type="fixed">
+    <origin xyz="0.1 0.1 0.1" rpy="0 0 0"/>
     <parent link="world"/>
     <child link="buffer_base_link"/>
@@ -406,3 +406,41 @@
       </joint>
   <link name="buffer_2"/>
+  <!-- CANDY MILL -->
+  <joint name="world_to_mill" type="fixed">
+    <origin xyz="0.4 0.25 0.1" rpy="0 0 0"/>
+    <parent link="world"/>
+    <child link="mill_base_link"/>
+  </joint>
+  <link name="mill_base_link"/>
+  <joint name="mill_base_to_stick" type="fixed">
+    <origin xyz="0 0 0.15" rpy="0 0 0"/>
+    <parent link="mill_base_link"/>
+    <child link="mill_stick"/>
+  </joint>
+  <link name="mill_stick"/>
+  <!-- SLIDERS -->
+  <joint name="world_to_slider" type="fixed">
+    <origin xyz="0.1 0 0.1" rpy="0 0 0"/>
+    <parent link="world"/>
+    <child link="slider_base_link"/>
+  </joint>
+  <link name="slider_base_link"/>
+  <joint name="slider_base_to_empty" type="fixed">
+    <origin xyz="0 0 0" rpy="0 0 0"/>
+    <parent link="slider_base_link"/>
+    <child link="empty_container"/>
+  </joint>
+  <link name="empty_container"/>
+  <joint name="sliders_empty_to_lid" type="fixed">
+        <origin xyz="0.1 0.0 0" rpy="0 0 0"/>
+        <parent link="empty_container"/>
+        <child link="lid"/>
+      </joint>
+  <link name="lid"/>
+  <joint name="sliders_base_to_full" type="fixed">
+        <origin xyz="0 -0.1 0" rpy="0 0 0"/>
+        <parent link="slider_base_link"/>
+        <child link="full_container"/>
+      </joint>
+  <link name="full_container"/>
 </robot>

Commit message: fix robot description: buffers and sliders wrong poses

File: mecademic_description/urdf/meca_500_r3.urdf.xacro (robot description, xacro)
@@ -195,5 +195,5 @@
 <!-- 2nd ROBOT -->
   <joint name="world_B" type="fixed">
-      <origin xyz="0.2 0.25 0" rpy="0 0 0"/>
+      <origin xyz="0.2 0.3 0" rpy="0 0 0"/>
       <parent link="world"/>
       <child link="meca_base_link_B"/>
@@ -389,5 +389,5 @@
   <!-- BUFFERS -->
   <joint name="world_to_buffer" type="fixed">
-    <origin xyz="0.1 0.1 0.1" rpy="0 0 0"/>
+    <origin xyz="0.2 0.1 0.1" rpy="0 0 0"/>
     <parent link="world"/>
     <child link="buffer_base_link"/>
@@ -400,7 +400,7 @@
   </joint>
   <link name="buffer_1"/>
-  <joint name="buffer_1_to_2" type="fixed">
+  <joint name="buffer_base_to_2" type="fixed">
         <origin xyz="0.1 0.0 0" rpy="0 0 0"/>
-        <parent link="buffer_1"/>
+        <parent link="buffer_base_link"/>
         <child link="buffer_2"/>
       </joint>
@@ -408,5 +408,5 @@
   <!-- CANDY MILL -->
   <joint name="world_to_mill" type="fixed">
-    <origin xyz="0.4 0.25 0.1" rpy="0 0 0"/>
+    <origin xyz="0.45 0.3 0.1" rpy="0 0 0"/>
     <parent link="world"/>
     <child link="mill_base_link"/>
@@ -421,5 +421,5 @@
   <!-- SLIDERS -->
   <joint name="world_to_slider" type="fixed">
-    <origin xyz="0.1 0 0.1" rpy="0 0 0"/>
+    <origin xyz="0.2 0 0.1" rpy="0 0 0"/>
     <parent link="world"/>
     <child link="slider_base_link"/>
@@ -432,7 +432,7 @@
   </joint>
   <link name="empty_container"/>
-  <joint name="sliders_empty_to_lid" type="fixed">
+  <joint name="sliders_base_to_lid" type="fixed">
         <origin xyz="0.1 0.0 0" rpy="0 0 0"/>
-        <parent link="empty_container"/>
+        <parent link="slider_base_link"/>
         <child link="lid"/>
       </joint>
