Commit message: add rotary joint under meca

File: mecademic_description/urdf/meca_500_r3.urdf.xacro (robot description, xacro)
@@ -1,5 +1,5 @@
 <robot name="meca_500_r3" xmlns:xacro="http://ros.org/wiki/xacro">
   <link name="world"/>
-  <joint name="world_A" type="fixed">
+  <joint name="world_to_meca_A" type="fixed">
     <parent link="world"/>
     <child link="meca_base_link_A"/>
@@ -194,31 +194,13 @@
   </joint>
 <!-- 2nd ROBOT -->
-  <joint name="world_B" type="fixed">
+  <joint name="world_to_meca_B" type="fixed">
       <origin xyz="0.2 0.3 0" rpy="0 0 0"/>
       <parent link="world"/>
-      <child link="meca_base_link_B"/>
+      <child link="base_link_B"/>
     </joint>
-    <!-- Base link is the center of the robot's bottom plate -->
-  <link name="meca_base_link_B">
-    <visual>
-      <origin xyz="0 0 0" rpy="0 0 0" />
-      <geometry>
-        <mesh filename="package://mecademic_description/meshes/meca_500_r3_base.dae" />
-      </geometry>
-    </visual>
-    <collision>
-      <origin xyz="0 0 0" rpy="0 0 0" />
-      <geometry>
-        <mesh filename="package://mecademic_description/meshes/meca_500_r3_base_collision.stl" />
-      </geometry>
-    </collision>
-    <inertial>
-      <mass value="1"/>
-      <inertia ixx="0.01" ixy="0" ixz="0" iyy="0.01" iyz="0" izz="0.01"/>
-    </inertial>
-  </link>
   <gazebo>
       <plugin filename="libxbot2_gz_joint_server.so" name="xbot2_gz_joint_server">
           <pid>
+            <pid name="J1_B" profile="small_mot"/>
             <pid name="meca_axis_1_joint_B" profile="small_mot"/>
             <pid name="meca_axis_2_joint_B" profile="small_mot"/>
@@ -231,4 +213,57 @@
       </plugin>
     </gazebo>
+  <link name="base_link_B">
+    <inertial>
+      <mass value="10.0"/>
+      <inertia ixx="1.0e-03" ixy="0.0" ixz="0.0" iyy="1.0e-03" iyz="0.0" izz="1.0e-03"/>
+    </inertial>
+  </link>
+  <joint name="J1_B" type="revolute">
+    <axis xyz="0 0 1"/>
+    <limit effort="1000.0" lower="-6.28" upper="6.28" velocity="100"/>
+    <origin rpy="0 0 0" xyz="0.0 0.0 0.05"/>
+    <parent link="base_link_B"/>
+    <child link="L_1_B"/>
+  </joint>
+  <link name="L_1_B">
+    <visual>
+      <geometry>
+        <cylinder length="0.1" radius="0.1"/>
+      </geometry>
+      <material name="blue">
+        <color rgba="0 0 .8 1"/>
+      </material>
+    </visual>
+    <collision>
+      <origin xyz="0 0 0" rpy="0 0 0" />
+      <geometry>
+        <cylinder length="0.1" radius="0.1"/>
+      </geometry>
+    </collision>
+  </link>
+  <joint name="L_1_B_to_meca_base_link_B" type="fixed">
+    <parent link="L_1_B"/>
+    <child link="meca_base_link_B"/>
+    <origin rpy="0 0.7854 0" xyz="0.0 0.0 0.1"/>
+  </joint>
+    <!-- Base link is the center of the robot's bottom plate -->
+  <link name="meca_base_link_B">
+    <visual>
+      <origin xyz="0 0 0" rpy="0 0 0" />
+      <geometry>
+        <mesh filename="package://mecademic_description/meshes/meca_500_r3_base.dae" />
+      </geometry>
+    </visual>
+    <collision>
+      <origin xyz="0 0 0" rpy="0 0 0" />
+      <geometry>
+        <mesh filename="package://mecademic_description/meshes/meca_500_r3_base_collision.stl" />
+      </geometry>
+    </collision>
+    <inertial>
+      <mass value="1"/>
+      <inertia ixx="0.01" ixy="0" ixz="0" iyy="0.01" iyz="0" izz="0.01"/>
+    </inertial>
+  </link>
   <!-- Joint 1 -->
   <link name="meca_axis_1_link_B">

File: mecademic_description/urdf/meca_500_r3_capsule.urdf.xacro (robot description, xacro)
@@ -278,9 +278,57 @@
   </joint>
 <!-- 2nd ROBOT -->
-  <joint name="world_B" type="fixed">
+ <joint name="world_to_meca_B" type="fixed">
       <origin xyz="0.2 0.3 0" rpy="0 0 0"/>
       <parent link="world"/>
-      <child link="meca_base_link_B"/>
+      <child link="base_link_B"/>
     </joint>
+  <gazebo>
+      <plugin filename="libxbot2_gz_joint_server.so" name="xbot2_gz_joint_server">
+          <pid>
+            <pid name="J1_B" profile="small_mot"/>
+            <pid name="meca_axis_1_joint_B" profile="small_mot"/>
+            <pid name="meca_axis_2_joint_B" profile="small_mot"/>
+            <pid name="meca_axis_3_joint_B" profile="small_mot"/>
+            <pid name="meca_axis_4_joint_B" profile="small_mot"/>
+            <pid name="meca_axis_5_joint_B" profile="small_mot"/>
+            <pid name="meca_axis_6_joint_B" profile="small_mot"/>
+          </pid>
+          <gain d="5" name="small_mot" p="100"/>
+      </plugin>
+    </gazebo>
+  <link name="base_link_B">
+    <inertial>
+      <mass value="10.0"/>
+      <inertia ixx="1.0e-03" ixy="0.0" ixz="0.0" iyy="1.0e-03" iyz="0.0" izz="1.0e-03"/>
+    </inertial>
+  </link>
+  <joint name="J1_B" type="revolute">
+    <axis xyz="0 0 1"/>
+    <limit effort="1000.0" lower="-6.28" upper="6.28" velocity="100"/>
+    <origin rpy="0 0 0" xyz="0.0 0.0 0.05"/>
+    <parent link="base_link_B"/>
+    <child link="L_1_B"/>
+  </joint>
+  <link name="L_1_B">
+    <visual>
+      <geometry>
+        <cylinder length="0.1" radius="0.1"/>
+      </geometry>
+      <material name="blue">
+        <color rgba="0 0 .8 1"/>
+      </material>
+    </visual>
+    <collision>
+      <origin xyz="0 0 0" rpy="0 0 0" />
+      <geometry>
+        <cylinder length="0.1" radius="0.1"/>
+      </geometry>
+    </collision>
+  </link>
+  <joint name="L_1_B_to_meca_base_link_B" type="fixed">
+    <parent link="L_1_B"/>
+    <child link="meca_base_link_B"/>
+    <origin rpy="0 0.7854 0" xyz="0.0 0.0 0.1"/>
+  </joint>
     <!-- Base link is the center of the robot's bottom plate -->
   <link name="meca_base_link_B">

Commit message: add linear joint

File: mecademic_description/urdf/meca_500_r3.urdf.xacro (robot description, xacro)
@@ -1,30 +1,13 @@
 <robot name="meca_500_r3" xmlns:xacro="http://ros.org/wiki/xacro">
   <link name="world"/>
-  <joint name="world_to_meca_A" type="fixed">
+  <joint name="world_to_base_A" type="fixed">
     <parent link="world"/>
-    <child link="meca_base_link_A"/>
-  </joint>
-  <!-- Base link is the center of the robot's bottom plate -->
-  <link name="meca_base_link_A">
-    <visual>
-      <origin xyz="0 0 0" rpy="0 0 0" />
-      <geometry>
-        <mesh filename="package://mecademic_description/meshes/meca_500_r3_base.dae" />
-      </geometry>
-    </visual>
-    <collision>
-      <origin xyz="0 0 0" rpy="0 0 0" />
-      <geometry>
-        <mesh filename="package://mecademic_description/meshes/meca_500_r3_base_collision.stl" />
-      </geometry>
-    </collision>
-    <inertial>
-      <mass value="1"/>
-      <inertia ixx="0.01" ixy="0" ixz="0" iyy="0.01" iyz="0" izz="0.01"/>
-    </inertial>
-  </link>
+    <child link="base_link_A"/>
+    <origin rpy="0 0 0" xyz="0.3 0.0 0.0"/>
+  </joint>
   <gazebo>
       <plugin filename="libxbot2_gz_joint_server.so" name="xbot2_gz_joint_server">
          <pid>
+            <pid name="J1_A" profile="small_mot"/>
             <pid name="meca_axis_1_joint_A" profile="small_mot"/>
             <pid name="meca_axis_2_joint_A" profile="small_mot"/>
@@ -37,4 +20,58 @@
       </plugin>
    </gazebo>
+  <link name="base_link_A">
+    <inertial>
+      <mass value="10.0"/>
+      <inertia ixx="1.0e-03" ixy="0.0" ixz="0.0" iyy="1.0e-03" iyz="0.0" izz="1.0e-03"/>
+    </inertial>
+  </link>
+  <joint name="fixed_L_1_A" type="fixed">
+    <parent link="base_link_A"/>
+    <child link="L_1_A"/>
+    <origin xyz="0.0 0.0 0.05" rpy="0 0 0" />
+  </joint>
+  <link name="L_1_A">
+    <visual>
+      <geometry>
+        <box size="0.6 0.1 0.1"/>
+      </geometry>
+      <material name="blue">
+        <color rgba="0 0 .8 1"/>
+      </material>
+      <origin xyz="0 0 0.0" rpy="0 0 0" />
+    </visual>
+    <collision>
+      <origin xyz="0 0 0" rpy="0 0 0" />
+      <geometry>
+        <box size="0.6 0.1 0.1"/>
+      </geometry>
+    </collision>
+  </link>
+  <joint name="J1_A" type="prismatic">
+    <axis xyz="0 1 0"/>
+    <parent link="L_1_A"/>
+    <child link="meca_base_link_A"/>
+    <limit effort="1000.0" lower="-0.3" upper="0.3" velocity="100"/>
+    <origin rpy="0 1.571 1.571" xyz="0 0.05 0.1"/>
+  </joint>
+  <!-- Base link is the center of the robot's bottom plate -->
+  <link name="meca_base_link_A">
+    <visual>
+      <origin xyz="0 0 0" rpy="0 0 0" />
+      <geometry>
+        <mesh filename="package://mecademic_description/meshes/meca_500_r3_base.dae" />
+      </geometry>
+    </visual>
+    <collision>
+      <origin xyz="0 0 0" rpy="0 0 0" />
+      <geometry>
+        <mesh filename="package://mecademic_description/meshes/meca_500_r3_base_collision.stl" />
+      </geometry>
+    </collision>
+    <inertial>
+      <mass value="1"/>
+      <inertia ixx="0.01" ixy="0" ixz="0" iyy="0.01" iyz="0" izz="0.01"/>
+    </inertial>
+  </link>
   <!-- Joint 1 -->
   <link name="meca_axis_1_link_A">
@@ -194,6 +231,6 @@
   </joint>
 <!-- 2nd ROBOT -->
-  <joint name="world_to_meca_B" type="fixed">
-      <origin xyz="0.2 0.3 0" rpy="0 0 0"/>
+  <joint name="world_to_base_B" type="fixed">
+      <origin xyz="0.3 0.6 0" rpy="0 0 0"/>
       <parent link="world"/>
       <child link="base_link_B"/>
@@ -222,5 +259,5 @@
     <axis xyz="0 0 1"/>
     <limit effort="1000.0" lower="-6.28" upper="6.28" velocity="100"/>
-    <origin rpy="0 0 0" xyz="0.0 0.0 0.05"/>
+    <origin rpy="0 0 0" xyz="0.0 0.0 0.075"/>
     <parent link="base_link_B"/>
     <child link="L_1_B"/>
@@ -229,5 +266,5 @@
     <visual>
       <geometry>
-        <cylinder length="0.1" radius="0.1"/>
+        <cylinder length="0.15" radius="0.1"/>
       </geometry>
       <material name="blue">
@@ -238,5 +275,5 @@
       <origin xyz="0 0 0" rpy="0 0 0" />
       <geometry>
-        <cylinder length="0.1" radius="0.1"/>
+        <cylinder length="0.15" radius="0.1"/>
       </geometry>
     </collision>
@@ -245,5 +282,5 @@
     <parent link="L_1_B"/>
     <child link="meca_base_link_B"/>
-    <origin rpy="0 0.7854 0" xyz="0.0 0.0 0.1"/>
+    <origin rpy="0 1.571 0" xyz="0.05 0.0 0.125"/>
   </joint>
     <!-- Base link is the center of the robot's bottom plate -->
@@ -424,5 +461,5 @@
   <!-- BUFFERS -->
   <joint name="world_to_buffer" type="fixed">
-    <origin xyz="0.2 0.1 0.1" rpy="0 0 0"/>
+    <origin xyz="0.2 0.25 0" rpy="0 0 0"/>
     <parent link="world"/>
     <child link="buffer_base_link"/>
@@ -436,5 +473,5 @@
   <link name="buffer_1"/>
   <joint name="buffer_base_to_2" type="fixed">
-        <origin xyz="0.1 0.0 0" rpy="0 0 0"/>
+        <origin xyz="0.15 0.0 0" rpy="0 0 0"/>
         <parent link="buffer_base_link"/>
         <child link="buffer_2"/>
@@ -443,5 +480,5 @@
   <!-- CANDY MILL -->
   <joint name="world_to_mill" type="fixed">
-    <origin xyz="0.45 0.3 0.1" rpy="0 0 0"/>
+    <origin xyz="0.65 0.6 0" rpy="0 0 0"/>
     <parent link="world"/>
     <child link="mill_base_link"/>
@@ -449,5 +486,5 @@
   <link name="mill_base_link"/>
   <joint name="mill_base_to_stick" type="fixed">
-    <origin xyz="0 0 0.15" rpy="0 0 0"/>
+    <origin xyz="0 0 0.2" rpy="0 0 0"/>
     <parent link="mill_base_link"/>
     <child link="mill_stick"/>
@@ -456,5 +493,5 @@
   <!-- SLIDERS -->
   <joint name="world_to_slider" type="fixed">
-    <origin xyz="0.2 0 0.1" rpy="0 0 0"/>
+    <origin xyz="0 0.15 0" rpy="0 0 0"/>
     <parent link="world"/>
     <child link="slider_base_link"/>
@@ -468,5 +505,5 @@
   <link name="empty_container"/>
   <joint name="sliders_base_to_lid" type="fixed">
-        <origin xyz="0.1 0.0 0" rpy="0 0 0"/>
+        <origin xyz="0.0 0.2 0" rpy="0 0 0"/>
         <parent link="slider_base_link"/>
         <child link="lid"/>
@@ -474,5 +511,5 @@
   <link name="lid"/>
   <joint name="sliders_base_to_full" type="fixed">
-        <origin xyz="0 -0.1 0" rpy="0 0 0"/>
+        <origin xyz="0.6 0 0" rpy="0 0 0"/>
         <parent link="slider_base_link"/>
         <child link="full_container"/>

File: mecademic_description/urdf/meca_500_r3_capsule.urdf.xacro (robot description, xacro)
@@ -1,42 +1,13 @@
 <robot name="meca_500_r3" xmlns:xacro="http://ros.org/wiki/xacro">
   <link name="world"/>
-  <joint name="world_A" type="fixed">
+  <joint name="world_to_base_A" type="fixed">
     <parent link="world"/>
-    <child link="meca_base_link_A"/>
-  </joint>
-  <!-- Base link is the center of the robot's bottom plate -->
-  <link name="meca_base_link_A">
-    <visual>
-      <origin xyz="0 0 0" rpy="0 0 0" />
-      <geometry>
-        <mesh filename="package://mecademic_description/meshes/meca_500_r3_base.dae" />
-      </geometry>
-    </visual>
-    <collision>
-      <origin rpy="-0.00464229562531 1.241639409 -0.00331992768483" xyz="0.002912665 2.5933825e-05 0.03195115"/>
-      <geometry>
-        <cylinder length="0.0247681427348" radius="0.069277"/>
-      </geometry>
-    </collision>
-    <collision>
-      <origin rpy="-0.00464229562531 1.241639409 -0.00331992768483" xyz="-0.008807 0.000007 0.027948"/>
-      <geometry>
-        <sphere radius="0.069277"/>
-      </geometry>
-    </collision>
-    <collision>
-      <origin rpy="-0.00464229562531 1.241639409 -0.00331992768483" xyz="0.014632 0.000045 0.035954"/>
-      <geometry>
-        <sphere radius="0.069277"/>
-      </geometry>
-    </collision>
-    <inertial>
-      <mass value="1"/>
-      <inertia ixx="0.01" ixy="0" ixz="0" iyy="0.01" iyz="0" izz="0.01"/>
-    </inertial>
-  </link>
+    <child link="base_link_A"/>
+    <origin rpy="0 0 0" xyz="0.3 0.0 0.0"/>
+  </joint>
   <gazebo>
       <plugin filename="libxbot2_gz_joint_server.so" name="xbot2_gz_joint_server">
          <pid>
+            <pid name="J1_A" profile="small_mot"/>
             <pid name="meca_axis_1_joint_A" profile="small_mot"/>
             <pid name="meca_axis_2_joint_A" profile="small_mot"/>
@@ -49,4 +20,70 @@
       </plugin>
    </gazebo>
+  <link name="base_link_A">
+    <inertial>
+      <mass value="10.0"/>
+      <inertia ixx="1.0e-03" ixy="0.0" ixz="0.0" iyy="1.0e-03" iyz="0.0" izz="1.0e-03"/>
+    </inertial>
+  </link>
+  <joint name="fixed_L_1_A" type="fixed">
+    <parent link="base_link_A"/>
+    <child link="L_1_A"/>
+    <origin xyz="0.0 0.0 0.05" rpy="0 0 0" />
+  </joint>
+  <link name="L_1_A">
+    <visual>
+      <geometry>
+        <box size="0.6 0.1 0.1"/>
+      </geometry>
+      <material name="blue">
+        <color rgba="0 0 .8 1"/>
+      </material>
+      <origin xyz="0 0 0.0" rpy="0 0 0" />
+    </visual>
+    <collision>
+      <origin xyz="0 0 0" rpy="0 0 0" />
+      <geometry>
+        <box size="0.6 0.1 0.1"/>
+      </geometry>
+    </collision>
+  </link>
+  <joint name="J1_A" type="prismatic">
+    <axis xyz="0 1 0"/>
+    <parent link="L_1_A"/>
+    <child link="meca_base_link_A"/>
+    <limit effort="1000.0" lower="-0.3" upper="0.3" velocity="100"/>
+    <origin rpy="0 1.571 1.571" xyz="0 0.05 0.1"/>
+  </joint>
+  <!-- Base link is the center of the robot's bottom plate -->
+  <link name="meca_base_link_A">
+    <visual>
+      <origin xyz="0 0 0" rpy="0 0 0" />
+      <geometry>
+        <mesh filename="package://mecademic_description/meshes/meca_500_r3_base.dae" />
+      </geometry>
+    </visual>
+    <collision>
+      <origin rpy="-0.00464229562531 1.241639409 -0.00331992768483" xyz="0.002912665 2.5933825e-05 0.03195115"/>
+      <geometry>
+        <cylinder length="0.0247681427348" radius="0.069277"/>
+      </geometry>
+    </collision>
+    <collision>
+      <origin rpy="-0.00464229562531 1.241639409 -0.00331992768483" xyz="-0.008807 0.000007 0.027948"/>
+      <geometry>
+        <sphere radius="0.069277"/>
+      </geometry>
+    </collision>
+    <collision>
+      <origin rpy="-0.00464229562531 1.241639409 -0.00331992768483" xyz="0.014632 0.000045 0.035954"/>
+      <geometry>
+        <sphere radius="0.069277"/>
+      </geometry>
+    </collision>
+    <inertial>
+      <mass value="1"/>
+      <inertia ixx="0.01" ixy="0" ixz="0" iyy="0.01" iyz="0" izz="0.01"/>
+    </inertial>
+  </link>
   <!-- Joint 1 -->
   <link name="meca_axis_1_link_A">
@@ -278,9 +315,9 @@
   </joint>
 <!-- 2nd ROBOT -->
- <joint name="world_to_meca_B" type="fixed">
-      <origin xyz="0.2 0.3 0" rpy="0 0 0"/>
-      <parent link="world"/>
-      <child link="base_link_B"/>
-    </joint>
+ <joint name="world_to_base_B" type="fixed">
+    <origin xyz="0.3 0.6 0" rpy="0 0 0"/>
+    <parent link="world"/>
+    <child link="base_link_B"/>
+  </joint>
   <gazebo>
       <plugin filename="libxbot2_gz_joint_server.so" name="xbot2_gz_joint_server">
@@ -306,5 +343,5 @@
     <axis xyz="0 0 1"/>
     <limit effort="1000.0" lower="-6.28" upper="6.28" velocity="100"/>
-    <origin rpy="0 0 0" xyz="0.0 0.0 0.05"/>
+    <origin rpy="0 0 0" xyz="0.0 0.0 0.075"/>
     <parent link="base_link_B"/>
     <child link="L_1_B"/>
@@ -313,5 +350,5 @@
     <visual>
       <geometry>
-        <cylinder length="0.1" radius="0.1"/>
+        <cylinder length="0.15" radius="0.1"/>
       </geometry>
       <material name="blue">
@@ -322,5 +359,5 @@
       <origin xyz="0 0 0" rpy="0 0 0" />
       <geometry>
-        <cylinder length="0.1" radius="0.1"/>
+        <cylinder length="0.15" radius="0.1"/>
       </geometry>
     </collision>
@@ -329,5 +366,5 @@
     <parent link="L_1_B"/>
     <child link="meca_base_link_B"/>
-    <origin rpy="0 0.7854 0" xyz="0.0 0.0 0.1"/>
+    <origin rpy="0 1.571 0" xyz="0.05 0.0 0.125"/>
   </joint>
     <!-- Base link is the center of the robot's bottom plate -->
@@ -605,5 +642,5 @@
   <!-- BUFFERS -->
   <joint name="world_to_buffer" type="fixed">
-    <origin xyz="0.2 0.1 0.1" rpy="0 0 0"/>
+    <origin xyz="0.2 0.25 0" rpy="0 0 0"/>
     <parent link="world"/>
     <child link="buffer_base_link"/>
@@ -617,5 +654,5 @@
   <link name="buffer_1"/>
   <joint name="buffer_base_to_2" type="fixed">
-        <origin xyz="0.1 0.0 0" rpy="0 0 0"/>
+        <origin xyz="0.15 0.0 0" rpy="0 0 0"/>
         <parent link="buffer_base_link"/>
         <child link="buffer_2"/>
@@ -624,5 +661,5 @@
   <!-- CANDY MILL -->
   <joint name="world_to_mill" type="fixed">
-    <origin xyz="0.45 0.3 0.1" rpy="0 0 0"/>
+    <origin xyz="0.65 0.6 0" rpy="0 0 0"/>
     <parent link="world"/>
     <child link="mill_base_link"/>
@@ -630,5 +667,5 @@
   <link name="mill_base_link"/>
   <joint name="mill_base_to_stick" type="fixed">
-    <origin xyz="0 0 0.15" rpy="0 0 0"/>
+    <origin xyz="0 0 0.2" rpy="0 0 0"/>
     <parent link="mill_base_link"/>
     <child link="mill_stick"/>
@@ -637,5 +674,5 @@
   <!-- SLIDERS -->
   <joint name="world_to_slider" type="fixed">
-    <origin xyz="0.2 0 0.1" rpy="0 0 0"/>
+    <origin xyz="0.0 0.15 0" rpy="0 0 0"/>
     <parent link="world"/>
     <child link="slider_base_link"/>
@@ -649,5 +686,5 @@
   <link name="empty_container"/>
   <joint name="sliders_base_to_lid" type="fixed">
-        <origin xyz="0.1 0.0 0" rpy="0 0 0"/>
+        <origin xyz="0.0 0.2 0" rpy="0 0 0"/>
         <parent link="slider_base_link"/>
         <child link="lid"/>
@@ -655,5 +692,5 @@
   <link name="lid"/>
   <joint name="sliders_base_to_full" type="fixed">
-        <origin xyz="0 -0.1 0" rpy="0 0 0"/>
+        <origin xyz="0.6 0 0" rpy="0 0 0"/>
         <parent link="slider_base_link"/>
         <child link="full_container"/>
