Commit message: use more realistic model of rotary table

File: mecademic_description/urdf/meca_500_r3.urdf.xacro (robot description, xacro)
@@ -4,5 +4,5 @@
     <parent link="world"/>
     <child link="base_link_A"/>
-    <origin rpy="0 0 0" xyz="0.3 0.0 0.0"/>
+    <origin rpy="0 0 0" xyz="0.3 -0.1 0.0"/>
   </joint>
   <gazebo>
@@ -53,5 +53,5 @@
     <child link="meca_base_link_A"/>
     <limit effort="1000.0" lower="-0.3" upper="0.3" velocity="100"/>
-    <origin rpy="0 1.571 1.571" xyz="0 0.05 0.1"/>
+    <origin rpy="0 2.356 1.571" xyz="0 0.05 0.1"/>
   </joint>
   <!-- Base link is the center of the robot's bottom plate -->
@@ -256,31 +256,89 @@
     </inertial>
   </link>
-  <joint name="J1_B" type="revolute">
-    <axis xyz="0 0 1"/>
-    <limit effort="1000.0" lower="-6.28" upper="6.28" velocity="100"/>
-    <origin rpy="0 0 0" xyz="0.0 0.0 0.075"/>
+  <joint name="fixed_BL4104C_1" type="fixed">
+    <axis rpy="0 0 0" xyz="0 0 1"/>
     <parent link="base_link_B"/>
+    <child link="BL4104C_1_stator"/>
+    <origin rpy="0.0 -0.0 0.0" xyz="0.0 0.0 0.0"/>
+  </joint>
+  <link name="BL4104C_1_stator">
+    <visual>
+      <!-- Load mesh. Rotate the origin frame (this is because of how the .stl was saved) -->
+      <origin rpy="0.0 0.0 0.0" xyz="0.0 0.0 0.105"/>
+      <geometry>
+        <cylinder length="0.21" radius="0.13"/>
+      </geometry>
+      <material name="grey"/>
+    </visual>
+    <collision>
+      <origin rpy="0.0 0.0 0.0" xyz="0.0 0.0 0.105"/>
+      <geometry>
+        <cylinder length="0.21" radius="0.13"/>
+      </geometry>
+    </collision>
+    <inertial>
+      <origin rpy="0 0 0" xyz="0.0 0.0 0.10614489"/>
+      <mass value="2.0554934"/>
+      <inertia ixx="0.01068855" ixy="-1.14168e-05" ixz="2.71689e-06" iyy="0.010584907" iyz="8.76312e-05" izz="0.0032026258"/>
+    </inertial>
+  </link>
+  <gazebo reference="BL4104C_1_stator">
+    <mu1>0.2</mu1>
+    <mu2>0.2</mu2>
+    <kp>1000000.0</kp>
+    <kd>1.0</kd>
+    <maxVel>0.0</maxVel>
+    <minDepth>0.0001</minDepth>
+    <material>Gazebo/Blue</material>
+  </gazebo>
+  <joint name="J1_B" type="continuous">
+    <axis rpy="0 0 0" xyz="0 0 1"/>
+    <parent link="BL4104C_1_stator"/>
     <child link="L_1_B"/>
-  </joint>
+    <origin rpy="0.0 -0.0 0.0" xyz="0.0 0.0 0.21"/>
+    <limit effort="147" lower="-2.8" upper="2.8" velocity="100000000"/>
+  </joint>
+  <!-- <xacro:property name="visual" value="package://sps-pkg/database/modular/meshes/yaw_base.stl"/> -->
   <link name="L_1_B">
     <visual>
-      <geometry>
-        <cylinder length="0.15" radius="0.1"/>
-      </geometry>
-      <material name="blue">
-        <color rgba="0 0 .8 1"/>
-      </material>
-    </visual>
-    <collision>
-      <origin xyz="0 0 0" rpy="0 0 0" />
-      <geometry>
-        <cylinder length="0.15" radius="0.1"/>
-      </geometry>
-    </collision>
+      <origin rpy="0.0 0.0 0.0" xyz="0.0 0.0 0.002"/>
+      <geometry>
+        <cylinder length="0.004" radius="0.063"/>
+      </geometry>
+      <material name="grey"/>
+    </visual>
+    <collision>
+      <origin rpy="0.0 0.0 0.0" xyz="0.0 0.0 0.002"/>
+      <geometry>
+        <cylinder length="0.004" radius="0.063"/>
+      </geometry>
+      <material name="grey"/>
+    </collision>
+    <inertial>
+      <origin rpy="0 0 0" xyz="0.0 0.0 -0.024438213"/>
+      <mass value="0.42322395"/>
+      <inertia ixx="0.00063746146" ixy="1.1903424e-05" ixz="6.7230372e-07" iyy="0.00064218987" iyz="2.203073e-05" izz="0.001009674"/>
+    </inertial>
+  </link>
+  <joint name="fixed_L_1_B_rotor_fast" type="fixed">
+    <axis rpy="0 0 0" xyz="0 0 1"/>
+    <parent link="L_1_B"/>
+    <child link="L_1_B_rotor_fast"/>
+    <origin rpy="0.0 -0.0 0.0" xyz="0.0 0.0 0.0"/>
+  </joint>
+  <link name="L_1_B_rotor_fast">
+    <inertial>
+      <origin rpy="0 0 0" xyz="0.0 0.0 -0.0978986"/>
+      <mass value="0.197124"/>
+      <inertia ixx="0.00016128216" ixy="-2.4229e-07" ixz="3.771218e-06" iyy="0.00016138868" iyz="-2.4900687e-06" izz="0.1287638"/>
+      <!-- ixz="0.0003771218" -->
+      <!-- iyz="-0.00024900687" -->
+      <!-- izz="1.287638e-05" -->
+    </inertial>
   </link>
   <joint name="L_1_B_to_meca_base_link_B" type="fixed">
     <parent link="L_1_B"/>
     <child link="meca_base_link_B"/>
-    <origin rpy="0 1.571 0" xyz="0.05 0.0 0.125"/>
+    <origin rpy="0 1.571 0" xyz="0.1 0.0 0.05"/>
   </joint>
     <!-- Base link is the center of the robot's bottom plate -->
@@ -459,5 +517,5 @@
     <limit effort="10.0" velocity="8.72665" lower="-4.712" upper="4.712" />
   </joint>
-  <!-- BUFFERS -->
+    <!-- BUFFERS -->
   <joint name="world_to_buffer" type="fixed">
     <origin xyz="0.2 0.25 0" rpy="0 0 0"/>
@@ -467,5 +525,5 @@
   <link name="buffer_base_link"/>
   <joint name="buffer_base_to_1" type="fixed">
-    <origin xyz="0 0 0" rpy="0 0 0"/>
+    <origin xyz="0 0 0" rpy="0 1.571 0"/>
     <parent link="buffer_base_link"/>
     <child link="buffer_1"/>
@@ -473,5 +531,5 @@
   <link name="buffer_1"/>
   <joint name="buffer_base_to_2" type="fixed">
-        <origin xyz="0.15 0.0 0" rpy="0 0 0"/>
+        <origin xyz="0.15 0.0 0" rpy="0 1.571 0"/>
         <parent link="buffer_base_link"/>
         <child link="buffer_2"/>
@@ -480,5 +538,5 @@
   <!-- CANDY MILL -->
   <joint name="world_to_mill" type="fixed">
-    <origin xyz="0.65 0.6 0" rpy="0 0 0"/>
+    <origin xyz="0.7 0.6 0" rpy="0 1.571 0"/>
     <parent link="world"/>
     <child link="mill_base_link"/>
@@ -486,5 +544,5 @@
   <link name="mill_base_link"/>
   <joint name="mill_base_to_stick" type="fixed">
-    <origin xyz="0 0 0.2" rpy="0 0 0"/>
+    <origin xyz="-0.2 0 0" rpy="0 -1.571 0"/>
     <parent link="mill_base_link"/>
     <child link="mill_stick"/>
@@ -493,5 +551,5 @@
   <!-- SLIDERS -->
   <joint name="world_to_slider" type="fixed">
-    <origin xyz="0 0.15 0" rpy="0 0 0"/>
+    <origin xyz="-0.05 0.05 0" rpy="0 0 0"/>
     <parent link="world"/>
     <child link="slider_base_link"/>
@@ -499,5 +557,5 @@
   <link name="slider_base_link"/>
   <joint name="slider_base_to_empty" type="fixed">
-    <origin xyz="0 0 0" rpy="0 0 0"/>
+    <origin xyz="0 0 0" rpy="0 1.571 0"/>
     <parent link="slider_base_link"/>
     <child link="empty_container"/>
@@ -505,5 +563,5 @@
   <link name="empty_container"/>
   <joint name="sliders_base_to_lid" type="fixed">
-        <origin xyz="0.0 0.2 0" rpy="0 0 0"/>
+        <origin xyz="-0.05 0.1 0" rpy="0 1.571 0"/>
         <parent link="slider_base_link"/>
         <child link="lid"/>
@@ -511,5 +569,5 @@
   <link name="lid"/>
   <joint name="sliders_base_to_full" type="fixed">
-        <origin xyz="0.6 0 0" rpy="0 0 0"/>
+        <origin xyz="0.6 0 0" rpy="0 1.571 0"/>
         <parent link="slider_base_link"/>
         <child link="full_container"/>

File: mecademic_description/urdf/meca_500_r3_capsule.urdf.xacro (robot description, xacro)
@@ -4,5 +4,5 @@
     <parent link="world"/>
     <child link="base_link_A"/>
-    <origin rpy="0 0 0" xyz="0.3 0.0 0.0"/>
+    <origin rpy="0 0 0" xyz="0.3 -0.1 0.0"/>
   </joint>
   <gazebo>
@@ -53,5 +53,5 @@
     <child link="meca_base_link_A"/>
     <limit effort="1000.0" lower="-0.3" upper="0.3" velocity="100"/>
-    <origin rpy="0 1.571 1.571" xyz="0 0.05 0.1"/>
+    <origin rpy="0 2.356 1.571" xyz="0 0.05 0.1"/>
   </joint>
   <!-- Base link is the center of the robot's bottom plate -->
@@ -340,31 +340,89 @@
     </inertial>
   </link>
-  <joint name="J1_B" type="revolute">
-    <axis xyz="0 0 1"/>
-    <limit effort="1000.0" lower="-6.28" upper="6.28" velocity="100"/>
-    <origin rpy="0 0 0" xyz="0.0 0.0 0.075"/>
+  <joint name="fixed_BL4104C_1" type="fixed">
+    <axis rpy="0 0 0" xyz="0 0 1"/>
     <parent link="base_link_B"/>
+    <child link="BL4104C_1_stator"/>
+    <origin rpy="0.0 -0.0 0.0" xyz="0.0 0.0 0.0"/>
+  </joint>
+  <link name="BL4104C_1_stator">
+    <visual>
+      <!-- Load mesh. Rotate the origin frame (this is because of how the .stl was saved) -->
+      <origin rpy="0.0 0.0 0.0" xyz="0.0 0.0 0.105"/>
+      <geometry>
+        <cylinder length="0.21" radius="0.13"/>
+      </geometry>
+      <material name="grey"/>
+    </visual>
+    <collision>
+      <origin rpy="0.0 0.0 0.0" xyz="0.0 0.0 0.105"/>
+      <geometry>
+        <cylinder length="0.21" radius="0.13"/>
+      </geometry>
+    </collision>
+    <inertial>
+      <origin rpy="0 0 0" xyz="0.0 0.0 0.10614489"/>
+      <mass value="2.0554934"/>
+      <inertia ixx="0.01068855" ixy="-1.14168e-05" ixz="2.71689e-06" iyy="0.010584907" iyz="8.76312e-05" izz="0.0032026258"/>
+    </inertial>
+  </link>
+  <gazebo reference="BL4104C_1_stator">
+    <mu1>0.2</mu1>
+    <mu2>0.2</mu2>
+    <kp>1000000.0</kp>
+    <kd>1.0</kd>
+    <maxVel>0.0</maxVel>
+    <minDepth>0.0001</minDepth>
+    <material>Gazebo/Blue</material>
+  </gazebo>
+  <joint name="J1_B" type="continuous">
+    <axis rpy="0 0 0" xyz="0 0 1"/>
+    <parent link="BL4104C_1_stator"/>
     <child link="L_1_B"/>
-  </joint>
+    <origin rpy="0.0 -0.0 0.0" xyz="0.0 0.0 0.21"/>
+    <limit effort="147" lower="-2.8" upper="2.8" velocity="100000000"/>
+  </joint>
+  <!-- <xacro:property name="visual" value="package://sps-pkg/database/modular/meshes/yaw_base.stl"/> -->
   <link name="L_1_B">
     <visual>
-      <geometry>
-        <cylinder length="0.15" radius="0.1"/>
-      </geometry>
-      <material name="blue">
-        <color rgba="0 0 .8 1"/>
-      </material>
-    </visual>
-    <collision>
-      <origin xyz="0 0 0" rpy="0 0 0" />
-      <geometry>
-        <cylinder length="0.15" radius="0.1"/>
-      </geometry>
-    </collision>
+      <origin rpy="0.0 0.0 0.0" xyz="0.0 0.0 0.002"/>
+      <geometry>
+        <cylinder length="0.004" radius="0.063"/>
+      </geometry>
+      <material name="grey"/>
+    </visual>
+    <collision>
+      <origin rpy="0.0 0.0 0.0" xyz="0.0 0.0 0.002"/>
+      <geometry>
+        <cylinder length="0.004" radius="0.063"/>
+      </geometry>
+      <material name="grey"/>
+    </collision>
+    <inertial>
+      <origin rpy="0 0 0" xyz="0.0 0.0 -0.024438213"/>
+      <mass value="0.42322395"/>
+      <inertia ixx="0.00063746146" ixy="1.1903424e-05" ixz="6.7230372e-07" iyy="0.00064218987" iyz="2.203073e-05" izz="0.001009674"/>
+    </inertial>
+  </link>
+  <joint name="fixed_L_1_B_rotor_fast" type="fixed">
+    <axis rpy="0 0 0" xyz="0 0 1"/>
+    <parent link="L_1_B"/>
+    <child link="L_1_B_rotor_fast"/>
+    <origin rpy="0.0 -0.0 0.0" xyz="0.0 0.0 0.0"/>
+  </joint>
+  <link name="L_1_B_rotor_fast">
+    <inertial>
+      <origin rpy="0 0 0" xyz="0.0 0.0 -0.0978986"/>
+      <mass value="0.197124"/>
+      <inertia ixx="0.00016128216" ixy="-2.4229e-07" ixz="3.771218e-06" iyy="0.00016138868" iyz="-2.4900687e-06" izz="0.1287638"/>
+      <!-- ixz="0.0003771218" -->
+      <!-- iyz="-0.00024900687" -->
+      <!-- izz="1.287638e-05" -->
+    </inertial>
   </link>
   <joint name="L_1_B_to_meca_base_link_B" type="fixed">
     <parent link="L_1_B"/>
     <child link="meca_base_link_B"/>
-    <origin rpy="0 1.571 0" xyz="0.05 0.0 0.125"/>
+    <origin rpy="0 1.571 0" xyz="0.1 0.0 0.05"/>
   </joint>
     <!-- Base link is the center of the robot's bottom plate -->
@@ -648,5 +706,5 @@
   <link name="buffer_base_link"/>
   <joint name="buffer_base_to_1" type="fixed">
-    <origin xyz="0 0 0" rpy="0 0 0"/>
+    <origin xyz="0 0 0" rpy="0 1.571 0"/>
     <parent link="buffer_base_link"/>
     <child link="buffer_1"/>
@@ -654,5 +712,5 @@
   <link name="buffer_1"/>
   <joint name="buffer_base_to_2" type="fixed">
-        <origin xyz="0.15 0.0 0" rpy="0 0 0"/>
+        <origin xyz="0.15 0.0 0" rpy="0 1.571 0"/>
         <parent link="buffer_base_link"/>
         <child link="buffer_2"/>
@@ -661,5 +719,5 @@
   <!-- CANDY MILL -->
   <joint name="world_to_mill" type="fixed">
-    <origin xyz="0.65 0.6 0" rpy="0 0 0"/>
+    <origin xyz="0.7 0.6 0" rpy="0 1.571 0"/>
     <parent link="world"/>
     <child link="mill_base_link"/>
@@ -667,5 +725,5 @@
   <link name="mill_base_link"/>
   <joint name="mill_base_to_stick" type="fixed">
-    <origin xyz="0 0 0.2" rpy="0 0 0"/>
+    <origin xyz="-0.2 0 0" rpy="0 -1.571 0"/>
     <parent link="mill_base_link"/>
     <child link="mill_stick"/>
@@ -674,5 +732,5 @@
   <!-- SLIDERS -->
   <joint name="world_to_slider" type="fixed">
-    <origin xyz="0.0 0.15 0" rpy="0 0 0"/>
+    <origin xyz="-0.05 0.05 0" rpy="0 0 0"/>
     <parent link="world"/>
     <child link="slider_base_link"/>
@@ -680,5 +738,5 @@
   <link name="slider_base_link"/>
   <joint name="slider_base_to_empty" type="fixed">
-    <origin xyz="0 0 0" rpy="0 0 0"/>
+    <origin xyz="0 0 0" rpy="0 1.571 0"/>
     <parent link="slider_base_link"/>
     <child link="empty_container"/>
@@ -686,5 +744,5 @@
   <link name="empty_container"/>
   <joint name="sliders_base_to_lid" type="fixed">
-        <origin xyz="0.0 0.2 0" rpy="0 0 0"/>
+        <origin xyz="-0.05 0.1 0" rpy="0 1.571 0"/>
         <parent link="slider_base_link"/>
         <child link="lid"/>
@@ -692,5 +750,5 @@
   <link name="lid"/>
   <joint name="sliders_base_to_full" type="fixed">
-        <origin xyz="0.6 0 0" rpy="0 0 0"/>
+        <origin xyz="0.6 0 0" rpy="0 1.571 0"/>
         <parent link="slider_base_link"/>
         <child link="full_container"/>

Commit message: add more realistic linear joint (not working with collision)

File: mecademic_description/urdf/meca_500_r3.urdf.xacro (robot description, xacro)
@@ -28,30 +28,52 @@
   <joint name="fixed_L_1_A" type="fixed">
     <parent link="base_link_A"/>
-    <child link="L_1_A"/>
-    <origin xyz="0.0 0.0 0.05" rpy="0 0 0" />
-  </joint>
-  <link name="L_1_A">
-    <visual>
-      <geometry>
-        <box size="0.6 0.1 0.1"/>
+    <child link="L_1_A_stator"/>
+    <origin xyz="0.0 0.0 0.06" rpy="0 0 0" />
+  </joint>
+  <link name="L_1_A_stator">
+    <visual>
+      <geometry>
+        <box size="0.72 0.12 0.1"/>
       </geometry>
       <material name="blue">
         <color rgba="0 0 .8 1"/>
       </material>
-      <origin xyz="0 0 0.0" rpy="0 0 0" />
-    </visual>
-    <collision>
-      <origin xyz="0 0 0" rpy="0 0 0" />
-      <geometry>
-        <box size="0.6 0.1 0.1"/>
+      <origin xyz="0 0 0" rpy="0 0 0" />
+    </visual>
+    <collision>
+      <origin xyz="0 0 0" rpy="0 0 0" />
+      <geometry>
+        <box size="0.72 0.12 0.1"/>
       </geometry>
     </collision>
   </link>
   <joint name="J1_A" type="prismatic">
-    <axis xyz="0 1 0"/>
+    <axis xyz="1 0 0"/>
+    <parent link="L_1_A_stator"/>
+    <child link="L_1_A"/>
+    <limit effort="1000.0" lower="-0.3" upper="0.3" velocity="100"/>
+    <origin rpy="0 0 0" xyz="0 0 0.09"/>
+  </joint>
+  <link name="L_1_A">
+    <visual>
+      <geometry>
+        <box size="0.2 0.2 0.04"/>
+      </geometry>
+      <material name="blue">
+        <color rgba="0 0 .8 1"/>
+      </material>
+      <origin xyz="0 0 -0.02" rpy="0 0 0" />
+    </visual>
+    <collision>
+      <origin xyz="0 0 -0.02" rpy="0 0 0" />
+      <geometry>
+        <box size="0.2 0.2 0.04"/>
+      </geometry>
+    </collision>
+  </link>
+  <joint name="L_1_A_to_meca_base_link_A" type="fixed">
     <parent link="L_1_A"/>
     <child link="meca_base_link_A"/>
-    <limit effort="1000.0" lower="-0.3" upper="0.3" velocity="100"/>
-    <origin rpy="0 2.356 1.571" xyz="0 0.05 0.1"/>
+    <origin rpy="0 1.571 1.571" xyz="0.0 0.05 0.05"/>
   </joint>
   <!-- Base link is the center of the robot's bottom plate -->

File: mecademic_description/urdf/meca_500_r3_capsule.urdf.xacro (robot description, xacro)
@@ -28,30 +28,52 @@
   <joint name="fixed_L_1_A" type="fixed">
     <parent link="base_link_A"/>
-    <child link="L_1_A"/>
-    <origin xyz="0.0 0.0 0.05" rpy="0 0 0" />
-  </joint>
-  <link name="L_1_A">
-    <visual>
-      <geometry>
-        <box size="0.6 0.1 0.1"/>
+    <child link="L_1_A_stator"/>
+    <origin xyz="0.0 0.0 0.06" rpy="0 0 0" />
+  </joint>
+  <link name="L_1_A_stator">
+    <visual>
+      <geometry>
+        <box size="0.72 0.12 0.1"/>
       </geometry>
       <material name="blue">
         <color rgba="0 0 .8 1"/>
       </material>
-      <origin xyz="0 0 0.0" rpy="0 0 0" />
-    </visual>
-    <collision>
-      <origin xyz="0 0 0" rpy="0 0 0" />
-      <geometry>
-        <box size="0.6 0.1 0.1"/>
+      <origin xyz="0 0 0" rpy="0 0 0" />
+    </visual>
+    <collision>
+      <origin xyz="0 0 0" rpy="0 0 0" />
+      <geometry>
+        <box size="0.72 0.12 0.1"/>
       </geometry>
     </collision>
   </link>
   <joint name="J1_A" type="prismatic">
-    <axis xyz="0 1 0"/>
+    <axis xyz="1 0 0"/>
+    <parent link="L_1_A_stator"/>
+    <child link="L_1_A"/>
+    <limit effort="1000.0" lower="-0.3" upper="0.3" velocity="100"/>
+    <origin rpy="0 0 0" xyz="0 0 0.09"/>
+  </joint>
+  <link name="L_1_A">
+    <visual>
+      <geometry>
+        <box size="0.2 0.2 0.04"/>
+      </geometry>
+      <material name="blue">
+        <color rgba="0 0 .8 1"/>
+      </material>
+      <origin xyz="0 0 -0.02" rpy="0 0 0" />
+    </visual>
+    <collision>
+      <origin xyz="0 0 -0.02" rpy="0 0 0" />
+      <geometry>
+        <box size="0.2 0.2 0.04"/>
+      </geometry>
+    </collision>
+  </link>
+  <joint name="L_1_A_to_meca_base_link_A" type="fixed">
     <parent link="L_1_A"/>
     <child link="meca_base_link_A"/>
-    <limit effort="1000.0" lower="-0.3" upper="0.3" velocity="100"/>
-    <origin rpy="0 2.356 1.571" xyz="0 0.05 0.1"/>
+    <origin rpy="0 1.571 1.571" xyz="0.0 0.05 0.05"/>
   </joint>
   <!-- Base link is the center of the robot's bottom plate -->
