Commit message: update scene and collision min distance

File: mecademic_description/urdf/meca_500_r3.urdf.xacro (robot description, xacro)
@@ -4,5 +4,5 @@
     <parent link="world"/>
     <child link="base_link_A"/>
-    <origin rpy="0 0 0" xyz="0.3 -0.1 0.0"/>
+    <origin rpy="0 0 0" xyz="0.3 0 0.0"/>
   </joint>
   <gazebo>
@@ -52,5 +52,5 @@
     <parent link="L_1_A_stator"/>
     <child link="L_1_A"/>
-    <limit effort="1000.0" lower="-0.3" upper="0.3" velocity="100"/>
+    <limit effort="1000.0" lower="-0.26" upper="0.26" velocity="100"/>
     <origin rpy="0 0 0" xyz="0 0 0.09"/>
   </joint>
@@ -75,5 +75,5 @@
     <parent link="L_1_A"/>
     <child link="meca_base_link_A"/>
-    <origin rpy="0 1.571 1.571" xyz="0.0 0.05 0.05"/>
+    <origin rpy="0 1.571 1.571" xyz="0.0 0 0.05"/>
   </joint>
   <!-- Base link is the center of the robot's bottom plate -->
@@ -254,5 +254,5 @@
 <!-- 2nd ROBOT -->
   <joint name="world_to_base_B" type="fixed">
-      <origin xyz="0.3 0.6 0" rpy="0 0 0"/>
+      <origin xyz="0.3 0.65 0" rpy="0 0 0"/>
       <parent link="world"/>
       <child link="base_link_B"/>
@@ -362,5 +362,5 @@
     <parent link="L_1_B"/>
     <child link="meca_base_link_B"/>
-    <origin rpy="0 1.571 0" xyz="0.1 0.0 0.05"/>
+    <origin rpy="0 1.571 0" xyz="0.05 0.0 0.05"/>
   </joint>
     <!-- Base link is the center of the robot's bottom plate -->
@@ -539,7 +539,7 @@
     <limit effort="10.0" velocity="8.72665" lower="-4.712" upper="4.712" />
   </joint>
-    <!-- BUFFERS -->
+  <!-- BUFFERS -->
   <joint name="world_to_buffer" type="fixed">
-    <origin xyz="0.2 0.25 0" rpy="0 0 0"/>
+    <origin xyz="0.2 0.35 0.05" rpy="0 0 0"/>
     <parent link="world"/>
     <child link="buffer_base_link"/>
@@ -547,5 +547,5 @@
   <link name="buffer_base_link"/>
   <joint name="buffer_base_to_1" type="fixed">
-    <origin xyz="0 0 0" rpy="0 1.571 0"/>
+    <origin xyz="0 0 0" rpy="0 0 0"/>
     <parent link="buffer_base_link"/>
     <child link="buffer_1"/>
@@ -553,5 +553,5 @@
   <link name="buffer_1"/>
   <joint name="buffer_base_to_2" type="fixed">
-        <origin xyz="0.15 0.0 0" rpy="0 1.571 0"/>
+        <origin xyz="0.3 0.0 0" rpy="0 0 0"/>
         <parent link="buffer_base_link"/>
         <child link="buffer_2"/>
@@ -560,5 +560,5 @@
   <!-- CANDY MILL -->
   <joint name="world_to_mill" type="fixed">
-    <origin xyz="0.7 0.6 0" rpy="0 1.571 0"/>
+    <origin xyz="0.65 0.85 0.05" rpy="0 0 0"/>
     <parent link="world"/>
     <child link="mill_base_link"/>
@@ -566,5 +566,5 @@
   <link name="mill_base_link"/>
   <joint name="mill_base_to_stick" type="fixed">
-    <origin xyz="-0.2 0 0" rpy="0 -1.571 0"/>
+    <origin xyz="0.0 0 0.2" rpy="0 0 0"/>
     <parent link="mill_base_link"/>
     <child link="mill_stick"/>
@@ -573,5 +573,5 @@
   <!-- SLIDERS -->
   <joint name="world_to_slider" type="fixed">
-    <origin xyz="-0.05 0.05 0" rpy="0 0 0"/>
+    <origin xyz="0 0.3 0.05" rpy="0 0 0"/>
     <parent link="world"/>
     <child link="slider_base_link"/>
@@ -579,5 +579,5 @@
   <link name="slider_base_link"/>
   <joint name="slider_base_to_empty" type="fixed">
-    <origin xyz="0 0 0" rpy="0 1.571 0"/>
+    <origin xyz="0 0 0" rpy="0 0 0"/>
     <parent link="slider_base_link"/>
     <child link="empty_container"/>
@@ -585,5 +585,5 @@
   <link name="empty_container"/>
   <joint name="sliders_base_to_lid" type="fixed">
-        <origin xyz="-0.05 0.1 0" rpy="0 1.571 0"/>
+        <origin xyz="0 0.05 0" rpy="0 0 0"/>
         <parent link="slider_base_link"/>
         <child link="lid"/>
@@ -591,5 +591,5 @@
   <link name="lid"/>
   <joint name="sliders_base_to_full" type="fixed">
-        <origin xyz="0.6 0 0" rpy="0 1.571 0"/>
+        <origin xyz="0.6 0 0" rpy="0 0 0"/>
         <parent link="slider_base_link"/>
         <child link="full_container"/>

File: mecademic_description/urdf/meca_500_r3_capsule.urdf.xacro (robot description, xacro)
@@ -4,5 +4,5 @@
     <parent link="world"/>
     <child link="base_link_A"/>
-    <origin rpy="0 0 0" xyz="0.3 -0.1 0.0"/>
+    <origin rpy="0 0 0" xyz="0.3 0 0.0"/>
   </joint>
   <gazebo>
@@ -52,5 +52,5 @@
     <parent link="L_1_A_stator"/>
     <child link="L_1_A"/>
-    <limit effort="1000.0" lower="-0.3" upper="0.3" velocity="100"/>
+    <limit effort="1000.0" lower="-0.26" upper="0.26" velocity="100"/>
     <origin rpy="0 0 0" xyz="0 0 0.09"/>
   </joint>
@@ -75,5 +75,5 @@
     <parent link="L_1_A"/>
     <child link="meca_base_link_A"/>
-    <origin rpy="0 1.571 1.571" xyz="0.0 0.05 0.05"/>
+    <origin rpy="0 1.571 1.571" xyz="0.0 0 0.05"/>
   </joint>
   <!-- Base link is the center of the robot's bottom plate -->
@@ -338,5 +338,5 @@
 <!-- 2nd ROBOT -->
  <joint name="world_to_base_B" type="fixed">
-    <origin xyz="0.3 0.6 0" rpy="0 0 0"/>
+    <origin xyz="0.3 0.65 0" rpy="0 0 0"/>
     <parent link="world"/>
     <child link="base_link_B"/>
@@ -446,5 +446,5 @@
     <parent link="L_1_B"/>
     <child link="meca_base_link_B"/>
-    <origin rpy="0 1.571 0" xyz="0.1 0.0 0.05"/>
+    <origin rpy="0 1.571 0" xyz="0.05 0.0 0.05"/>
   </joint>
     <!-- Base link is the center of the robot's bottom plate -->
@@ -722,5 +722,5 @@
   <!-- BUFFERS -->
   <joint name="world_to_buffer" type="fixed">
-    <origin xyz="0.2 0.25 0" rpy="0 0 0"/>
+    <origin xyz="0.2 0.35 0.05" rpy="0 0 0"/>
     <parent link="world"/>
     <child link="buffer_base_link"/>
@@ -728,5 +728,5 @@
   <link name="buffer_base_link"/>
   <joint name="buffer_base_to_1" type="fixed">
-    <origin xyz="0 0 0" rpy="0 1.571 0"/>
+    <origin xyz="0 0 0" rpy="0 0 0"/>
     <parent link="buffer_base_link"/>
     <child link="buffer_1"/>
@@ -734,5 +734,5 @@
   <link name="buffer_1"/>
   <joint name="buffer_base_to_2" type="fixed">
-        <origin xyz="0.15 0.0 0" rpy="0 1.571 0"/>
+        <origin xyz="0.3 0.0 0" rpy="0 0 0"/>
         <parent link="buffer_base_link"/>
         <child link="buffer_2"/>
@@ -741,5 +741,5 @@
   <!-- CANDY MILL -->
   <joint name="world_to_mill" type="fixed">
-    <origin xyz="0.7 0.6 0" rpy="0 1.571 0"/>
+    <origin xyz="0.65 0.85 0.05" rpy="0 0 0"/>
     <parent link="world"/>
     <child link="mill_base_link"/>
@@ -747,5 +747,5 @@
   <link name="mill_base_link"/>
   <joint name="mill_base_to_stick" type="fixed">
-    <origin xyz="-0.2 0 0" rpy="0 -1.571 0"/>
+    <origin xyz="0.0 0 0.2" rpy="0 0 0"/>
     <parent link="mill_base_link"/>
     <child link="mill_stick"/>
@@ -754,5 +754,5 @@
   <!-- SLIDERS -->
   <joint name="world_to_slider" type="fixed">
-    <origin xyz="-0.05 0.05 0" rpy="0 0 0"/>
+    <origin xyz="0 0.3 0.05" rpy="0 0 0"/>
     <parent link="world"/>
     <child link="slider_base_link"/>
@@ -760,5 +760,5 @@
   <link name="slider_base_link"/>
   <joint name="slider_base_to_empty" type="fixed">
-    <origin xyz="0 0 0" rpy="0 1.571 0"/>
+    <origin xyz="0 0 0" rpy="0 0 0"/>
     <parent link="slider_base_link"/>
     <child link="empty_container"/>
@@ -766,5 +766,5 @@
   <link name="empty_container"/>
   <joint name="sliders_base_to_lid" type="fixed">
-        <origin xyz="-0.05 0.1 0" rpy="0 1.571 0"/>
+        <origin xyz="0 0.05 0" rpy="0 0 0"/>
         <parent link="slider_base_link"/>
         <child link="lid"/>
@@ -772,5 +772,5 @@
   <link name="lid"/>
   <joint name="sliders_base_to_full" type="fixed">
-        <origin xyz="0.6 0 0" rpy="0 1.571 0"/>
+        <origin xyz="0.6 0 0" rpy="0 0 0"/>
         <parent link="slider_base_link"/>
         <child link="full_container"/>

Commit message: wip: on weekly

File: mecademic_description/urdf/meca_500_r3.urdf.xacro (robot description, xacro)
@@ -596,3 +596,26 @@
       </joint>
   <link name="full_container"/>
+  <!-- FLOOR -->
+  <joint name="world_to_floor" type="fixed">
+    <origin xyz="0 0 0" rpy="0 0 0"/>
+    <parent link="world"/>
+    <child link="floor_link"/>
+  </joint>
+  <link name="floor_link">
+    <visual>
+      <geometry>
+        <box size="2 2 0"/>
+      </geometry>
+      <material name="grey">
+        <color rgba="0.232 0.232 0.232 1"/>
+      </material>
+      <origin xyz="0 0 0" rpy="0 0 0" />
+    </visual>
+    <collision>
+      <origin xyz="0 0 0" rpy="0 0 0" />
+      <geometry>
+        <box size="2 2 0"/>
+      </geometry>
+    </collision>
+  </link>
 </robot>

File: mecademic_description/urdf/meca_500_r3_capsule.urdf.xacro (robot description, xacro)
@@ -777,3 +777,26 @@
       </joint>
   <link name="full_container"/>
+  <!-- FLOOR -->
+  <joint name="world_to_floor" type="fixed">
+    <origin xyz="0 0 0" rpy="0 0 0"/>
+    <parent link="world"/>
+    <child link="floor_link"/>
+  </joint>
+  <link name="floor_link">
+    <visual>
+      <geometry>
+        <box size="2 2 0"/>
+      </geometry>
+      <material name="grey">
+        <color rgba="0.232 0.232 0.232 1"/>
+      </material>
+      <origin xyz="0 0 0" rpy="0 0 0" />
+    </visual>
+    <collision>
+      <origin xyz="0 0 0" rpy="0 0 0" />
+      <geometry>
+        <box size="2 2 0"/>
+      </geometry>
+    </collision>
+  </link>
 </robot>

Commit message: modify joint limits to be more conservative
this to avoid floating point representation issues.
the robot will go in error if it receives a value higher than the limit

File: mecademic_description/urdf/meca_500_r3.urdf.xacro (robot description, xacro)
@@ -120,5 +120,5 @@
     <child link="meca_axis_1_link_A" />
     <axis xyz="0 0 1" />
-    <limit effort="10.0" velocity="2.61799" lower="-3.05433" upper="3.05433" />
+   <limit effort="10.0" velocity="2.61799" lower="-3.05" upper="3.05" />
   </joint>
   <!-- Joint 2 -->
@@ -146,5 +146,5 @@
     <child link="meca_axis_2_link_A" />
     <axis xyz="0 1 0" />
-    <limit effort="10.0" velocity="2.61799" lower="-1.22173048" upper="1.5708" />
+    <limit effort="10.0" velocity="2.61799" lower="-1.22" upper="1.57" />
   </joint>
   <!-- Joint 3 -->
@@ -172,5 +172,5 @@
     <child link="meca_axis_3_link_A" />
     <axis xyz="0 1 0" />
-    <limit effort="10.0" velocity="3.14159" lower="-2.35619" upper="1.22173048" />
+    <limit effort="10.0" velocity="3.14159" lower="-2.35" upper="1.22" />
   </joint>
   <!-- Joint 4 -->
@@ -198,5 +198,5 @@
     <child link="meca_axis_4_link_A" />
     <axis xyz="1 0 0" />
-    <limit effort="10.0" velocity="5.23599" lower="-2.96706" upper="2.96706" />
+    <limit effort="10.0" velocity="5.23599" lower="-2.96" upper="2.96" />
   </joint>
   <!-- Joint 5 -->
@@ -224,5 +224,5 @@
     <child link="meca_axis_5_link_A" />
     <axis xyz="0 1 0" />
-    <limit effort="10.0" velocity="5.23599" lower="-2.00713" upper="2.00713" />
+    <limit effort="10.0" velocity="5.23599" lower="-2.00" upper="2.00" />
   </joint>
   <!-- Joint 6 -->
@@ -250,5 +250,5 @@
     <child link="meca_axis_6_link_A" />
     <axis xyz="1 0 0" />
-    <limit effort="10.0" velocity="8.72665" lower="-4.712" upper="4.712" />
+    <limit effort="10.0" velocity="8.72665" lower="-3.142" upper="3.142" />
   </joint>
 <!-- 2nd ROBOT -->
@@ -407,5 +407,5 @@
     <child link="meca_axis_1_link_B" />
     <axis xyz="0 0 1" />
-    <limit effort="10.0" velocity="2.61799" lower="-3.05433" upper="3.05433" />
+    <limit effort="10.0" velocity="2.61799" lower="-3.05" upper="3.05" />
   </joint>
   <!-- Joint 2 -->
@@ -433,5 +433,5 @@
     <child link="meca_axis_2_link_B" />
     <axis xyz="0 1 0" />
-    <limit effort="10.0" velocity="2.61799" lower="-1.22173048" upper="1.5708" />
+    <limit effort="10.0" velocity="2.61799" lower="-1.22" upper="1.57" />
   </joint>
   <!-- Joint 3 -->
@@ -459,5 +459,5 @@
     <child link="meca_axis_3_link_B" />
     <axis xyz="0 1 0" />
-    <limit effort="10.0" velocity="3.14159" lower="-2.35619" upper="1.22173048" />
+    <limit effort="10.0" velocity="3.14159" lower="-2.35" upper="1.22" />
   </joint>
   <!-- Joint 4 -->
@@ -485,5 +485,5 @@
     <child link="meca_axis_4_link_B" />
     <axis xyz="1 0 0" />
-    <limit effort="10.0" velocity="5.23599" lower="-2.96706" upper="2.96706" />
+    <limit effort="10.0" velocity="5.23599" lower="-2.96" upper="2.96" />
   </joint>
   <!-- Joint 5 -->
@@ -511,5 +511,5 @@
     <child link="meca_axis_5_link_B" />
     <axis xyz="0 1 0" />
-    <limit effort="10.0" velocity="5.23599" lower="-2.00713" upper="2.00713" />
+    <limit effort="10.0" velocity="5.23599" lower="-2.00" upper="2.00" />
   </joint>
   <!-- Joint 6 -->
@@ -537,5 +537,5 @@
     <child link="meca_axis_6_link_B" />
     <axis xyz="1 0 0" />
-    <limit effort="10.0" velocity="8.72665" lower="-4.712" upper="4.712" />
+    <limit effort="10.0" velocity="8.72665" lower="-3.142" upper="3.142" />
   </joint>
   <!-- BUFFERS -->

File: mecademic_description/urdf/meca_500_r3_capsule.urdf.xacro (robot description, xacro)
@@ -140,9 +140,9 @@
   </link>
   <joint name="meca_axis_1_joint_A" type="revolute">
-    <origin xyz="0.012498 0 0.091" rpy="0 0 0" />
-    <parent link="meca_base_link_A" />
-    <child link="meca_axis_1_link_A" />
-    <axis xyz="0 0 1" />
-    <limit effort="10.0" velocity="2.61799" lower="-3.05433" upper="3.05433" />
+    <origin rpy="0.0 0.0 0.0" xyz="0.012498 0.0 0.091"/>
+    <axis xyz="0.0 0.0 1.0"/>
+    <parent link="meca_base_link_A"/>
+    <child link="meca_axis_1_link_A"/>
+    <limit effort="10.0" lower="-3.05" upper="3.05" velocity="2.61799"/>
   </joint>
   <!-- Joint 2 -->
@@ -178,9 +178,9 @@
   </link>
   <joint name="meca_axis_2_joint_A" type="revolute">
-    <origin xyz="0 0 0.044" rpy="0 0 0" />
-    <parent link="meca_axis_1_link_A" />
-    <child link="meca_axis_2_link_A" />
-    <axis xyz="0 1 0" />
-    <limit effort="10.0" velocity="2.61799" lower="-1.22173048" upper="1.5708" />
+    <origin rpy="0.0 0.0 0.0" xyz="0.0 0.0 0.044"/>
+    <axis xyz="0.0 1.0 0.0"/>
+    <parent link="meca_axis_1_link_A"/>
+    <child link="meca_axis_2_link_A"/>
+    <limit effort="10.0" lower="-1.22" upper="1.57" velocity="2.61799"/>
   </joint>
   <!-- Joint 3 -->
@@ -216,9 +216,9 @@
   </link>
   <joint name="meca_axis_3_joint_A" type="revolute">
-    <origin xyz="0 0 0.135" rpy="0 0 0" />
-    <parent link="meca_axis_2_link_A" />
-    <child link="meca_axis_3_link_A" />
-    <axis xyz="0 1 0" />
-    <limit effort="10.0" velocity="3.14159" lower="-2.35619" upper="1.22173048" />
+    <origin rpy="0.0 0.0 0.0" xyz="0.0 0.0 0.135"/>
+    <axis xyz="0.0 1.0 0.0"/>
+    <parent link="meca_axis_2_link_A"/>
+    <child link="meca_axis_3_link_A"/>
+    <limit effort="10.0" lower="-2.35" upper="1.22" velocity="3.14159"/>
   </joint>
   <!-- Joint 4 -->
@@ -254,9 +254,9 @@
   </link>
   <joint name="meca_axis_4_joint_A" type="revolute">
-    <origin xyz="0 0 0.038" rpy="0 0 0" />
-    <parent link="meca_axis_3_link_A" />
-    <child link="meca_axis_4_link_A" />
-    <axis xyz="1 0 0" />
-    <limit effort="10.0" velocity="5.23599" lower="-2.96706" upper="2.96706" />
+    <origin rpy="0.0 0.0 0.0" xyz="0.0 0.0 0.038"/>
+    <axis xyz="1.0 0.0 0.0"/>
+    <parent link="meca_axis_3_link_A"/>
+    <child link="meca_axis_4_link_A"/>
+    <limit effort="10.0" lower="-2.96" upper="2.96" velocity="5.23599"/>
   </joint>
   <!-- Joint 5 -->
@@ -292,9 +292,9 @@
   </link>
   <joint name="meca_axis_5_joint_A" type="revolute">
-    <origin xyz="0.12 0 0" rpy="0 0 0" />
-    <parent link="meca_axis_4_link_A" />
-    <child link="meca_axis_5_link_A" />
-    <axis xyz="0 1 0" />
-    <limit effort="10.0" velocity="5.23599" lower="-2.00713" upper="2.00713" />
+    <origin rpy="0.0 0.0 0.0" xyz="0.12 0.0 0.0"/>
+    <axis xyz="0.0 1.0 0.0"/>
+    <parent link="meca_axis_4_link_A"/>
+    <child link="meca_axis_5_link_A"/>
+    <limit effort="10.0" lower="-2.00" upper="2.00" velocity="5.23599"/>
   </joint>
   <!-- Joint 6 -->
@@ -330,11 +330,11 @@
   </link>
   <joint name="meca_axis_6_joint_A" type="revolute">
-    <origin xyz="0.07 0 0" rpy="0 0 0" />
-    <parent link="meca_axis_5_link_A" />
-    <child link="meca_axis_6_link_A" />
-    <axis xyz="1 0 0" />
-    <limit effort="10.0" velocity="8.72665" lower="-4.712" upper="4.712" />
-  </joint>
-<!-- 2nd ROBOT -->
+    <origin rpy="0.0 0.0 0.0" xyz="0.07 0.0 0.0"/>
+    <axis xyz="1.0 0.0 0.0"/>
+    <parent link="meca_axis_5_link_A"/>
+    <child link="meca_axis_6_link_A"/>
+    <limit effort="10.0" lower="-3.142" upper="3.142" velocity="8.72665"/>
+  </joint>
+  <!-- 2nd ROBOT -->
  <joint name="world_to_base_B" type="fixed">
     <origin xyz="0.3 0.65 0" rpy="0 0 0"/>
@@ -528,5 +528,5 @@
     <child link="meca_axis_1_link_B" />
     <axis xyz="0 0 1" />
-    <limit effort="10.0" velocity="2.61799" lower="-3.05433" upper="3.05433" />
+    <limit effort="10.0" lower="-3.05" upper="3.05" velocity="2.61799"/>
   </joint>
   <!-- Joint 2 -->
@@ -566,5 +566,5 @@
     <child link="meca_axis_2_link_B" />
     <axis xyz="0 1 0" />
-    <limit effort="10.0" velocity="2.61799" lower="-1.22173048" upper="1.5708" />
+    <limit effort="10.0" lower="-1.22" upper="1.57" velocity="2.61799"/>
   </joint>
   <!-- Joint 3 -->
@@ -604,5 +604,5 @@
     <child link="meca_axis_3_link_B" />
     <axis xyz="0 1 0" />
-    <limit effort="10.0" velocity="3.14159" lower="-2.35619" upper="1.22173048" />
+    <limit effort="10.0" lower="-2.35" upper="1.22" velocity="3.14159"/>
   </joint>
   <!-- Joint 4 -->
@@ -642,5 +642,5 @@
     <child link="meca_axis_4_link_B" />
     <axis xyz="1 0 0" />
-    <limit effort="10.0" velocity="5.23599" lower="-2.96706" upper="2.96706" />
+   <limit effort="10.0" lower="-2.96" upper="2.96" velocity="5.23599"/>
   </joint>
   <!-- Joint 5 -->
@@ -680,5 +680,5 @@
     <child link="meca_axis_5_link_B" />
     <axis xyz="0 1 0" />
-    <limit effort="10.0" velocity="5.23599" lower="-2.00713" upper="2.00713" />
+    <limit effort="10.0" lower="-2.00" upper="2.00" velocity="5.23599"/>
   </joint>
   <!-- Joint 6 -->
@@ -718,5 +718,5 @@
     <child link="meca_axis_6_link_B" />
     <axis xyz="1 0 0" />
-    <limit effort="10.0" velocity="8.72665" lower="-4.712" upper="4.712" />
+    <limit effort="10.0" lower="-3.142" upper="3.142" velocity="8.72665"/>
   </joint>
   <!-- BUFFERS -->
