Commit message: remove meca_A

File: mecademic_description/urdf/meca_500_r3.urdf.xacro (robot description, xacro)
@@ -1,255 +1,4 @@
 <robot name="meca_500_r3" xmlns:xacro="http://ros.org/wiki/xacro">
   <link name="world"/>
-  <joint name="world_to_base_A" type="fixed">
-    <parent link="world"/>
-    <child link="base_link_A"/>
-    <origin rpy="0 0 0" xyz="0.3 0 0.0"/>
-  </joint>
-  <gazebo>
-      <plugin filename="libxbot2_gz_joint_server.so" name="xbot2_gz_joint_server">
-         <pid>
-            <pid name="J1_A" profile="small_mot"/>
-            <pid name="meca_axis_1_joint_A" profile="small_mot"/>
-            <pid name="meca_axis_2_joint_A" profile="small_mot"/>
-            <pid name="meca_axis_3_joint_A" profile="small_mot"/>
-            <pid name="meca_axis_4_joint_A" profile="small_mot"/>
-            <pid name="meca_axis_5_joint_A" profile="small_mot"/>
-            <pid name="meca_axis_6_joint_A" profile="small_mot"/>
-         </pid>
-         <gain d="5" name="small_mot" p="100"/>
-      </plugin>
-   </gazebo>
-  <link name="base_link_A">
-    <inertial>
-      <mass value="10.0"/>
-      <inertia ixx="1.0e-03" ixy="0.0" ixz="0.0" iyy="1.0e-03" iyz="0.0" izz="1.0e-03"/>
-    </inertial>
-  </link>
-  <joint name="fixed_L_1_A" type="fixed">
-    <parent link="base_link_A"/>
-    <child link="L_1_A_stator"/>
-    <origin xyz="0.0 0.0 0.06" rpy="0 0 0" />
-  </joint>
-  <link name="L_1_A_stator">
-    <visual>
-      <geometry>
-        <box size="0.72 0.12 0.1"/>
-      </geometry>
-      <material name="blue">
-        <color rgba="0 0 .8 1"/>
-      </material>
-      <origin xyz="0 0 0" rpy="0 0 0" />
-    </visual>
-    <collision>
-      <origin xyz="0 0 0" rpy="0 0 0" />
-      <geometry>
-        <box size="0.72 0.12 0.1"/>
-      </geometry>
-    </collision>
-  </link>
-  <joint name="J1_A" type="prismatic">
-    <axis xyz="1 0 0"/>
-    <parent link="L_1_A_stator"/>
-    <child link="L_1_A"/>
-    <limit effort="1000.0" lower="-0.26" upper="0.26" velocity="100"/>
-    <origin rpy="0 0 0" xyz="0 0 0.09"/>
-  </joint>
-  <link name="L_1_A">
-    <visual>
-      <geometry>
-        <box size="0.2 0.2 0.04"/>
-      </geometry>
-      <material name="blue">
-        <color rgba="0 0 .8 1"/>
-      </material>
-      <origin xyz="0 0 -0.02" rpy="0 0 0" />
-    </visual>
-    <collision>
-      <origin xyz="0 0 -0.02" rpy="0 0 0" />
-      <geometry>
-        <box size="0.2 0.2 0.04"/>
-      </geometry>
-    </collision>
-  </link>
-  <joint name="L_1_A_to_meca_base_link_A" type="fixed">
-    <parent link="L_1_A"/>
-    <child link="meca_base_link_A"/>
-    <origin rpy="0 1.571 1.571" xyz="0.0 0 0.05"/>
-  </joint>
-  <!-- Base link is the center of the robot's bottom plate -->
-  <link name="meca_base_link_A">
-    <visual>
-      <origin xyz="0 0 0" rpy="0 0 0" />
-      <geometry>
-        <mesh filename="package://mecademic_description/meshes/meca_500_r3_base.dae" />
-      </geometry>
-    </visual>
-    <collision>
-      <origin xyz="0 0 0" rpy="0 0 0" />
-      <geometry>
-        <mesh filename="package://mecademic_description/meshes/meca_500_r3_base_collision.stl" />
-      </geometry>
-    </collision>
-    <inertial>
-      <mass value="1"/>
-      <inertia ixx="0.01" ixy="0" ixz="0" iyy="0.01" iyz="0" izz="0.01"/>
-    </inertial>
-  </link>
-  <!-- Joint 1 -->
-  <link name="meca_axis_1_link_A">
-    <visual>
-      <origin xyz="0 0 0" rpy="0 0 0" />
-      <geometry>
-        <mesh filename="package://mecademic_description/meshes/meca_500_r3_j1.dae" />
-      </geometry>
-    </visual>
-    <collision>
-      <origin xyz="0 0 0" rpy="0 0 0" />
-      <geometry>
-        <mesh filename="package://mecademic_description/meshes/meca_500_r3_j1_collision.stl" />
-      </geometry>
-    </collision>
-    <inertial>
-      <mass value="1"/>
-      <inertia ixx="0.01" ixy="0" ixz="0" iyy="0.01" iyz="0" izz="0.01"/>
-    </inertial>
-  </link>
-  <joint name="meca_axis_1_joint_A" type="revolute">
-    <origin xyz="0.012498 0 0.091" rpy="0 0 0" />
-    <parent link="meca_base_link_A" />
-    <child link="meca_axis_1_link_A" />
-    <axis xyz="0 0 1" />
-   <limit effort="10.0" velocity="2.61799" lower="-3.05" upper="3.05" />
-  </joint>
-  <!-- Joint 2 -->
-  <link name="meca_axis_2_link_A">
-    <visual>
-      <origin xyz="0 0 0" rpy="0 0 0" />
-      <geometry>
-        <mesh filename="package://mecademic_description/meshes/meca_500_r3_j2.dae" />
-      </geometry>
-    </visual>
-    <collision>
-      <origin xyz="0 0 0" rpy="0 0 0" />
-      <geometry>
-        <mesh filename="package://mecademic_description/meshes/meca_500_r3_j2_collision.stl" />
-      </geometry>
-    </collision>
-    <inertial>
-      <mass value="1"/>
-      <inertia ixx="0.01" ixy="0" ixz="0" iyy="0.01" iyz="0" izz="0.01"/>
-    </inertial>
-  </link>
-  <joint name="meca_axis_2_joint_A" type="revolute">
-    <origin xyz="0 0 0.044" rpy="0 0 0" />
-    <parent link="meca_axis_1_link_A" />
-    <child link="meca_axis_2_link_A" />
-    <axis xyz="0 1 0" />
-    <limit effort="10.0" velocity="2.61799" lower="-1.22" upper="1.57" />
-  </joint>
-  <!-- Joint 3 -->
-  <link name="meca_axis_3_link_A">
-    <visual>
-      <origin xyz="0 0 0" rpy="0 0 0" />
-      <geometry>
-        <mesh filename="package://mecademic_description/meshes/meca_500_r3_j3.dae" />
-      </geometry>
-    </visual>
-    <collision>
-      <origin xyz="0 0 0" rpy="0 0 0" />
-      <geometry>
-        <mesh filename="package://mecademic_description/meshes/meca_500_r3_j3_collision.stl" />
-      </geometry>
-    </collision>
-    <inertial>
-      <mass value="1"/>
-      <inertia ixx="0.01" ixy="0" ixz="0" iyy="0.01" iyz="0" izz="0.01"/>
-    </inertial>
-  </link>
-  <joint name="meca_axis_3_joint_A" type="revolute">
-    <origin xyz="0 0 0.135" rpy="0 0 0" />
-    <parent link="meca_axis_2_link_A" />
-    <child link="meca_axis_3_link_A" />
-    <axis xyz="0 1 0" />
-    <limit effort="10.0" velocity="3.14159" lower="-2.35" upper="1.22" />
-  </joint>
-  <!-- Joint 4 -->
-  <link name="meca_axis_4_link_A">
-    <visual>
-      <origin xyz="0 0 0" rpy="0 0 0" />
-      <geometry>
-        <mesh filename="package://mecademic_description/meshes/meca_500_r3_j4.dae" />
-      </geometry>
-    </visual>
-    <collision>
-      <origin xyz="0 0 0" rpy="0 0 0" />
-      <geometry>
-        <mesh filename="package://mecademic_description/meshes/meca_500_r3_j4_collision.stl" />
-      </geometry>
-    </collision>
-    <inertial>
-      <mass value="1"/>
-      <inertia ixx="0.01" ixy="0" ixz="0" iyy="0.01" iyz="0" izz="0.01"/>
-    </inertial>
-  </link>
-  <joint name="meca_axis_4_joint_A" type="revolute">
-    <origin xyz="0 0 0.038" rpy="0 0 0" />
-    <parent link="meca_axis_3_link_A" />
-    <child link="meca_axis_4_link_A" />
-    <axis xyz="1 0 0" />
-    <limit effort="10.0" velocity="5.23599" lower="-2.96" upper="2.96" />
-  </joint>
-  <!-- Joint 5 -->
-  <link name="meca_axis_5_link_A">
-    <visual>
-      <origin xyz="0 0 0" rpy="0 0 0" />
-      <geometry>
-        <mesh filename="package://mecademic_description/meshes/meca_500_r3_j5.dae" />
-      </geometry>
-    </visual>
-    <collision>
-      <origin xyz="0 0 0" rpy="0 0 0" />
-      <geometry>
-        <mesh filename="package://mecademic_description/meshes/meca_500_r3_j5_collision.stl" />
-      </geometry>
-    </collision>
-    <inertial>
-      <mass value="1"/>
-      <inertia ixx="0.01" ixy="0" ixz="0" iyy="0.01" iyz="0" izz="0.01"/>
-    </inertial>
-  </link>
-  <joint name="meca_axis_5_joint_A" type="revolute">
-    <origin xyz="0.12 0 0" rpy="0 0 0" />
-    <parent link="meca_axis_4_link_A" />
-    <child link="meca_axis_5_link_A" />
-    <axis xyz="0 1 0" />
-    <limit effort="10.0" velocity="5.23599" lower="-2.00" upper="2.00" />
-  </joint>
-  <!-- Joint 6 -->
-  <link name="meca_axis_6_link_A">
-    <visual>
-      <origin xyz="0 0 0" rpy="0 0 0" />
-      <geometry>
-        <mesh filename="package://mecademic_description/meshes/meca_500_r3_j6.dae" />
-      </geometry>
-    </visual>
-    <collision>
-      <origin xyz="0 0 0" rpy="0 0 0" />
-      <geometry>
-        <mesh filename="package://mecademic_description/meshes/meca_500_r3_j6_collision.stl" />
-      </geometry>
-    </collision>
-    <inertial>
-      <mass value="1"/>
-      <inertia ixx="0.01" ixy="0" ixz="0" iyy="0.01" iyz="0" izz="0.01"/>
-    </inertial>
-  </link>
-  <joint name="meca_axis_6_joint_A" type="revolute">
-    <origin xyz="0.07 0 0" rpy="0 0 0" />
-    <parent link="meca_axis_5_link_A" />
-    <child link="meca_axis_6_link_A" />
-    <axis xyz="1 0 0" />
-    <limit effort="10.0" velocity="8.72665" lower="-3.142" upper="3.142" />
-  </joint>
 <!-- 2nd ROBOT -->
   <joint name="world_to_base_B" type="fixed">

File: mecademic_description/urdf/meca_500_r3_capsule.urdf.xacro (robot description, xacro)
@@ -1,340 +1,5 @@
 <robot name="meca_500_r3" xmlns:xacro="http://ros.org/wiki/xacro">
   <link name="world"/>
-  <joint name="world_to_base_A" type="fixed">
-    <parent link="world"/>
-    <child link="base_link_A"/>
-    <origin rpy="0 0 0" xyz="0.3 0 0.0"/>
-  </joint>
-  <gazebo>
-      <plugin filename="libxbot2_gz_joint_server.so" name="xbot2_gz_joint_server">
-         <pid>
-            <pid name="J1_A" profile="small_mot"/>
-            <pid name="meca_axis_1_joint_A" profile="small_mot"/>
-            <pid name="meca_axis_2_joint_A" profile="small_mot"/>
-            <pid name="meca_axis_3_joint_A" profile="small_mot"/>
-            <pid name="meca_axis_4_joint_A" profile="small_mot"/>
-            <pid name="meca_axis_5_joint_A" profile="small_mot"/>
-            <pid name="meca_axis_6_joint_A" profile="small_mot"/>
-         </pid>
-         <gain d="5" name="small_mot" p="100"/>
-      </plugin>
-   </gazebo>
-  <link name="base_link_A">
-    <inertial>
-      <mass value="10.0"/>
-      <inertia ixx="1.0e-03" ixy="0.0" ixz="0.0" iyy="1.0e-03" iyz="0.0" izz="1.0e-03"/>
-    </inertial>
-  </link>
-  <joint name="fixed_L_1_A" type="fixed">
-    <parent link="base_link_A"/>
-    <child link="L_1_A_stator"/>
-    <origin xyz="0.0 0.0 0.06" rpy="0 0 0" />
-  </joint>
-  <link name="L_1_A_stator">
-    <visual>
-      <geometry>
-        <box size="0.72 0.12 0.1"/>
-      </geometry>
-      <material name="blue">
-        <color rgba="0 0 .8 1"/>
-      </material>
-      <origin xyz="0 0 0" rpy="0 0 0" />
-    </visual>
-    <collision>
-      <origin xyz="0 0 0" rpy="0 0 0" />
-      <geometry>
-        <box size="0.72 0.12 0.1"/>
-      </geometry>
-    </collision>
-  </link>
-  <joint name="J1_A" type="prismatic">
-    <axis xyz="1 0 0"/>
-    <parent link="L_1_A_stator"/>
-    <child link="L_1_A"/>
-    <limit effort="1000.0" lower="-0.26" upper="0.26" velocity="100"/>
-    <origin rpy="0 0 0" xyz="0 0 0.09"/>
-  </joint>
-  <link name="L_1_A">
-    <visual>
-      <geometry>
-        <box size="0.2 0.2 0.04"/>
-      </geometry>
-      <material name="blue">
-        <color rgba="0 0 .8 1"/>
-      </material>
-      <origin xyz="0 0 -0.02" rpy="0 0 0" />
-    </visual>
-    <collision>
-      <origin xyz="0 0 -0.02" rpy="0 0 0" />
-      <geometry>
-        <box size="0.2 0.2 0.04"/>
-      </geometry>
-    </collision>
-  </link>
-  <joint name="L_1_A_to_meca_base_link_A" type="fixed">
-    <parent link="L_1_A"/>
-    <child link="meca_base_link_A"/>
-    <origin rpy="0 1.571 1.571" xyz="0.0 0 0.05"/>
-  </joint>
-  <!-- Base link is the center of the robot's bottom plate -->
-  <link name="meca_base_link_A">
-    <visual>
-      <origin xyz="0 0 0" rpy="0 0 0" />
-      <geometry>
-        <mesh filename="package://mecademic_description/meshes/meca_500_r3_base.dae" />
-      </geometry>
-    </visual>
-    <collision>
-      <origin rpy="-0.00464229562531 1.241639409 -0.00331992768483" xyz="0.002912665 2.5933825e-05 0.03195115"/>
-      <geometry>
-        <cylinder length="0.0247681427348" radius="0.069277"/>
-      </geometry>
-    </collision>
-    <collision>
-      <origin rpy="-0.00464229562531 1.241639409 -0.00331992768483" xyz="-0.008807 0.000007 0.027948"/>
-      <geometry>
-        <sphere radius="0.069277"/>
-      </geometry>
-    </collision>
-    <collision>
-      <origin rpy="-0.00464229562531 1.241639409 -0.00331992768483" xyz="0.014632 0.000045 0.035954"/>
-      <geometry>
-        <sphere radius="0.069277"/>
-      </geometry>
-    </collision>
-    <inertial>
-      <mass value="1"/>
-      <inertia ixx="0.01" ixy="0" ixz="0" iyy="0.01" iyz="0" izz="0.01"/>
-    </inertial>
-  </link>
-  <!-- Joint 1 -->
-  <link name="meca_axis_1_link_A">
-    <visual>
-      <origin xyz="0 0 0" rpy="0 0 0" />
-      <geometry>
-        <mesh filename="package://mecademic_description/meshes/meca_500_r3_j1.dae" />
-      </geometry>
-    </visual>
-    <collision>
-      <origin rpy="-1.5643390872 0.00108905813092 -0.00108204843032" xyz="1.404e-07 -0.00017605 0.03168225"/>
-      <geometry>
-        <cylinder length="0.0388249324419" radius="0.0530516"/>
-      </geometry>
-    </collision>
-    <collision>
-      <origin rpy="-1.5643390872 0.00108905813092 -0.00108204843032" xyz="-0.000021 -0.019588 0.031557"/>
-      <geometry>
-        <sphere radius="0.0530516"/>
-      </geometry>
-    </collision>
-    <collision>
-      <origin rpy="-1.5643390872 0.00108905813092 -0.00108204843032" xyz="0.000021 0.019236 0.031808"/>
-      <geometry>
-        <sphere radius="0.0530516"/>
-      </geometry>
-    </collision>
-    <inertial>
-      <mass value="1"/>
-      <inertia ixx="0.01" ixy="0" ixz="0" iyy="0.01" iyz="0" izz="0.01"/>
-    </inertial>
-  </link>
-  <joint name="meca_axis_1_joint_A" type="revolute">
-    <origin rpy="0.0 0.0 0.0" xyz="0.012498 0.0 0.091"/>
-    <axis xyz="0.0 0.0 1.0"/>
-    <parent link="meca_base_link_A"/>
-    <child link="meca_axis_1_link_A"/>
-    <limit effort="10.0" lower="-3.05" upper="3.05" velocity="2.61799"/>
-  </joint>
-  <!-- Joint 2 -->
-  <link name="meca_axis_2_link_A">
-    <visual>
-      <origin xyz="0 0 0" rpy="0 0 0" />
-      <geometry>
-        <mesh filename="package://mecademic_description/meshes/meca_500_r3_j2.dae" />
-      </geometry>
-    </visual>
-    <collision>
-      <origin rpy="3.14150631803 -0.0666872950524 -3.13900434911" xyz="-0.007204205 2.561655e-06 0.07263715"/>
-      <geometry>
-        <cylinder length="0.121249210008" radius="0.0578403"/>
-      </geometry>
-    </collision>
-    <collision>
-      <origin rpy="3.14150631803 -0.0666872950524 -3.13900434911" xyz="-0.003164 0.000008 0.133127"/>
-      <geometry>
-        <sphere radius="0.0578403"/>
-      </geometry>
-    </collision>
-    <collision>
-      <origin rpy="3.14150631803 -0.0666872950524 -3.13900434911" xyz="-0.011244 -0.000003 0.012147"/>
-      <geometry>
-        <sphere radius="0.0578403"/>
-      </geometry>
-    </collision>
-    <inertial>
-      <mass value="1"/>
-      <inertia ixx="0.01" ixy="0" ixz="0" iyy="0.01" iyz="0" izz="0.01"/>
-    </inertial>
-  </link>
-  <joint name="meca_axis_2_joint_A" type="revolute">
-    <origin rpy="0.0 0.0 0.0" xyz="0.0 0.0 0.044"/>
-    <axis xyz="0.0 1.0 0.0"/>
-    <parent link="meca_axis_1_link_A"/>
-    <child link="meca_axis_2_link_A"/>
-    <limit effort="10.0" lower="-1.22" upper="1.57" velocity="2.61799"/>
-  </joint>
-  <!-- Joint 3 -->
-  <link name="meca_axis_3_link_A">
-    <visual>
-      <origin xyz="0 0 0" rpy="0 0 0" />
-      <geometry>
-        <mesh filename="package://mecademic_description/meshes/meca_500_r3_j3.dae" />
-      </geometry>
-    </visual>
-    <collision>
-      <origin rpy="-0.0775632999618 0.486298597709 -0.0192491912301" xyz="0.009983498 -0.000990284 0.020095595"/>
-      <geometry>
-        <cylinder length="0.0408120816515" radius="0.0503272"/>
-      </geometry>
-    </collision>
-    <collision>
-      <origin rpy="-0.0775632999618 0.486298597709 -0.0192491912301" xyz="0.000447 -0.002388 0.002109"/>
-      <geometry>
-        <sphere radius="0.0503272"/>
-      </geometry>
-    </collision>
-    <collision>
-      <origin rpy="-0.0775632999618 0.486298597709 -0.0192491912301" xyz="0.019520 0.000408 0.038082"/>
-      <geometry>
-        <sphere radius="0.0503272"/>
-      </geometry>
-    </collision>
-    <inertial>
-      <mass value="1"/>
-      <inertia ixx="0.01" ixy="0" ixz="0" iyy="0.01" iyz="0" izz="0.01"/>
-    </inertial>
-  </link>
-  <joint name="meca_axis_3_joint_A" type="revolute">
-    <origin rpy="0.0 0.0 0.0" xyz="0.0 0.0 0.135"/>
-    <axis xyz="0.0 1.0 0.0"/>
-    <parent link="meca_axis_2_link_A"/>
-    <child link="meca_axis_3_link_A"/>
-    <limit effort="10.0" lower="-2.35" upper="1.22" velocity="3.14159"/>
-  </joint>
-  <!-- Joint 4 -->
-  <link name="meca_axis_4_link_A">
-    <visual>
-      <origin xyz="0 0 0" rpy="0 0 0" />
-      <geometry>
-        <mesh filename="package://mecademic_description/meshes/meca_500_r3_j4.dae" />
-      </geometry>
-    </visual>
-    <collision>
-      <origin rpy="-1.61527511752 1.5509782436 -1.59546790677" xyz="0.1018437 -0.00037629375 0.0004856635"/>
-      <geometry>
-        <cylinder length="0.0362997282424" radius="0.0387182"/>
-      </geometry>
-    </collision>
-    <collision>
-      <origin rpy="-1.61527511752 1.5509782436 -1.59546790677" xyz="0.083697 -0.000736 0.000502"/>
-      <geometry>
-        <sphere radius="0.0387182"/>
-      </geometry>
-    </collision>
-    <collision>
-      <origin rpy="-1.61527511752 1.5509782436 -1.59546790677" xyz="0.119990 -0.000017 0.000470"/>
-      <geometry>
-        <sphere radius="0.0387182"/>
-      </geometry>
-    </collision>
-    <inertial>
-      <mass value="1"/>
-      <inertia ixx="0.01" ixy="0" ixz="0" iyy="0.01" iyz="0" izz="0.01"/>
-    </inertial>
-  </link>
-  <joint name="meca_axis_4_joint_A" type="revolute">
-    <origin rpy="0.0 0.0 0.0" xyz="0.0 0.0 0.038"/>
-    <axis xyz="1.0 0.0 0.0"/>
-    <parent link="meca_axis_3_link_A"/>
-    <child link="meca_axis_4_link_A"/>
-    <limit effort="10.0" lower="-2.96" upper="2.96" velocity="5.23599"/>
-  </joint>
-  <!-- Joint 5 -->
-  <link name="meca_axis_5_link_A">
-    <visual>
-      <origin xyz="0 0 0" rpy="0 0 0" />
-      <geometry>
-        <mesh filename="package://mecademic_description/meshes/meca_500_r3_j5.dae" />
-      </geometry>
-    </visual>
-    <collision>
-      <origin rpy="-1.56738494938 1.42197043963 -1.41859762505" xyz="0.022533785 0.002385127 -0.000338951"/>
-      <geometry>
-        <cylinder length="0.0337980384654" radius="0.0373293"/>
-      </geometry>
-    </collision>
-    <collision>
-      <origin rpy="-1.56738494938 1.42197043963 -1.41859762505" xyz="0.005822 -0.000121 -0.000347"/>
-      <geometry>
-        <sphere radius="0.0373293"/>
-      </geometry>
-    </collision>
-    <collision>
-      <origin rpy="-1.56738494938 1.42197043963 -1.41859762505" xyz="0.039246 0.004891 -0.000330"/>
-      <geometry>
-        <sphere radius="0.0373293"/>
-      </geometry>
-    </collision>
-    <inertial>
-      <mass value="1"/>
-      <inertia ixx="0.01" ixy="0" ixz="0" iyy="0.01" iyz="0" izz="0.01"/>
-    </inertial>
-  </link>
-  <joint name="meca_axis_5_joint_A" type="revolute">
-    <origin rpy="0.0 0.0 0.0" xyz="0.12 0.0 0.0"/>
-    <axis xyz="0.0 1.0 0.0"/>
-    <parent link="meca_axis_4_link_A"/>
-    <child link="meca_axis_5_link_A"/>
-    <limit effort="10.0" lower="-2.00" upper="2.00" velocity="5.23599"/>
-  </joint>
-  <!-- Joint 6 -->
-  <link name="meca_axis_6_link_A">
-    <visual>
-      <origin xyz="0 0 0" rpy="0 0 0" />
-      <geometry>
-        <mesh filename="package://mecademic_description/meshes/meca_500_r3_j6.dae" />
-      </geometry>
-    </visual>
-    <collision>
-      <origin rpy="3.14152943169 -0.0847389814668 -3.14010139052" xyz="-0.002858345 7.482995e-07 -1.9915e-05"/>
-      <geometry>
-        <cylinder length="0.00588946257883" radius="0.0134707"/>
-      </geometry>
-    </collision>
-    <collision>
-      <origin rpy="3.14152943169 -0.0847389814668 -3.14010139052" xyz="-0.002609 0.000001 0.002914"/>
-      <geometry>
-        <sphere radius="0.0134707"/>
-      </geometry>
-    </collision>
-    <collision>
-      <origin rpy="3.14152943169 -0.0847389814668 -3.14010139052" xyz="-0.003108 0.000001 -0.002954"/>
-      <geometry>
-        <sphere radius="0.0134707"/>
-      </geometry>
-    </collision>
-    <inertial>
-      <mass value="1"/>
-      <inertia ixx="0.01" ixy="0" ixz="0" iyy="0.01" iyz="0" izz="0.01"/>
-    </inertial>
-  </link>
-  <joint name="meca_axis_6_joint_A" type="revolute">
-    <origin rpy="0.0 0.0 0.0" xyz="0.07 0.0 0.0"/>
-    <axis xyz="1.0 0.0 0.0"/>
-    <parent link="meca_axis_5_link_A"/>
-    <child link="meca_axis_6_link_A"/>
-    <limit effort="10.0" lower="-3.142" upper="3.142" velocity="8.72665"/>
-  </joint>
-  <!-- 2nd ROBOT -->
+ <!-- 2nd ROBOT -->
  <joint name="world_to_base_B" type="fixed">
     <origin xyz="0.3 0.65 0" rpy="0 0 0"/>

Commit message: fix 1st joint name

File: mecademic_description/urdf/meca_500_r3.urdf.xacro (robot description, xacro)
@@ -10,5 +10,5 @@
       <plugin filename="libxbot2_gz_joint_server.so" name="xbot2_gz_joint_server">
           <pid>
-            <pid name="J1_B" profile="small_mot"/>
+            <pid name="BL4104C_1" profile="small_mot"/>
             <pid name="meca_axis_1_joint_B" profile="small_mot"/>
             <pid name="meca_axis_2_joint_B" profile="small_mot"/>
@@ -63,5 +63,5 @@
     <material>Gazebo/Blue</material>
   </gazebo>
-  <joint name="J1_B" type="continuous">
+  <joint name="BL4104C_1" type="continuous">
     <axis rpy="0 0 0" xyz="0 0 1"/>
     <parent link="BL4104C_1_stator"/>

File: mecademic_description/urdf/meca_500_r3_capsule.urdf.xacro (robot description, xacro)
@@ -10,5 +10,5 @@
       <plugin filename="libxbot2_gz_joint_server.so" name="xbot2_gz_joint_server">
           <pid>
-            <pid name="J1_B" profile="small_mot"/>
+            <pid name="BL4104C_1" profile="small_mot"/>
             <pid name="meca_axis_1_joint_B" profile="small_mot"/>
             <pid name="meca_axis_2_joint_B" profile="small_mot"/>
@@ -63,5 +63,5 @@
     <material>Gazebo/Blue</material>
   </gazebo>
-  <joint name="J1_B" type="continuous">
+  <joint name="BL4104C_1" type="continuous">
     <axis rpy="0 0 0" xyz="0 0 1"/>
     <parent link="BL4104C_1_stator"/>
