Commit message: fix: rotary table joint should be revolute and not continuous

File: mecademic_description/urdf/meca_500_r3.urdf.xacro (robot description, xacro)
@@ -1,3 +1,27 @@
 <robot name="meca_500_r3" xmlns:xacro="http://ros.org/wiki/xacro">
+<material name="blue">
+    <color rgba="0 0 0.8 1"/>
+  </material>
+  <material name="black">
+    <color rgba="0 0 0 1"/>
+  </material>
+  <material name="white">
+    <color rgba="1 1 1 1"/>
+  </material>
+  <material name="grey">
+    <color rgba="0.5 0.5 0.5 1"/>
+  </material>
+  <material name="red">
+    <color rgba="1 0 0 1"/>
+  </material>
+  <material name="green">
+    <color rgba="0 1 0 1"/>
+  </material>
+  <material name="yellow">
+    <color rgba="1 1 0 1"/>
+  </material>
+  <material name="tree_green">
+    <color rgba="0.13 0.54 0.13 1"/>
+  </material>
   <link name="world"/>
 <!-- 2nd ROBOT -->
@@ -10,5 +34,5 @@
       <plugin filename="libxbot2_gz_joint_server.so" name="xbot2_gz_joint_server">
           <pid>
-            <pid name="BL4104C_1" profile="small_mot"/>
+            <pid name="BL4104C_1" profile="medium_mot"/>
             <pid name="meca_axis_1_joint_B" profile="small_mot"/>
             <pid name="meca_axis_2_joint_B" profile="small_mot"/>
@@ -23,5 +47,5 @@
   <link name="base_link_B">
     <inertial>
-      <mass value="10.0"/>
+      <mass value="0.1"/>
       <inertia ixx="1.0e-03" ixy="0.0" ixz="0.0" iyy="1.0e-03" iyz="0.0" izz="1.0e-03"/>
     </inertial>
@@ -63,10 +87,10 @@
     <material>Gazebo/Blue</material>
   </gazebo>
-  <joint name="BL4104C_1" type="continuous">
+  <joint name="BL4104C_1" type="revolute">
     <axis rpy="0 0 0" xyz="0 0 1"/>
     <parent link="BL4104C_1_stator"/>
     <child link="L_1_B"/>
     <origin rpy="0.0 -0.0 0.0" xyz="0.0 0.0 0.21"/>
-    <limit effort="147" lower="-2.8" upper="2.8" velocity="100000000"/>
+    <limit effort="147" lower="-2.0" upper="2.0" velocity="1"/>
   </joint>
   <!-- <xacro:property name="visual" value="package://sps-pkg/database/modular/meshes/yaw_base.stl"/> -->

File: mecademic_description/urdf/meca_500_r3_capsule.urdf.xacro (robot description, xacro)
@@ -1,3 +1,27 @@
 <robot name="meca_500_r3" xmlns:xacro="http://ros.org/wiki/xacro">
+<material name="blue">
+    <color rgba="0 0 0.8 1"/>
+  </material>
+  <material name="black">
+    <color rgba="0 0 0 1"/>
+  </material>
+  <material name="white">
+    <color rgba="1 1 1 1"/>
+  </material>
+  <material name="grey">
+    <color rgba="0.5 0.5 0.5 1"/>
+  </material>
+  <material name="red">
+    <color rgba="1 0 0 1"/>
+  </material>
+  <material name="green">
+    <color rgba="0 1 0 1"/>
+  </material>
+  <material name="yellow">
+    <color rgba="1 1 0 1"/>
+  </material>
+  <material name="tree_green">
+    <color rgba="0.13 0.54 0.13 1"/>
+  </material>
   <link name="world"/>
  <!-- 2nd ROBOT -->
@@ -10,5 +34,5 @@
       <plugin filename="libxbot2_gz_joint_server.so" name="xbot2_gz_joint_server">
           <pid>
-            <pid name="BL4104C_1" profile="small_mot"/>
+            <pid name="BL4104C_1" profile="medium_mot"/>
             <pid name="meca_axis_1_joint_B" profile="small_mot"/>
             <pid name="meca_axis_2_joint_B" profile="small_mot"/>
@@ -23,5 +47,5 @@
   <link name="base_link_B">
     <inertial>
-      <mass value="10.0"/>
+      <mass value="0.1"/>
       <inertia ixx="1.0e-03" ixy="0.0" ixz="0.0" iyy="1.0e-03" iyz="0.0" izz="1.0e-03"/>
     </inertial>
@@ -63,10 +87,10 @@
     <material>Gazebo/Blue</material>
   </gazebo>
-  <joint name="BL4104C_1" type="continuous">
+  <joint name="BL4104C_1" type="revolute">
     <axis rpy="0 0 0" xyz="0 0 1"/>
     <parent link="BL4104C_1_stator"/>
     <child link="L_1_B"/>
     <origin rpy="0.0 -0.0 0.0" xyz="0.0 0.0 0.21"/>
-    <limit effort="147" lower="-2.8" upper="2.8" velocity="100000000"/>
+    <limit effort="147" lower="-2.0" upper="2.0" velocity="1"/>
   </joint>
   <!-- <xacro:property name="visual" value="package://sps-pkg/database/modular/meshes/yaw_base.stl"/> -->
@@ -144,17 +168,4 @@
     </inertial>
   </link>
-  <gazebo>
-      <plugin filename="libxbot2_gz_joint_server.so" name="xbot2_gz_joint_server">
-          <pid>
-            <pid name="meca_axis_1_joint_B" profile="small_mot"/>
-            <pid name="meca_axis_2_joint_B" profile="small_mot"/>
-            <pid name="meca_axis_3_joint_B" profile="small_mot"/>
-            <pid name="meca_axis_4_joint_B" profile="small_mot"/>
-            <pid name="meca_axis_5_joint_B" profile="small_mot"/>
-            <pid name="meca_axis_6_joint_B" profile="small_mot"/>
-          </pid>
-          <gain d="5" name="small_mot" p="100"/>
-      </plugin>
-    </gazebo>
   <!-- Joint 1 -->
   <link name="meca_axis_1_link_B">

Commit message: new homing state and small urdf fixes

File: mecademic_description/urdf/meca_500_r3.urdf.xacro (robot description, xacro)
@@ -91,5 +91,5 @@
     <parent link="BL4104C_1_stator"/>
     <child link="L_1_B"/>
-    <origin rpy="0.0 -0.0 0.0" xyz="0.0 0.0 0.21"/>
+    <origin rpy="0.0 -0.0 -1.57" xyz="0.0 0.0 0.21"/>
     <limit effort="147" lower="-2.0" upper="2.0" velocity="1"/>
   </joint>
@@ -135,5 +135,5 @@
     <parent link="L_1_B"/>
     <child link="meca_base_link_B"/>
-    <origin rpy="0 1.571 0" xyz="0.05 0.0 0.05"/>
+    <origin rpy="0 1.571 0" xyz="0.05 0.0 0.065"/>
   </joint>
     <!-- Base link is the center of the robot's bottom plate -->

File: mecademic_description/urdf/meca_500_r3_capsule.urdf.xacro (robot description, xacro)
@@ -91,5 +91,5 @@
     <parent link="BL4104C_1_stator"/>
     <child link="L_1_B"/>
-    <origin rpy="0.0 -0.0 0.0" xyz="0.0 0.0 0.21"/>
+    <origin rpy="0.0 -0.0 -1.57" xyz="0.0 0.0 0.21"/>
     <limit effort="147" lower="-2.0" upper="2.0" velocity="1"/>
   </joint>
@@ -135,5 +135,5 @@
     <parent link="L_1_B"/>
     <child link="meca_base_link_B"/>
-    <origin rpy="0 1.571 0" xyz="0.05 0.0 0.05"/>
+    <origin rpy="0 1.571 0" xyz="0.05 0.0 0.065"/>
   </joint>
     <!-- Base link is the center of the robot's bottom plate -->

Commit message: [urdf] better limits for the last joint

File: mecademic_description/urdf/meca_500_r3.urdf.xacro (robot description, xacro)
@@ -310,5 +310,5 @@
     <child link="meca_axis_6_link_B" />
     <axis xyz="1 0 0" />
-    <limit effort="10.0" velocity="8.72665" lower="-3.142" upper="3.142" />
+    <limit effort="10.0" velocity="8.72665" lower="-4.0" upper="4.0" />
   </joint>
   <!-- BUFFERS -->

File: mecademic_description/urdf/meca_500_r3_capsule.urdf.xacro (robot description, xacro)
@@ -394,5 +394,5 @@
     <child link="meca_axis_6_link_B" />
     <axis xyz="1 0 0" />
-    <limit effort="10.0" lower="-3.142" upper="3.142" velocity="8.72665"/>
+    <limit effort="10.0" lower="-4.0" upper="4.0" velocity="8.72665"/>
   </joint>
   <!-- BUFFERS -->

Commit message: add second robot meca_A

File: mecademic_description/urdf/meca_500_r3.urdf.xacro (robot description, xacro)
@@ -25,9 +25,9 @@
   </material>
   <link name="world"/>
-<!-- 2nd ROBOT -->
-  <joint name="world_to_base_B" type="fixed">
+<!-- 1st ROBOT -->
+  <joint name="world_to_base_A" type="fixed">
       <origin xyz="0.3 0.65 0" rpy="0 0 0"/>
       <parent link="world"/>
-      <child link="base_link_B"/>
+      <child link="base_link_A"/>
     </joint>
   <gazebo>
@@ -35,15 +35,15 @@
           <pid>
             <pid name="BL4104C_1" profile="medium_mot"/>
-            <pid name="meca_axis_1_joint_B" profile="small_mot"/>
-            <pid name="meca_axis_2_joint_B" profile="small_mot"/>
-            <pid name="meca_axis_3_joint_B" profile="small_mot"/>
-            <pid name="meca_axis_4_joint_B" profile="small_mot"/>
-            <pid name="meca_axis_5_joint_B" profile="small_mot"/>
-            <pid name="meca_axis_6_joint_B" profile="small_mot"/>
+            <pid name="meca_axis_1_joint_A" profile="small_mot"/>
+            <pid name="meca_axis_2_joint_A" profile="small_mot"/>
+            <pid name="meca_axis_3_joint_A" profile="small_mot"/>
+            <pid name="meca_axis_4_joint_A" profile="small_mot"/>
+            <pid name="meca_axis_5_joint_A" profile="small_mot"/>
+            <pid name="meca_axis_6_joint_A" profile="small_mot"/>
           </pid>
           <gain d="5" name="small_mot" p="100"/>
       </plugin>
     </gazebo>
-  <link name="base_link_B">
+  <link name="base_link_A">
     <inertial>
       <mass value="0.1"/>
@@ -53,5 +53,5 @@
   <joint name="fixed_BL4104C_1" type="fixed">
     <axis rpy="0 0 0" xyz="0 0 1"/>
-    <parent link="base_link_B"/>
+    <parent link="base_link_A"/>
     <child link="BL4104C_1_stator"/>
     <origin rpy="0.0 -0.0 0.0" xyz="0.0 0.0 0.0"/>
@@ -90,4 +90,291 @@
     <axis rpy="0 0 0" xyz="0 0 1"/>
     <parent link="BL4104C_1_stator"/>
+    <child link="L_1_A"/>
+    <origin rpy="0.0 -0.0 -1.57" xyz="0.0 0.0 0.21"/>
+    <limit effort="147" lower="-2.0" upper="2.0" velocity="1"/>
+  </joint>
+  <!-- <xacro:property name="visual" value="package://sps-pkg/database/modular/meshes/yaw_base.stl"/> -->
+  <link name="L_1_A">
+    <visual>
+      <origin rpy="0.0 0.0 0.0" xyz="0.0 0.0 0.002"/>
+      <geometry>
+        <cylinder length="0.004" radius="0.063"/>
+      </geometry>
+      <material name="grey"/>
+    </visual>
+    <collision>
+      <origin rpy="0.0 0.0 0.0" xyz="0.0 0.0 0.002"/>
+      <geometry>
+        <cylinder length="0.004" radius="0.063"/>
+      </geometry>
+      <material name="grey"/>
+    </collision>
+    <inertial>
+      <origin rpy="0 0 0" xyz="0.0 0.0 -0.024438213"/>
+      <mass value="0.42322395"/>
+      <inertia ixx="0.00063746146" ixy="1.1903424e-05" ixz="6.7230372e-07" iyy="0.00064218987" iyz="2.203073e-05" izz="0.001009674"/>
+    </inertial>
+  </link>
+  <joint name="fixed_L_1_A_rotor_fast" type="fixed">
+    <axis rpy="0 0 0" xyz="0 0 1"/>
+    <parent link="L_1_A"/>
+    <child link="L_1_A_rotor_fast"/>
+    <origin rpy="0.0 -0.0 0.0" xyz="0.0 0.0 0.0"/>
+  </joint>
+  <link name="L_1_A_rotor_fast">
+    <inertial>
+      <origin rpy="0 0 0" xyz="0.0 0.0 -0.0978986"/>
+      <mass value="0.197124"/>
+      <inertia ixx="0.00016128216" ixy="-2.4229e-07" ixz="3.771218e-06" iyy="0.00016138868" iyz="-2.4900687e-06" izz="0.1287638"/>
+      <!-- ixz="0.0003771218" -->
+      <!-- iyz="-0.00024900687" -->
+      <!-- izz="1.287638e-05" -->
+    </inertial>
+  </link>
+  <joint name="L_1_A_to_meca_base_link_A" type="fixed">
+    <parent link="L_1_A"/>
+    <child link="meca_base_link_A"/>
+    <origin rpy="0 1.571 0" xyz="0.05 0.0 0.065"/>
+  </joint>
+    <!-- Base link is the center of the robot's bottom plate -->
+  <link name="meca_base_link_A">
+    <visual>
+      <origin xyz="0 0 0" rpy="0 0 0" />
+      <geometry>
+        <mesh filename="package://mecademic_description/meshes/meca_500_r3_base.dae" />
+      </geometry>
+    </visual>
+    <collision>
+      <origin xyz="0 0 0" rpy="0 0 0" />
+      <geometry>
+        <mesh filename="package://mecademic_description/meshes/meca_500_r3_base_collision.stl" />
+      </geometry>
+    </collision>
+    <inertial>
+      <mass value="1"/>
+      <inertia ixx="0.01" ixy="0" ixz="0" iyy="0.01" iyz="0" izz="0.01"/>
+    </inertial>
+  </link>
+  <!-- Joint 1 -->
+  <link name="meca_axis_1_link_A">
+    <visual>
+      <origin xyz="0 0 0" rpy="0 0 0" />
+      <geometry>
+        <mesh filename="package://mecademic_description/meshes/meca_500_r3_j1.dae" />
+      </geometry>
+    </visual>
+    <collision>
+      <origin xyz="0 0 0" rpy="0 0 0" />
+      <geometry>
+        <mesh filename="package://mecademic_description/meshes/meca_500_r3_j1_collision.stl" />
+      </geometry>
+    </collision>
+    <inertial>
+      <mass value="1"/>
+      <inertia ixx="0.01" ixy="0" ixz="0" iyy="0.01" iyz="0" izz="0.01"/>
+    </inertial>
+  </link>
+  <joint name="meca_axis_1_joint_A" type="revolute">
+    <origin xyz="0.012498 0 0.091" rpy="0 0 0" />
+    <parent link="meca_base_link_A" />
+    <child link="meca_axis_1_link_A" />
+    <axis xyz="0 0 1" />
+    <limit effort="10.0" velocity="2.61799" lower="-3.05" upper="3.05" />
+  </joint>
+  <!-- Joint 2 -->
+  <link name="meca_axis_2_link_A">
+    <visual>
+      <origin xyz="0 0 0" rpy="0 0 0" />
+      <geometry>
+        <mesh filename="package://mecademic_description/meshes/meca_500_r3_j2.dae" />
+      </geometry>
+    </visual>
+    <collision>
+      <origin xyz="0 0 0" rpy="0 0 0" />
+      <geometry>
+        <mesh filename="package://mecademic_description/meshes/meca_500_r3_j2_collision.stl" />
+      </geometry>
+    </collision>
+    <inertial>
+      <mass value="1"/>
+      <inertia ixx="0.01" ixy="0" ixz="0" iyy="0.01" iyz="0" izz="0.01"/>
+    </inertial>
+  </link>
+  <joint name="meca_axis_2_joint_A" type="revolute">
+    <origin xyz="0 0 0.044" rpy="0 0 0" />
+    <parent link="meca_axis_1_link_A" />
+    <child link="meca_axis_2_link_A" />
+    <axis xyz="0 1 0" />
+    <limit effort="10.0" velocity="2.61799" lower="-1.22" upper="1.57" />
+  </joint>
+  <!-- Joint 3 -->
+  <link name="meca_axis_3_link_A">
+    <visual>
+      <origin xyz="0 0 0" rpy="0 0 0" />
+      <geometry>
+        <mesh filename="package://mecademic_description/meshes/meca_500_r3_j3.dae" />
+      </geometry>
+    </visual>
+    <collision>
+      <origin xyz="0 0 0" rpy="0 0 0" />
+      <geometry>
+        <mesh filename="package://mecademic_description/meshes/meca_500_r3_j3_collision.stl" />
+      </geometry>
+    </collision>
+    <inertial>
+      <mass value="1"/>
+      <inertia ixx="0.01" ixy="0" ixz="0" iyy="0.01" iyz="0" izz="0.01"/>
+    </inertial>
+  </link>
+  <joint name="meca_axis_3_joint_A" type="revolute">
+    <origin xyz="0 0 0.135" rpy="0 0 0" />
+    <parent link="meca_axis_2_link_A" />
+    <child link="meca_axis_3_link_A" />
+    <axis xyz="0 1 0" />
+    <limit effort="10.0" velocity="3.14159" lower="-2.35" upper="1.22" />
+  </joint>
+  <!-- Joint 4 -->
+  <link name="meca_axis_4_link_A">
+    <visual>
+      <origin xyz="0 0 0" rpy="0 0 0" />
+      <geometry>
+        <mesh filename="package://mecademic_description/meshes/meca_500_r3_j4.dae" />
+      </geometry>
+    </visual>
+    <collision>
+      <origin xyz="0 0 0" rpy="0 0 0" />
+      <geometry>
+        <mesh filename="package://mecademic_description/meshes/meca_500_r3_j4_collision.stl" />
+      </geometry>
+    </collision>
+    <inertial>
+      <mass value="1"/>
+      <inertia ixx="0.01" ixy="0" ixz="0" iyy="0.01" iyz="0" izz="0.01"/>
+    </inertial>
+  </link>
+  <joint name="meca_axis_4_joint_A" type="revolute">
+    <origin xyz="0 0 0.038" rpy="0 0 0" />
+    <parent link="meca_axis_3_link_A" />
+    <child link="meca_axis_4_link_A" />
+    <axis xyz="1 0 0" />
+    <limit effort="10.0" velocity="5.23599" lower="-2.96" upper="2.96" />
+  </joint>
+  <!-- Joint 5 -->
+  <link name="meca_axis_5_link_A">
+    <visual>
+      <origin xyz="0 0 0" rpy="0 0 0" />
+      <geometry>
+        <mesh filename="package://mecademic_description/meshes/meca_500_r3_j5.dae" />
+      </geometry>
+    </visual>
+    <collision>
+      <origin xyz="0 0 0" rpy="0 0 0" />
+      <geometry>
+        <mesh filename="package://mecademic_description/meshes/meca_500_r3_j5_collision.stl" />
+      </geometry>
+    </collision>
+    <inertial>
+      <mass value="1"/>
+      <inertia ixx="0.01" ixy="0" ixz="0" iyy="0.01" iyz="0" izz="0.01"/>
+    </inertial>
+  </link>
+  <joint name="meca_axis_5_joint_A" type="revolute">
+    <origin xyz="0.12 0 0" rpy="0 0 0" />
+    <parent link="meca_axis_4_link_A" />
+    <child link="meca_axis_5_link_A" />
+    <axis xyz="0 1 0" />
+    <limit effort="10.0" velocity="5.23599" lower="-2.00" upper="2.00" />
+  </joint>
+  <!-- Joint 6 -->
+  <link name="meca_axis_6_link_A">
+    <visual>
+      <origin xyz="0 0 0" rpy="0 0 0" />
+      <geometry>
+        <mesh filename="package://mecademic_description/meshes/meca_500_r3_j6.dae" />
+      </geometry>
+    </visual>
+    <collision>
+      <origin xyz="0 0 0" rpy="0 0 0" />
+      <geometry>
+        <mesh filename="package://mecademic_description/meshes/meca_500_r3_j6_collision.stl" />
+      </geometry>
+    </collision>
+    <inertial>
+      <mass value="1"/>
+      <inertia ixx="0.01" ixy="0" ixz="0" iyy="0.01" iyz="0" izz="0.01"/>
+    </inertial>
+  </link>
+  <joint name="meca_axis_6_joint_A" type="revolute">
+    <origin xyz="0.07 0 0" rpy="0 0 0" />
+    <parent link="meca_axis_5_link_A" />
+    <child link="meca_axis_6_link_A" />
+    <axis xyz="1 0 0" />
+    <limit effort="10.0" velocity="8.72665" lower="-4.0" upper="4.0" />
+  </joint>
+<!-- 2nd ROBOT -->
+  <joint name="world_to_base_B" type="fixed">
+      <origin xyz="0.3 0.65 0" rpy="0 0 0"/>
+      <parent link="world"/>
+      <child link="base_link_B"/>
+    </joint>
+  <gazebo>
+      <plugin filename="libxbot2_gz_joint_server.so" name="xbot2_gz_joint_server">
+          <pid>
+            <pid name="BL4104C_2" profile="medium_mot"/>
+            <pid name="meca_axis_1_joint_B" profile="small_mot"/>
+            <pid name="meca_axis_2_joint_B" profile="small_mot"/>
+            <pid name="meca_axis_3_joint_B" profile="small_mot"/>
+            <pid name="meca_axis_4_joint_B" profile="small_mot"/>
+            <pid name="meca_axis_5_joint_B" profile="small_mot"/>
+            <pid name="meca_axis_6_joint_B" profile="small_mot"/>
+          </pid>
+          <gain d="5" name="small_mot" p="100"/>
+      </plugin>
+    </gazebo>
+  <link name="base_link_B">
+    <inertial>
+      <mass value="0.1"/>
+      <inertia ixx="1.0e-03" ixy="0.0" ixz="0.0" iyy="1.0e-03" iyz="0.0" izz="1.0e-03"/>
+    </inertial>
+  </link>
+  <joint name="fixed_BL4104C_2" type="fixed">
+    <axis rpy="0 0 0" xyz="0 0 1"/>
+    <parent link="base_link_B"/>
+    <child link="BL4104C_2_stator"/>
+    <origin rpy="0.0 -0.0 0.0" xyz="0.0 0.0 0.0"/>
+  </joint>
+  <link name="BL4104C_2_stator">
+    <visual>
+      <!-- Load mesh. Rotate the origin frame (this is because of how the .stl was saved) -->
+      <origin rpy="0.0 0.0 0.0" xyz="0.0 0.0 0.105"/>
+      <geometry>
+        <cylinder length="0.21" radius="0.13"/>
+      </geometry>
+      <material name="grey"/>
+    </visual>
+    <collision>
+      <origin rpy="0.0 0.0 0.0" xyz="0.0 0.0 0.105"/>
+      <geometry>
+        <cylinder length="0.21" radius="0.13"/>
+      </geometry>
+    </collision>
+    <inertial>
+      <origin rpy="0 0 0" xyz="0.0 0.0 0.10614489"/>
+      <mass value="2.0554934"/>
+      <inertia ixx="0.01068855" ixy="-1.14168e-05" ixz="2.71689e-06" iyy="0.010584907" iyz="8.76312e-05" izz="0.0032026258"/>
+    </inertial>
+  </link>
+  <gazebo reference="BL4104C_2_stator">
+    <mu1>0.2</mu1>
+    <mu2>0.2</mu2>
+    <kp>1000000.0</kp>
+    <kd>1.0</kd>
+    <maxVel>0.0</maxVel>
+    <minDepth>0.0001</minDepth>
+    <material>Gazebo/Blue</material>
+  </gazebo>
+  <joint name="BL4104C_2" type="revolute">
+    <axis rpy="0 0 0" xyz="0 0 1"/>
+    <parent link="BL4104C_2_stator"/>
     <child link="L_1_B"/>
     <origin rpy="0.0 -0.0 -1.57" xyz="0.0 0.0 0.21"/>
