Commit message: merge urdf with mr/sps

File: mecademic_description/urdf/meca_500_r3.urdf.xacro (robot description, xacro)
@@ -27,8 +27,8 @@
 <!-- 1st ROBOT -->
   <joint name="world_to_base_A" type="fixed">
-      <origin xyz="0.3 0.65 0" rpy="0 0 0"/>
-      <parent link="world"/>
-      <child link="base_link_A"/>
-    </joint>
+    <parent link="world"/>
+    <child link="base_link_A"/>
+    <origin rpy="0 0 0" xyz="0.3 0 0.0"/>
+  </joint>
   <gazebo>
       <plugin filename="libxbot2_gz_joint_server.so" name="xbot2_gz_joint_server">
@@ -55,19 +55,20 @@
     <parent link="base_link_A"/>
     <child link="BL4104C_1_stator"/>
-    <origin rpy="0.0 -0.0 0.0" xyz="0.0 0.0 0.0"/>
+    <origin xyz="0.0 0.0 0.06" rpy="0 0 0" />
   </joint>
   <link name="BL4104C_1_stator">
     <visual>
-      <!-- Load mesh. Rotate the origin frame (this is because of how the .stl was saved) -->
-      <origin rpy="0.0 0.0 0.0" xyz="0.0 0.0 0.105"/>
-      <geometry>
-        <cylinder length="0.21" radius="0.13"/>
-      </geometry>
-      <material name="grey"/>
-    </visual>
-    <collision>
-      <origin rpy="0.0 0.0 0.0" xyz="0.0 0.0 0.105"/>
-      <geometry>
-        <cylinder length="0.21" radius="0.13"/>
+      <geometry>
+        <box size="0.72 0.12 0.1"/>
+      </geometry>
+      <material name="blue">
+        <color rgba="0 0 .8 1"/>
+      </material>
+      <origin xyz="0 0 0" rpy="0 0 0" />
+    </visual>
+    <collision>
+      <origin xyz="0 0 0" rpy="0 0 0" />
+      <geometry>
+        <box size="0.72 0.12 0.1"/>
       </geometry>
     </collision>
@@ -87,26 +88,26 @@
     <material>Gazebo/Blue</material>
   </gazebo>
-  <joint name="BL4104C_1" type="revolute">
-    <axis rpy="0 0 0" xyz="0 0 1"/>
+  <joint name="BL4104C_1" type="prismatic">
+    <axis xyz="1 0 0"/>
     <parent link="BL4104C_1_stator"/>
     <child link="L_1_A"/>
-    <origin rpy="0.0 -0.0 -1.57" xyz="0.0 0.0 0.21"/>
-    <limit effort="147" lower="-2.0" upper="2.0" velocity="1"/>
-  </joint>
-  <!-- <xacro:property name="visual" value="package://sps-pkg/database/modular/meshes/yaw_base.stl"/> -->
+    <limit effort="1000.0" lower="-0.26" upper="0.26" velocity="100"/>
+    <origin rpy="0 0 0" xyz="0 0 0.09"/>
+  </joint>
   <link name="L_1_A">
     <visual>
-      <origin rpy="0.0 0.0 0.0" xyz="0.0 0.0 0.002"/>
-      <geometry>
-        <cylinder length="0.004" radius="0.063"/>
-      </geometry>
-      <material name="grey"/>
-    </visual>
-    <collision>
-      <origin rpy="0.0 0.0 0.0" xyz="0.0 0.0 0.002"/>
-      <geometry>
-        <cylinder length="0.004" radius="0.063"/>
-      </geometry>
-      <material name="grey"/>
+      <geometry>
+        <box size="0.2 0.2 0.04"/>
+      </geometry>
+      <material name="blue">
+        <color rgba="0 0 .8 1"/>
+      </material>
+      <origin xyz="0 0 -0.02" rpy="0 0 0" />
+    </visual>
+    <collision>
+      <origin xyz="0 0 -0.02" rpy="0 0 0" />
+      <geometry>
+        <box size="0.2 0.2 0.04"/>
+      </geometry>
     </collision>
     <inertial>
@@ -116,24 +117,8 @@
     </inertial>
   </link>
-  <joint name="fixed_L_1_A_rotor_fast" type="fixed">
-    <axis rpy="0 0 0" xyz="0 0 1"/>
-    <parent link="L_1_A"/>
-    <child link="L_1_A_rotor_fast"/>
-    <origin rpy="0.0 -0.0 0.0" xyz="0.0 0.0 0.0"/>
-  </joint>
-  <link name="L_1_A_rotor_fast">
-    <inertial>
-      <origin rpy="0 0 0" xyz="0.0 0.0 -0.0978986"/>
-      <mass value="0.197124"/>
-      <inertia ixx="0.00016128216" ixy="-2.4229e-07" ixz="3.771218e-06" iyy="0.00016138868" iyz="-2.4900687e-06" izz="0.1287638"/>
-      <!-- ixz="0.0003771218" -->
-      <!-- iyz="-0.00024900687" -->
-      <!-- izz="1.287638e-05" -->
-    </inertial>
-  </link>
   <joint name="L_1_A_to_meca_base_link_A" type="fixed">
     <parent link="L_1_A"/>
     <child link="meca_base_link_A"/>
-    <origin rpy="0 1.571 0" xyz="0.05 0.0 0.065"/>
+    <origin rpy="0 1.571 1.571" xyz="0.0 0 0.05"/>
   </joint>
     <!-- Base link is the center of the robot's bottom plate -->

File: mecademic_description/urdf/meca_500_r3_capsule.urdf.xacro (robot description, xacro)
@@ -26,8 +26,8 @@
   <link name="world"/>
 <!-- 1st ROBOT -->
- <joint name="world_to_base_A" type="fixed">
-    <origin xyz="0.3 0.65 0" rpy="0 0 0"/>
+  <joint name="world_to_base_A" type="fixed">
     <parent link="world"/>
     <child link="base_link_A"/>
+    <origin rpy="0 0 0" xyz="0.3 0 0.0"/>
   </joint>
   <gazebo>
@@ -55,19 +55,20 @@
     <parent link="base_link_A"/>
     <child link="BL4104C_1_stator"/>
-    <origin rpy="0.0 -0.0 0.0" xyz="0.0 0.0 0.0"/>
+    <origin xyz="0.0 0.0 0.06" rpy="0 0 0" />
   </joint>
   <link name="BL4104C_1_stator">
     <visual>
-      <!-- Load mesh. Rotate the origin frame (this is because of how the .stl was saved) -->
-      <origin rpy="0.0 0.0 0.0" xyz="0.0 0.0 0.105"/>
-      <geometry>
-        <cylinder length="0.21" radius="0.13"/>
-      </geometry>
-      <material name="grey"/>
-    </visual>
-    <collision>
-      <origin rpy="0.0 0.0 0.0" xyz="0.0 0.0 0.105"/>
-      <geometry>
-        <cylinder length="0.21" radius="0.13"/>
+      <geometry>
+        <box size="0.72 0.12 0.1"/>
+      </geometry>
+      <material name="blue">
+        <color rgba="0 0 .8 1"/>
+      </material>
+      <origin xyz="0 0 0" rpy="0 0 0" />
+    </visual>
+    <collision>
+      <origin xyz="0 0 0" rpy="0 0 0" />
+      <geometry>
+        <box size="0.72 0.12 0.1"/>
       </geometry>
     </collision>
@@ -87,26 +88,26 @@
     <material>Gazebo/Blue</material>
   </gazebo>
-  <joint name="BL4104C_1" type="revolute">
-    <axis rpy="0 0 0" xyz="0 0 1"/>
+  <joint name="BL4104C_1" type="prismatic">
+    <axis xyz="1 0 0"/>
     <parent link="BL4104C_1_stator"/>
     <child link="L_1_A"/>
-    <origin rpy="0.0 -0.0 -1.57" xyz="0.0 0.0 0.21"/>
-    <limit effort="147" lower="-2.0" upper="2.0" velocity="1"/>
-  </joint>
-  <!-- <xacro:property name="visual" value="package://sps-pkg/database/modular/meshes/yaw_base.stl"/> -->
+    <limit effort="1000.0" lower="-0.26" upper="0.26" velocity="100"/>
+    <origin rpy="0 0 0" xyz="0 0 0.09"/>
+  </joint>
   <link name="L_1_A">
     <visual>
-      <origin rpy="0.0 0.0 0.0" xyz="0.0 0.0 0.002"/>
-      <geometry>
-        <cylinder length="0.004" radius="0.063"/>
-      </geometry>
-      <material name="grey"/>
-    </visual>
-    <collision>
-      <origin rpy="0.0 0.0 0.0" xyz="0.0 0.0 0.002"/>
-      <geometry>
-        <cylinder length="0.004" radius="0.063"/>
-      </geometry>
-      <material name="grey"/>
+      <geometry>
+        <box size="0.2 0.2 0.04"/>
+      </geometry>
+      <material name="blue">
+        <color rgba="0 0 .8 1"/>
+      </material>
+      <origin xyz="0 0 -0.02" rpy="0 0 0" />
+    </visual>
+    <collision>
+      <origin xyz="0 0 -0.02" rpy="0 0 0" />
+      <geometry>
+        <box size="0.2 0.2 0.04"/>
+      </geometry>
     </collision>
     <inertial>
@@ -116,24 +117,8 @@
     </inertial>
   </link>
-  <joint name="fixed_L_1_A_rotor_fast" type="fixed">
-    <axis rpy="0 0 0" xyz="0 0 1"/>
-    <parent link="L_1_A"/>
-    <child link="L_1_A_rotor_fast"/>
-    <origin rpy="0.0 -0.0 0.0" xyz="0.0 0.0 0.0"/>
-  </joint>
-  <link name="L_1_A_rotor_fast">
-    <inertial>
-      <origin rpy="0 0 0" xyz="0.0 0.0 -0.0978986"/>
-      <mass value="0.197124"/>
-      <inertia ixx="0.00016128216" ixy="-2.4229e-07" ixz="3.771218e-06" iyy="0.00016138868" iyz="-2.4900687e-06" izz="0.1287638"/>
-      <!-- ixz="0.0003771218" -->
-      <!-- iyz="-0.00024900687" -->
-      <!-- izz="1.287638e-05" -->
-    </inertial>
-  </link>
   <joint name="L_1_A_to_meca_base_link_A" type="fixed">
     <parent link="L_1_A"/>
     <child link="meca_base_link_A"/>
-    <origin rpy="0 1.571 0" xyz="0.05 0.0 0.065"/>
+    <origin rpy="0 1.571 1.571" xyz="0.0 0 0.05"/>
   </joint>
     <!-- Base link is the center of the robot's bottom plate -->
@@ -425,8 +410,8 @@
     <axis rpy="0 0 0" xyz="0 0 1"/>
     <parent link="base_link_B"/>
-    <child link="BL4104C_1_stator"/>
+    <child link="BL4104C_2_stator"/>
     <origin rpy="0.0 -0.0 0.0" xyz="0.0 0.0 0.0"/>
   </joint>
-  <link name="BL4104C_1_stator">
+  <link name="BL4104C_2_stator">
     <visual>
       <!-- Load mesh. Rotate the origin frame (this is because of how the .stl was saved) -->
@@ -449,5 +434,5 @@
     </inertial>
   </link>
-  <gazebo reference="BL4104C_1_stator">
+  <gazebo reference="BL4104C_2_stator">
     <mu1>0.2</mu1>
     <mu2>0.2</mu2>

Commit message: refactor: Change joint name according to: repo: albero_xbot2-config-files commit: c0ab0293ad

File: mecademic_description/urdf/meca_500_r3.urdf.xacro (robot description, xacro)
@@ -51,11 +51,11 @@
     </inertial>
   </link>
-  <joint name="fixed_BL4104C_1" type="fixed">
+  <joint name="fixed_linear_motor" type="fixed">
     <axis rpy="0 0 0" xyz="0 0 1"/>
     <parent link="base_link_A"/>
-    <child link="BL4104C_1_stator"/>
+    <child link="linear_motor_stator"/>
     <origin xyz="0.0 0.0 0.06" rpy="0 0 0" />
   </joint>
-  <link name="BL4104C_1_stator">
+  <link name="linear_motor_stator">
     <visual>
       <geometry>
@@ -79,5 +79,5 @@
     </inertial>
   </link>
-  <gazebo reference="BL4104C_1_stator">
+  <gazebo reference="linear_motor_stator">
     <mu1>0.2</mu1>
     <mu2>0.2</mu2>
@@ -88,10 +88,10 @@
     <material>Gazebo/Blue</material>
   </gazebo>
-  <joint name="BL4104C_1" type="prismatic">
+  <joint name="linear_motor" type="prismatic">
     <axis xyz="1 0 0"/>
-    <parent link="BL4104C_1_stator"/>
+    <parent link="linear_motor_stator"/>
     <child link="L_1_A"/>
-    <limit effort="1000.0" lower="-0.26" upper="0.26" velocity="100"/>
-    <origin rpy="0 0 0" xyz="0 0 0.09"/>
+    <limit effort="100.0" lower="-0.002" upper="0.400" velocity="0.5"/>
+    <origin rpy="0 0 0" xyz="-0.26 0 0.09"/>
   </joint>
   <link name="L_1_A">
@@ -323,11 +323,11 @@
     </inertial>
   </link>
-  <joint name="fixed_BL4104C_2" type="fixed">
+  <joint name="fixed_rotary_table" type="fixed">
     <axis rpy="0 0 0" xyz="0 0 1"/>
     <parent link="base_link_B"/>
-    <child link="BL4104C_2_stator"/>
+    <child link="rotary_table_stator"/>
     <origin rpy="0.0 -0.0 0.0" xyz="0.0 0.0 0.0"/>
   </joint>
-  <link name="BL4104C_2_stator">
+  <link name="rotary_table_stator">
     <visual>
       <!-- Load mesh. Rotate the origin frame (this is because of how the .stl was saved) -->
@@ -350,5 +350,5 @@
     </inertial>
   </link>
-  <gazebo reference="BL4104C_2_stator">
+  <gazebo reference="rotary_table_stator">
     <mu1>0.2</mu1>
     <mu2>0.2</mu2>
@@ -359,7 +359,7 @@
     <material>Gazebo/Blue</material>
   </gazebo>
-  <joint name="BL4104C_2" type="revolute">
+  <joint name="rotary_table" type="revolute">
     <axis rpy="0 0 0" xyz="0 0 1"/>
-    <parent link="BL4104C_2_stator"/>
+    <parent link="rotary_table_stator"/>
     <child link="L_1_B"/>
     <origin rpy="0.0 -0.0 -1.57" xyz="0.0 0.0 0.21"/>

File: mecademic_description/urdf/meca_500_r3_capsule.urdf.xacro (robot description, xacro)
@@ -51,11 +51,11 @@
     </inertial>
   </link>
-  <joint name="fixed_BL4104C_1" type="fixed">
+  <joint name="fixed_linear_motor" type="fixed">
     <axis rpy="0 0 0" xyz="0 0 1"/>
     <parent link="base_link_A"/>
-    <child link="BL4104C_1_stator"/>
+    <child link="linear_motor_stator"/>
     <origin xyz="0.0 0.0 0.06" rpy="0 0 0" />
   </joint>
-  <link name="BL4104C_1_stator">
+  <link name="linear_motor_stator">
     <visual>
       <geometry>
@@ -79,5 +79,5 @@
     </inertial>
   </link>
-  <gazebo reference="BL4104C_1_stator">
+  <gazebo reference="linear_motor_stator">
     <mu1>0.2</mu1>
     <mu2>0.2</mu2>
@@ -88,10 +88,10 @@
     <material>Gazebo/Blue</material>
   </gazebo>
-  <joint name="BL4104C_1" type="prismatic">
+  <joint name="linear_motor" type="prismatic">
     <axis xyz="1 0 0"/>
-    <parent link="BL4104C_1_stator"/>
+    <parent link="linear_motor_stator"/>
     <child link="L_1_A"/>
-    <limit effort="1000.0" lower="-0.26" upper="0.26" velocity="100"/>
-    <origin rpy="0 0 0" xyz="0 0 0.09"/>
+    <limit effort="100.0" lower="-0.002" upper="0.400" velocity="0.5"/>
+    <origin rpy="0 0 0" xyz="-0.26 0 0.09"/>
   </joint>
   <link name="L_1_A">
@@ -407,11 +407,11 @@
     </inertial>
   </link>
-  <joint name="fixed_BL4104C_2" type="fixed">
+  <joint name="fixed_rotary_table" type="fixed">
     <axis rpy="0 0 0" xyz="0 0 1"/>
     <parent link="base_link_B"/>
-    <child link="BL4104C_2_stator"/>
+    <child link="rotary_table_stator"/>
     <origin rpy="0.0 -0.0 0.0" xyz="0.0 0.0 0.0"/>
   </joint>
-  <link name="BL4104C_2_stator">
+  <link name="rotary_table_stator">
     <visual>
       <!-- Load mesh. Rotate the origin frame (this is because of how the .stl was saved) -->
@@ -434,5 +434,5 @@
     </inertial>
   </link>
-  <gazebo reference="BL4104C_2_stator">
+  <gazebo reference="rotary_table_stator">
     <mu1>0.2</mu1>
     <mu2>0.2</mu2>
@@ -443,7 +443,7 @@
     <material>Gazebo/Blue</material>
   </gazebo>
-  <joint name="BL4104C_2" type="revolute">
+  <joint name="rotary_table" type="revolute">
     <axis rpy="0 0 0" xyz="0 0 1"/>
-    <parent link="BL4104C_2_stator"/>
+    <parent link="rotary_table_stator"/>
     <child link="L_1_B"/>
     <origin rpy="0.0 -0.0 -1.57" xyz="0.0 0.0 0.21"/>

Commit message: update urdf to reflect lab setup

File: mecademic_description/urdf/meca_500_r3.urdf.xacro (robot description, xacro)
@@ -29,5 +29,5 @@
     <parent link="world"/>
     <child link="base_link_A"/>
-    <origin rpy="0 0 0" xyz="0.3 0 0.0"/>
+    <origin rpy="0 0 0" xyz="0.509 0.12 0.0"/>
   </joint>
   <gazebo>
@@ -51,14 +51,42 @@
     </inertial>
   </link>
+  <joint name="fixed_gear_box" type="fixed">
+    <axis rpy="0 0 0" xyz="0 0 0"/>
+    <parent link="base_link_A"/>
+    <child link="gear_box"/>
+    <origin xyz="0.431 0.0 0.05" rpy="0 0 1.571" />
+  </joint>
+ <link name="gear_box">
+    <visual>
+      <geometry>
+        <cylinder length="0.366" radius="0.12"/>
+      </geometry>
+      <material name="blue">
+        <color rgba="0 0 .8 1"/>
+      </material>
+      <origin xyz="0.183 0 0" rpy="0 1.571 0" />
+    </visual>
+    <collision>
+      <origin xyz="0.183 0 0" rpy="0 1.571 0" />
+      <geometry>
+        <cylinder length="0.366" radius="0.12" />
+      </geometry>
+    </collision>
+    <inertial>
+      <origin rpy="0 0 0" xyz="0.0 0.0 0.10614489"/>
+      <mass value="2.0554934"/>
+      <inertia ixx="0.01068855" ixy="-1.14168e-05" ixz="2.71689e-06" iyy="0.010584907" iyz="8.76312e-05" izz="0.0032026258"/>
+    </inertial>
+  </link>
   <joint name="fixed_linear_motor" type="fixed">
     <axis rpy="0 0 0" xyz="0 0 1"/>
     <parent link="base_link_A"/>
     <child link="linear_motor_stator"/>
-    <origin xyz="0.0 0.0 0.06" rpy="0 0 0" />
+    <origin xyz="0.0 0.0 0.05" rpy="0 0 0" />
   </joint>
   <link name="linear_motor_stator">
     <visual>
       <geometry>
-        <box size="0.72 0.12 0.1"/>
+        <box size="0.98 0.12 0.1"/>
       </geometry>
       <material name="blue">
@@ -70,5 +98,5 @@
       <origin xyz="0 0 0" rpy="0 0 0" />
       <geometry>
-        <box size="0.72 0.12 0.1"/>
+        <box size="0.98 0.12 0.1"/>
       </geometry>
     </collision>
@@ -299,5 +327,5 @@
 <!-- 2nd ROBOT -->
   <joint name="world_to_base_B" type="fixed">
-      <origin xyz="0.3 0.65 0" rpy="0 0 0"/>
+      <origin xyz="0.456 0.572 0" rpy="0 0 -1.571"/>
       <parent link="world"/>
       <child link="base_link_B"/>
@@ -318,4 +346,19 @@
     </gazebo>
   <link name="base_link_B">
+    <visual>
+      <geometry>
+        <box size="0.450 0.167 0.03"/>
+      </geometry>
+      <material name="blue">
+        <color rgba="0 0 .8 1"/>
+      </material>
+      <origin xyz="0 0 0" rpy="0 0 0" />
+    </visual>
+    <collision>
+      <origin xyz="0 0 0" rpy="0 1.571 0" />
+      <geometry>
+        <cylinder length="0.450" radius="0.15"/>
+      </geometry>
+    </collision>
     <inertial>
       <mass value="0.1"/>
@@ -341,5 +384,5 @@
       <origin rpy="0.0 0.0 0.0" xyz="0.0 0.0 0.105"/>
       <geometry>
-        <cylinder length="0.21" radius="0.13"/>
+        <cylinder length="0.21" radius="0.132"/>
       </geometry>
     </collision>
@@ -363,5 +406,5 @@
     <parent link="rotary_table_stator"/>
     <child link="L_1_B"/>
-    <origin rpy="0.0 -0.0 -1.57" xyz="0.0 0.0 0.21"/>
+    <origin rpy="0.0 -0.0 0" xyz="0.0 0.0 0.21"/>
     <limit effort="147" lower="-2.0" upper="2.0" velocity="1"/>
   </joint>
@@ -407,5 +450,5 @@
     <parent link="L_1_B"/>
     <child link="meca_base_link_B"/>
-    <origin rpy="0 1.571 0" xyz="0.05 0.0 0.065"/>
+    <origin rpy="0 1.571 0" xyz="0.095 0.0 0.0645"/>
   </joint>
     <!-- Base link is the center of the robot's bottom plate -->

File: mecademic_description/urdf/meca_500_r3_capsule.urdf.xacro (robot description, xacro)
@@ -29,5 +29,5 @@
     <parent link="world"/>
     <child link="base_link_A"/>
-    <origin rpy="0 0 0" xyz="0.3 0 0.0"/>
+    <origin rpy="0 0 0" xyz="0.509 0.12 0.0"/>
   </joint>
   <gazebo>
@@ -51,14 +51,42 @@
     </inertial>
   </link>
+  <joint name="fixed_gear_box" type="fixed">
+    <axis rpy="0 0 0" xyz="0 0 0"/>
+    <parent link="base_link_A"/>
+    <child link="gear_box"/>
+    <origin xyz="0.431 0.0 0.05" rpy="0 0 1.571" />
+  </joint>
+  <link name="gear_box">
+    <visual>
+      <geometry>
+        <cylinder length="0.366" radius="0.12"/>
+      </geometry>
+      <material name="blue">
+        <color rgba="0 0 .8 1"/>
+      </material>
+      <origin xyz="0.183 0 0" rpy="0 1.571 0" />
+    </visual>
+    <collision>
+      <origin xyz="0.183 0 0" rpy="0 1.571 0" />
+      <geometry>
+        <cylinder length="0.366" radius="0.12" />
+      </geometry>
+    </collision>
+    <inertial>
+      <origin rpy="0 0 0" xyz="0.0 0.0 0.10614489"/>
+      <mass value="2.0554934"/>
+      <inertia ixx="0.01068855" ixy="-1.14168e-05" ixz="2.71689e-06" iyy="0.010584907" iyz="8.76312e-05" izz="0.0032026258"/>
+    </inertial>
+  </link>
   <joint name="fixed_linear_motor" type="fixed">
     <axis rpy="0 0 0" xyz="0 0 1"/>
     <parent link="base_link_A"/>
     <child link="linear_motor_stator"/>
-    <origin xyz="0.0 0.0 0.06" rpy="0 0 0" />
+    <origin xyz="0.0 0.0 0.05" rpy="0 0 0" />
   </joint>
   <link name="linear_motor_stator">
     <visual>
       <geometry>
-        <box size="0.72 0.12 0.1"/>
+        <box size="0.98 0.12 0.1"/>
       </geometry>
       <material name="blue">
@@ -68,7 +96,7 @@
     </visual>
     <collision>
-      <origin xyz="0 0 0" rpy="0 0 0" />
-      <geometry>
-        <box size="0.72 0.12 0.1"/>
+      <origin xyz="0 0 0.05" rpy="0 1.571 0" />
+      <geometry>
+        <cylinder length="0.98" radius="0.12" />
       </geometry>
     </collision>
@@ -383,5 +411,5 @@
  <!-- 2nd ROBOT -->
  <joint name="world_to_base_B" type="fixed">
-    <origin xyz="0.3 0.65 0" rpy="0 0 0"/>
+    <origin xyz="0.456 0.572 0" rpy="0 0 0"/>
     <parent link="world"/>
     <child link="base_link_B"/>
@@ -402,4 +430,19 @@
     </gazebo>
   <link name="base_link_B">
+    <visual>
+      <geometry>
+        <box size="0.450 0.167 0.03"/>
+      </geometry>
+      <material name="blue">
+        <color rgba="0 0 .8 1"/>
+      </material>
+      <origin xyz="0 0 0" rpy="0 0 0" />
+    </visual>
+    <collision>
+      <origin xyz="0 0 0" rpy="0 1.571 0" />
+      <geometry>
+        <cylinder length="0.450" radius="0.15"/>
+      </geometry>
+    </collision>
     <inertial>
       <mass value="0.1"/>
@@ -411,5 +454,5 @@
     <parent link="base_link_B"/>
     <child link="rotary_table_stator"/>
-    <origin rpy="0.0 -0.0 0.0" xyz="0.0 0.0 0.0"/>
+    <origin rpy="0.0 -0.0 0.0" xyz="0.0 0.0 0.03"/>
   </joint>
   <link name="rotary_table_stator">
@@ -425,5 +468,5 @@
       <origin rpy="0.0 0.0 0.0" xyz="0.0 0.0 0.105"/>
       <geometry>
-        <cylinder length="0.21" radius="0.13"/>
+        <cylinder length="0.21" radius="0.132"/>
       </geometry>
     </collision>
@@ -491,5 +534,5 @@
     <parent link="L_1_B"/>
     <child link="meca_base_link_B"/>
-    <origin rpy="0 1.571 0" xyz="0.05 0.0 0.065"/>
+    <origin rpy="0 1.571 0" xyz="0.095 0.0 0.0645"/>
   </joint>
     <!-- Base link is the center of the robot's bottom plate -->

Commit message: remove visual and collision from base link

File: mecademic_description/urdf/meca_500_r3.urdf.xacro (robot description, xacro)
@@ -52,5 +52,5 @@
   </link>
   <joint name="fixed_gear_box" type="fixed">
-    <axis rpy="0 0 0" xyz="0 0 0"/>
+    <axis rpy="0 0 0" xyz="0 0 1"/>
     <parent link="base_link_A"/>
     <child link="gear_box"/>
@@ -346,4 +346,16 @@
     </gazebo>
   <link name="base_link_B">
+    <inertial>
+      <mass value="0.1"/>
+      <inertia ixx="1.0e-03" ixy="0.0" ixz="0.0" iyy="1.0e-03" iyz="0.0" izz="1.0e-03"/>
+    </inertial>
+  </link>
+  <joint name="base_to_platform" type="fixed">
+    <axis rpy="0 0 0" xyz="0 0 1"/>
+    <parent link="base_link_B"/>
+    <child link="platform"/>
+    <origin rpy="0.0 -0.0 0.0" xyz="0.0 0.0 0.0"/>
+  </joint>
+  <link name="platform">
     <visual>
       <geometry>
@@ -368,7 +380,7 @@
   <joint name="fixed_rotary_table" type="fixed">
     <axis rpy="0 0 0" xyz="0 0 1"/>
-    <parent link="base_link_B"/>
+    <parent link="platform"/>
     <child link="rotary_table_stator"/>
-    <origin rpy="0.0 -0.0 0.0" xyz="0.0 0.0 0.0"/>
+    <origin rpy="0.0 -0.0 0.0" xyz="0.0 0.0 0.03"/>
   </joint>
   <link name="rotary_table_stator">

File: mecademic_description/urdf/meca_500_r3_capsule.urdf.xacro (robot description, xacro)
@@ -52,5 +52,5 @@
   </link>
   <joint name="fixed_gear_box" type="fixed">
-    <axis rpy="0 0 0" xyz="0 0 0"/>
+    <axis rpy="0 0 0" xyz="0 0 1"/>
     <parent link="base_link_A"/>
     <child link="gear_box"/>
@@ -430,4 +430,16 @@
     </gazebo>
   <link name="base_link_B">
+    <inertial>
+      <mass value="0.1"/>
+      <inertia ixx="1.0e-03" ixy="0.0" ixz="0.0" iyy="1.0e-03" iyz="0.0" izz="1.0e-03"/>
+    </inertial>
+  </link>
+  <joint name="base_to_platform" type="fixed">
+    <axis rpy="0 0 0" xyz="0 0 1"/>
+    <parent link="base_link_B"/>
+    <child link="platform"/>
+    <origin rpy="0.0 -0.0 0.0" xyz="0.0 0.0 0.0"/>
+  </joint>
+  <link name="platform">
     <visual>
       <geometry>
@@ -452,5 +464,5 @@
   <joint name="fixed_rotary_table" type="fixed">
     <axis rpy="0 0 0" xyz="0 0 1"/>
-    <parent link="base_link_B"/>
+    <parent link="platform"/>
     <child link="rotary_table_stator"/>
     <origin rpy="0.0 -0.0 0.0" xyz="0.0 0.0 0.03"/>
