Commit message: remove axis from fixed joints

File: mecademic_description/urdf/meca_500_r3.urdf.xacro (robot description, xacro)
@@ -52,5 +52,4 @@
   </link>
   <joint name="fixed_gear_box" type="fixed">
-    <axis rpy="0 0 0" xyz="0 0 1"/>
     <parent link="base_link_A"/>
     <child link="gear_box"/>
@@ -80,5 +79,4 @@
   </link>
   <joint name="fixed_linear_motor" type="fixed">
-    <axis rpy="0 0 0" xyz="0 0 1"/>
     <parent link="base_link_A"/>
     <child link="linear_motor_stator"/>
@@ -352,5 +350,4 @@
   </link>
   <joint name="base_to_platform" type="fixed">
-    <axis rpy="0 0 0" xyz="0 0 1"/>
     <parent link="base_link_B"/>
     <child link="platform"/>
@@ -379,5 +376,4 @@
   </link>
   <joint name="fixed_rotary_table" type="fixed">
-    <axis rpy="0 0 0" xyz="0 0 1"/>
     <parent link="platform"/>
     <child link="rotary_table_stator"/>
@@ -444,5 +440,4 @@
   </link>
   <joint name="fixed_L_1_B_rotor_fast" type="fixed">
-    <axis rpy="0 0 0" xyz="0 0 1"/>
     <parent link="L_1_B"/>
     <child link="L_1_B_rotor_fast"/>

File: mecademic_description/urdf/meca_500_r3_capsule.urdf.xacro (robot description, xacro)
@@ -52,5 +52,4 @@
   </link>
   <joint name="fixed_gear_box" type="fixed">
-    <axis rpy="0 0 0" xyz="0 0 1"/>
     <parent link="base_link_A"/>
     <child link="gear_box"/>
@@ -80,5 +79,4 @@
   </link>
   <joint name="fixed_linear_motor" type="fixed">
-    <axis rpy="0 0 0" xyz="0 0 1"/>
     <parent link="base_link_A"/>
     <child link="linear_motor_stator"/>
@@ -436,5 +434,4 @@
   </link>
   <joint name="base_to_platform" type="fixed">
-    <axis rpy="0 0 0" xyz="0 0 1"/>
     <parent link="base_link_B"/>
     <child link="platform"/>
@@ -463,5 +460,4 @@
   </link>
   <joint name="fixed_rotary_table" type="fixed">
-    <axis rpy="0 0 0" xyz="0 0 1"/>
     <parent link="platform"/>
     <child link="rotary_table_stator"/>
@@ -528,5 +524,4 @@
   </link>
   <joint name="fixed_L_1_B_rotor_fast" type="fixed">
-    <axis rpy="0 0 0" xyz="0 0 1"/>
     <parent link="L_1_B"/>
     <child link="L_1_B_rotor_fast"/>

Commit message: fix urdf collision

File: mecademic_description/urdf/meca_500_r3.urdf.xacro (robot description, xacro)
@@ -94,7 +94,7 @@
     </visual>
     <collision>
-      <origin xyz="0 0 0" rpy="0 0 0" />
-      <geometry>
-        <box size="0.98 0.12 0.1"/>
+      <origin xyz="0 0 0.05" rpy="0 1.571 0" />
+      <geometry>
+        <cylinder length="0.98" radius="0.12" />
       </geometry>
     </collision>
@@ -352,5 +352,5 @@
     <parent link="base_link_B"/>
     <child link="platform"/>
-    <origin rpy="0.0 -0.0 0.0" xyz="0.0 0.0 0.0"/>
+    <origin rpy="0.0 -0.0 0" xyz="0.0 0.0 0.0"/>
   </joint>
   <link name="platform">
@@ -362,8 +362,8 @@
         <color rgba="0 0 .8 1"/>
       </material>
-      <origin xyz="0 0 0" rpy="0 0 0" />
-    </visual>
-    <collision>
-      <origin xyz="0 0 0" rpy="0 1.571 0" />
+      <origin xyz="0 0 0.015" rpy="0 0 1.571" />
+    </visual>
+    <collision>
+      <origin xyz="0 0 0" rpy="1.571 0 0" />
       <geometry>
         <cylinder length="0.450" radius="0.15"/>

File: mecademic_description/urdf/meca_500_r3_capsule.urdf.xacro (robot description, xacro)
@@ -407,10 +407,10 @@
     <limit effort="10.0" lower="-4.0" upper="4.0" velocity="8.72665"/>
   </joint>
- <!-- 2nd ROBOT -->
- <joint name="world_to_base_B" type="fixed">
-    <origin xyz="0.456 0.572 0" rpy="0 0 0"/>
-    <parent link="world"/>
-    <child link="base_link_B"/>
-  </joint>
+<!-- 2nd ROBOT -->
+  <joint name="world_to_base_B" type="fixed">
+      <origin xyz="0.456 0.572 0" rpy="0 0 -1.571"/>
+      <parent link="world"/>
+      <child link="base_link_B"/>
+    </joint>
   <gazebo>
       <plugin filename="libxbot2_gz_joint_server.so" name="xbot2_gz_joint_server">
@@ -436,5 +436,5 @@
     <parent link="base_link_B"/>
     <child link="platform"/>
-    <origin rpy="0.0 -0.0 0.0" xyz="0.0 0.0 0.0"/>
+    <origin rpy="0.0 -0.0 0" xyz="0.0 0.0 0.0"/>
   </joint>
   <link name="platform">
@@ -446,8 +446,8 @@
         <color rgba="0 0 .8 1"/>
       </material>
-      <origin xyz="0 0 0" rpy="0 0 0" />
-    </visual>
-    <collision>
-      <origin xyz="0 0 0" rpy="0 1.571 0" />
+      <origin xyz="0 0 0.015" rpy="0 0 1.571" />
+    </visual>
+    <collision>
+      <origin xyz="0 0 0" rpy="1.571 0 0" />
       <geometry>
         <cylinder length="0.450" radius="0.15"/>
@@ -498,5 +498,5 @@
     <parent link="rotary_table_stator"/>
     <child link="L_1_B"/>
-    <origin rpy="0.0 -0.0 -1.57" xyz="0.0 0.0 0.21"/>
+    <origin rpy="0.0 -0.0 0" xyz="0.0 0.0 0.21"/>
     <limit effort="147" lower="-2.0" upper="2.0" velocity="1"/>
   </joint>

Commit message: remove meca on linear actuator

File: mecademic_description/urdf/meca_500_r3.urdf.xacro (robot description, xacro)
@@ -114,5 +114,5 @@
     <material>Gazebo/Blue</material>
   </gazebo>
-  <joint name="linear_motor" type="prismatic">
+  <joint name="linear_motor" type="fixed">
     <axis xyz="1 0 0"/>
     <parent link="linear_motor_stator"/>
@@ -143,184 +143,4 @@
     </inertial>
   </link>
-  <joint name="L_1_A_to_meca_base_link_A" type="fixed">
-    <parent link="L_1_A"/>
-    <child link="meca_base_link_A"/>
-    <origin rpy="0 1.571 1.571" xyz="0.0 0 0.05"/>
-  </joint>
-    <!-- Base link is the center of the robot's bottom plate -->
-  <link name="meca_base_link_A">
-    <visual>
-      <origin xyz="0 0 0" rpy="0 0 0" />
-      <geometry>
-        <mesh filename="package://mecademic_description/meshes/meca_500_r3_base.dae" />
-      </geometry>
-    </visual>
-    <collision>
-      <origin xyz="0 0 0" rpy="0 0 0" />
-      <geometry>
-        <mesh filename="package://mecademic_description/meshes/meca_500_r3_base_collision.stl" />
-      </geometry>
-    </collision>
-    <inertial>
-      <mass value="1"/>
-      <inertia ixx="0.01" ixy="0" ixz="0" iyy="0.01" iyz="0" izz="0.01"/>
-    </inertial>
-  </link>
-  <!-- Joint 1 -->
-  <link name="meca_axis_1_link_A">
-    <visual>
-      <origin xyz="0 0 0" rpy="0 0 0" />
-      <geometry>
-        <mesh filename="package://mecademic_description/meshes/meca_500_r3_j1.dae" />
-      </geometry>
-    </visual>
-    <collision>
-      <origin xyz="0 0 0" rpy="0 0 0" />
-      <geometry>
-        <mesh filename="package://mecademic_description/meshes/meca_500_r3_j1_collision.stl" />
-      </geometry>
-    </collision>
-    <inertial>
-      <mass value="1"/>
-      <inertia ixx="0.01" ixy="0" ixz="0" iyy="0.01" iyz="0" izz="0.01"/>
-    </inertial>
-  </link>
-  <joint name="meca_axis_1_joint_A" type="revolute">
-    <origin xyz="0.012498 0 0.091" rpy="0 0 0" />
-    <parent link="meca_base_link_A" />
-    <child link="meca_axis_1_link_A" />
-    <axis xyz="0 0 1" />
-    <limit effort="10.0" velocity="2.61799" lower="-3.05" upper="3.05" />
-  </joint>
-  <!-- Joint 2 -->
-  <link name="meca_axis_2_link_A">
-    <visual>
-      <origin xyz="0 0 0" rpy="0 0 0" />
-      <geometry>
-        <mesh filename="package://mecademic_description/meshes/meca_500_r3_j2.dae" />
-      </geometry>
-    </visual>
-    <collision>
-      <origin xyz="0 0 0" rpy="0 0 0" />
-      <geometry>
-        <mesh filename="package://mecademic_description/meshes/meca_500_r3_j2_collision.stl" />
-      </geometry>
-    </collision>
-    <inertial>
-      <mass value="1"/>
-      <inertia ixx="0.01" ixy="0" ixz="0" iyy="0.01" iyz="0" izz="0.01"/>
-    </inertial>
-  </link>
-  <joint name="meca_axis_2_joint_A" type="revolute">
-    <origin xyz="0 0 0.044" rpy="0 0 0" />
-    <parent link="meca_axis_1_link_A" />
-    <child link="meca_axis_2_link_A" />
-    <axis xyz="0 1 0" />
-    <limit effort="10.0" velocity="2.61799" lower="-1.22" upper="1.57" />
-  </joint>
-  <!-- Joint 3 -->
-  <link name="meca_axis_3_link_A">
-    <visual>
-      <origin xyz="0 0 0" rpy="0 0 0" />
-      <geometry>
-        <mesh filename="package://mecademic_description/meshes/meca_500_r3_j3.dae" />
-      </geometry>
-    </visual>
-    <collision>
-      <origin xyz="0 0 0" rpy="0 0 0" />
-      <geometry>
-        <mesh filename="package://mecademic_description/meshes/meca_500_r3_j3_collision.stl" />
-      </geometry>
-    </collision>
-    <inertial>
-      <mass value="1"/>
-      <inertia ixx="0.01" ixy="0" ixz="0" iyy="0.01" iyz="0" izz="0.01"/>
-    </inertial>
-  </link>
-  <joint name="meca_axis_3_joint_A" type="revolute">
-    <origin xyz="0 0 0.135" rpy="0 0 0" />
-    <parent link="meca_axis_2_link_A" />
-    <child link="meca_axis_3_link_A" />
-    <axis xyz="0 1 0" />
-    <limit effort="10.0" velocity="3.14159" lower="-2.35" upper="1.22" />
-  </joint>
-  <!-- Joint 4 -->
-  <link name="meca_axis_4_link_A">
-    <visual>
-      <origin xyz="0 0 0" rpy="0 0 0" />
-      <geometry>
-        <mesh filename="package://mecademic_description/meshes/meca_500_r3_j4.dae" />
-      </geometry>
-    </visual>
-    <collision>
-      <origin xyz="0 0 0" rpy="0 0 0" />
-      <geometry>
-        <mesh filename="package://mecademic_description/meshes/meca_500_r3_j4_collision.stl" />
-      </geometry>
-    </collision>
-    <inertial>
-      <mass value="1"/>
-      <inertia ixx="0.01" ixy="0" ixz="0" iyy="0.01" iyz="0" izz="0.01"/>
-    </inertial>
-  </link>
-  <joint name="meca_axis_4_joint_A" type="revolute">
-    <origin xyz="0 0 0.038" rpy="0 0 0" />
-    <parent link="meca_axis_3_link_A" />
-    <child link="meca_axis_4_link_A" />
-    <axis xyz="1 0 0" />
-    <limit effort="10.0" velocity="5.23599" lower="-2.96" upper="2.96" />
-  </joint>
-  <!-- Joint 5 -->
-  <link name="meca_axis_5_link_A">
-    <visual>
-      <origin xyz="0 0 0" rpy="0 0 0" />
-      <geometry>
-        <mesh filename="package://mecademic_description/meshes/meca_500_r3_j5.dae" />
-      </geometry>
-    </visual>
-    <collision>
-      <origin xyz="0 0 0" rpy="0 0 0" />
-      <geometry>
-        <mesh filename="package://mecademic_description/meshes/meca_500_r3_j5_collision.stl" />
-      </geometry>
-    </collision>
-    <inertial>
-      <mass value="1"/>
-      <inertia ixx="0.01" ixy="0" ixz="0" iyy="0.01" iyz="0" izz="0.01"/>
-    </inertial>
-  </link>
-  <joint name="meca_axis_5_joint_A" type="revolute">
-    <origin xyz="0.12 0 0" rpy="0 0 0" />
-    <parent link="meca_axis_4_link_A" />
-    <child link="meca_axis_5_link_A" />
-    <axis xyz="0 1 0" />
-    <limit effort="10.0" velocity="5.23599" lower="-2.00" upper="2.00" />
-  </joint>
-  <!-- Joint 6 -->
-  <link name="meca_axis_6_link_A">
-    <visual>
-      <origin xyz="0 0 0" rpy="0 0 0" />
-      <geometry>
-        <mesh filename="package://mecademic_description/meshes/meca_500_r3_j6.dae" />
-      </geometry>
-    </visual>
-    <collision>
-      <origin xyz="0 0 0" rpy="0 0 0" />
-      <geometry>
-        <mesh filename="package://mecademic_description/meshes/meca_500_r3_j6_collision.stl" />
-      </geometry>
-    </collision>
-    <inertial>
-      <mass value="1"/>
-      <inertia ixx="0.01" ixy="0" ixz="0" iyy="0.01" iyz="0" izz="0.01"/>
-    </inertial>
-  </link>
-  <joint name="meca_axis_6_joint_A" type="revolute">
-    <origin xyz="0.07 0 0" rpy="0 0 0" />
-    <parent link="meca_axis_5_link_A" />
-    <child link="meca_axis_6_link_A" />
-    <axis xyz="1 0 0" />
-    <limit effort="10.0" velocity="8.72665" lower="-4.0" upper="4.0" />
-  </joint>
 <!-- 2nd ROBOT -->
   <joint name="world_to_base_B" type="fixed">

File: mecademic_description/urdf/meca_500_r3_capsule.urdf.xacro (robot description, xacro)
@@ -114,5 +114,5 @@
     <material>Gazebo/Blue</material>
   </gazebo>
-  <joint name="linear_motor" type="prismatic">
+  <joint name="linear_motor" type="fixed">
     <axis xyz="1 0 0"/>
     <parent link="linear_motor_stator"/>
@@ -143,268 +143,4 @@
     </inertial>
   </link>
-  <joint name="L_1_A_to_meca_base_link_A" type="fixed">
-    <parent link="L_1_A"/>
-    <child link="meca_base_link_A"/>
-    <origin rpy="0 1.571 1.571" xyz="0.0 0 0.05"/>
-  </joint>
-    <!-- Base link is the center of the robot's bottom plate -->
-  <link name="meca_base_link_A">
-    <visual>
-      <origin xyz="0 0 0" rpy="0 0 0" />
-      <geometry>
-        <mesh filename="package://mecademic_description/meshes/meca_500_r3_base.dae" />
-      </geometry>
-    </visual>
-    <collision>
-      <origin rpy="-0.00464229562531 1.241639409 -0.00331992768483" xyz="0.002912665 2.5933825e-05 0.03195115"/>
-      <geometry>
-        <cylinder length="0.0247681427348" radius="0.069277"/>
-      </geometry>
-    </collision>
-    <collision>
-      <origin rpy="-0.00464229562531 1.241639409 -0.00331992768483" xyz="-0.008807 0.000007 0.027948"/>
-      <geometry>
-        <sphere radius="0.069277"/>
-      </geometry>
-    </collision>
-    <collision>
-      <origin rpy="-0.00464229562531 1.241639409 -0.00331992768483" xyz="0.014632 0.000045 0.035954"/>
-      <geometry>
-        <sphere radius="0.069277"/>
-      </geometry>
-    </collision>
-    <inertial>
-      <mass value="1"/>
-      <inertia ixx="0.01" ixy="0" ixz="0" iyy="0.01" iyz="0" izz="0.01"/>
-    </inertial>
-  </link>
-  <!-- Joint 1 -->
-  <link name="meca_axis_1_link_A">
-    <visual>
-      <origin xyz="0 0 0" rpy="0 0 0" />
-      <geometry>
-        <mesh filename="package://mecademic_description/meshes/meca_500_r3_j1.dae" />
-      </geometry>
-    </visual>
-    <collision>
-      <origin rpy="-1.5643390872 0.00108905813092 -0.00108204843032" xyz="1.404e-07 -0.00017605 0.03168225"/>
-      <geometry>
-        <cylinder length="0.0388249324419" radius="0.0530516"/>
-      </geometry>
-    </collision>
-    <collision>
-      <origin rpy="-1.5643390872 0.00108905813092 -0.00108204843032" xyz="-0.000021 -0.019588 0.031557"/>
-      <geometry>
-        <sphere radius="0.0530516"/>
-      </geometry>
-    </collision>
-    <collision>
-      <origin rpy="-1.5643390872 0.00108905813092 -0.00108204843032" xyz="0.000021 0.019236 0.031808"/>
-      <geometry>
-        <sphere radius="0.0530516"/>
-      </geometry>
-    </collision>
-    <inertial>
-      <mass value="1"/>
-      <inertia ixx="0.01" ixy="0" ixz="0" iyy="0.01" iyz="0" izz="0.01"/>
-    </inertial>
-  </link>
-  <joint name="meca_axis_1_joint_A" type="revolute">
-    <origin xyz="0.012498 0 0.091" rpy="0 0 0" />
-    <parent link="meca_base_link_A" />
-    <child link="meca_axis_1_link_A" />
-    <axis xyz="0 0 1" />
-    <limit effort="10.0" lower="-3.05" upper="3.05" velocity="2.61799"/>
-  </joint>
-  <!-- Joint 2 -->
-  <link name="meca_axis_2_link_A">
-    <visual>
-      <origin xyz="0 0 0" rpy="0 0 0" />
-      <geometry>
-        <mesh filename="package://mecademic_description/meshes/meca_500_r3_j2.dae" />
-      </geometry>
-    </visual>
-    <collision>
-      <origin rpy="3.14150631803 -0.0666872950524 -3.13900434911" xyz="-0.007204205 2.561655e-06 0.07263715"/>
-      <geometry>
-        <cylinder length="0.121249210008" radius="0.0578403"/>
-      </geometry>
-    </collision>
-    <collision>
-      <origin rpy="3.14150631803 -0.0666872950524 -3.13900434911" xyz="-0.003164 0.000008 0.133127"/>
-      <geometry>
-        <sphere radius="0.0578403"/>
-      </geometry>
-    </collision>
-    <collision>
-      <origin rpy="3.14150631803 -0.0666872950524 -3.13900434911" xyz="-0.011244 -0.000003 0.012147"/>
-      <geometry>
-        <sphere radius="0.0578403"/>
-      </geometry>
-    </collision>
-    <inertial>
-      <mass value="1"/>
-      <inertia ixx="0.01" ixy="0" ixz="0" iyy="0.01" iyz="0" izz="0.01"/>
-    </inertial>
-  </link>
-  <joint name="meca_axis_2_joint_A" type="revolute">
-    <origin xyz="0 0 0.044" rpy="0 0 0" />
-    <parent link="meca_axis_1_link_A" />
-    <child link="meca_axis_2_link_A" />
-    <axis xyz="0 1 0" />
-    <limit effort="10.0" lower="-1.22" upper="1.57" velocity="2.61799"/>
-  </joint>
-  <!-- Joint 3 -->
-  <link name="meca_axis_3_link_A">
-    <visual>
-      <origin xyz="0 0 0" rpy="0 0 0" />
-      <geometry>
-        <mesh filename="package://mecademic_description/meshes/meca_500_r3_j3.dae" />
-      </geometry>
-    </visual>
-    <collision>
-      <origin rpy="-0.0775632999618 0.486298597709 -0.0192491912301" xyz="0.009983498 -0.000990284 0.020095595"/>
-      <geometry>
-        <cylinder length="0.0408120816515" radius="0.0503272"/>
-      </geometry>
-    </collision>
-    <collision>
-      <origin rpy="-0.0775632999618 0.486298597709 -0.0192491912301" xyz="0.000447 -0.002388 0.002109"/>
-      <geometry>
-        <sphere radius="0.0503272"/>
-      </geometry>
-    </collision>
-    <collision>
-      <origin rpy="-0.0775632999618 0.486298597709 -0.0192491912301" xyz="0.019520 0.000408 0.038082"/>
-      <geometry>
-        <sphere radius="0.0503272"/>
-      </geometry>
-    </collision>
-    <inertial>
-      <mass value="1"/>
-      <inertia ixx="0.01" ixy="0" ixz="0" iyy="0.01" iyz="0" izz="0.01"/>
-    </inertial>
-  </link>
-  <joint name="meca_axis_3_joint_A" type="revolute">
-    <origin xyz="0 0 0.135" rpy="0 0 0" />
-    <parent link="meca_axis_2_link_A" />
-    <child link="meca_axis_3_link_A" />
-    <axis xyz="0 1 0" />
-    <limit effort="10.0" lower="-2.35" upper="1.22" velocity="3.14159"/>
-  </joint>
-  <!-- Joint 4 -->
-  <link name="meca_axis_4_link_A">
-    <visual>
-      <origin xyz="0 0 0" rpy="0 0 0" />
-      <geometry>
-        <mesh filename="package://mecademic_description/meshes/meca_500_r3_j4.dae" />
-      </geometry>
-    </visual>
-    <collision>
-      <origin rpy="-1.61527511752 1.5509782436 -1.59546790677" xyz="0.1018437 -0.00037629375 0.0004856635"/>
-      <geometry>
-        <cylinder length="0.0362997282424" radius="0.0387182"/>
-      </geometry>
-    </collision>
-    <collision>
-      <origin rpy="-1.61527511752 1.5509782436 -1.59546790677" xyz="0.083697 -0.000736 0.000502"/>
-      <geometry>
-        <sphere radius="0.0387182"/>
-      </geometry>
-    </collision>
-    <collision>
-      <origin rpy="-1.61527511752 1.5509782436 -1.59546790677" xyz="0.119990 -0.000017 0.000470"/>
-      <geometry>
-        <sphere radius="0.0387182"/>
-      </geometry>
-    </collision>
-    <inertial>
-      <mass value="1"/>
-      <inertia ixx="0.01" ixy="0" ixz="0" iyy="0.01" iyz="0" izz="0.01"/>
-    </inertial>
-  </link>
-  <joint name="meca_axis_4_joint_A" type="revolute">
-    <origin xyz="0 0 0.038" rpy="0 0 0" />
-    <parent link="meca_axis_3_link_A" />
-    <child link="meca_axis_4_link_A" />
-    <axis xyz="1 0 0" />
-   <limit effort="10.0" lower="-2.96" upper="2.96" velocity="5.23599"/>
-  </joint>
-  <!-- Joint 5 -->
-  <link name="meca_axis_5_link_A">
-    <visual>
-      <origin xyz="0 0 0" rpy="0 0 0" />
-      <geometry>
-        <mesh filename="package://mecademic_description/meshes/meca_500_r3_j5.dae" />
-      </geometry>
-    </visual>
-    <collision>
-      <origin rpy="-1.56738494938 1.42197043963 -1.41859762505" xyz="0.022533785 0.002385127 -0.000338951"/>
-      <geometry>
-        <cylinder length="0.0337980384654" radius="0.0373293"/>
-      </geometry>
-    </collision>
-    <collision>
-      <origin rpy="-1.56738494938 1.42197043963 -1.41859762505" xyz="0.005822 -0.000121 -0.000347"/>
-      <geometry>
-        <sphere radius="0.0373293"/>
-      </geometry>
-    </collision>
-    <collision>
-      <origin rpy="-1.56738494938 1.42197043963 -1.41859762505" xyz="0.039246 0.004891 -0.000330"/>
-      <geometry>
-        <sphere radius="0.0373293"/>
-      </geometry>
-    </collision>
-    <inertial>
-      <mass value="1"/>
-      <inertia ixx="0.01" ixy="0" ixz="0" iyy="0.01" iyz="0" izz="0.01"/>
-    </inertial>
-  </link>
-  <joint name="meca_axis_5_joint_A" type="revolute">
-    <origin xyz="0.12 0 0" rpy="0 0 0" />
-    <parent link="meca_axis_4_link_A" />
-    <child link="meca_axis_5_link_A" />
-    <axis xyz="0 1 0" />
-    <limit effort="10.0" lower="-2.00" upper="2.00" velocity="5.23599"/>
-  </joint>
-  <!-- Joint 6 -->
-  <link name="meca_axis_6_link_A">
-    <visual>
-      <origin xyz="0 0 0" rpy="0 0 0" />
-      <geometry>
-        <mesh filename="package://mecademic_description/meshes/meca_500_r3_j6.dae" />
-      </geometry>
-    </visual>
-    <collision>
-      <origin rpy="3.14152943169 -0.0847389814668 -3.14010139052" xyz="-0.002858345 7.482995e-07 -1.9915e-05"/>
-      <geometry>
-        <cylinder length="0.00588946257883" radius="0.0134707"/>
-      </geometry>
-    </collision>
-    <collision>
-      <origin rpy="3.14152943169 -0.0847389814668 -3.14010139052" xyz="-0.002609 0.000001 0.002914"/>
-      <geometry>
-        <sphere radius="0.0134707"/>
-      </geometry>
-    </collision>
-    <collision>
-      <origin rpy="3.14152943169 -0.0847389814668 -3.14010139052" xyz="-0.003108 0.000001 -0.002954"/>
-      <geometry>
-        <sphere radius="0.0134707"/>
-      </geometry>
-    </collision>
-    <inertial>
-      <mass value="1"/>
-      <inertia ixx="0.01" ixy="0" ixz="0" iyy="0.01" iyz="0" izz="0.01"/>
-    </inertial>
-  </link>
-  <joint name="meca_axis_6_joint_A" type="revolute">
-    <origin xyz="0.07 0 0" rpy="0 0 0" />
-    <parent link="meca_axis_5_link_A" />
-    <child link="meca_axis_6_link_A" />
-    <axis xyz="1 0 0" />
-    <limit effort="10.0" lower="-4.0" upper="4.0" velocity="8.72665"/>
-  </joint>
 <!-- 2nd ROBOT -->
   <joint name="world_to_base_B" type="fixed">

Commit message: fix collision radius of rotary actuator stator to protect sensor

File: mecademic_description/urdf/meca_500_r3.urdf.xacro (robot description, xacro)
@@ -392,5 +392,5 @@
       <origin rpy="0.0 0.0 0.0" xyz="0.0 0.0 0.105"/>
       <geometry>
-        <cylinder length="0.21" radius="0.132"/>
+        <cylinder length="0.21" radius="0.16"/>
       </geometry>
     </collision>

File: mecademic_description/urdf/meca_500_r3_capsule.urdf.xacro (robot description, xacro)
@@ -476,5 +476,5 @@
       <origin rpy="0.0 0.0 0.0" xyz="0.0 0.0 0.105"/>
       <geometry>
-        <cylinder length="0.21" radius="0.132"/>
+        <cylinder length="0.21" radius="0.16"/>
       </geometry>
     </collision>

Commit message: fix collision radius of rotary actuator stator to protect sensor

File: mecademic_description/urdf/meca_500_r3.urdf.xacro (robot description, xacro)
@@ -212,5 +212,5 @@
       <origin rpy="0.0 0.0 0.0" xyz="0.0 0.0 0.105"/>
       <geometry>
-        <cylinder length="0.21" radius="0.132"/>
+        <cylinder length="0.21" radius="0.16"/>
       </geometry>
     </collision>

File: mecademic_description/urdf/meca_500_r3_capsule.urdf.xacro (robot description, xacro)
@@ -212,5 +212,5 @@
       <origin rpy="0.0 0.0 0.0" xyz="0.0 0.0 0.105"/>
       <geometry>
-        <cylinder length="0.21" radius="0.132"/>
+        <cylinder length="0.21" radius="0.16"/>
       </geometry>
     </collision>
