Commit message: add end-effector collision sphere

File: mecademic_description/urdf/meca_500_r3.urdf.xacro (robot description, xacro)
@@ -454,4 +454,27 @@
     <limit effort="10.0" velocity="8.72665" lower="-4.0" upper="4.0" />
   </joint>
+  <link name="ee_sphere">
+    <visual>
+      <origin xyz="0 0 0" rpy="0 0 0" />
+      <geometry>
+        <sphere radius="0.06" />
+      </geometry>
+    </visual>
+    <collision>
+      <origin xyz="0 0 0" rpy="0 0 0" />
+      <geometry>
+        <sphere radius="0.06" />
+      </geometry>
+    </collision>
+    <inertial>
+      <mass value="0.1"/>
+      <inertia ixx="0.01" ixy="0" ixz="0" iyy="0.01" iyz="0" izz="0.01"/>
+    </inertial>
+  </link>
+  <joint name="meca_axis_6_to_ee_sphere" type="fixed">
+    <origin xyz="0 0 0" rpy="0 0 0" />
+    <parent link="meca_axis_6_link_B" />
+    <child link="ee_sphere" />
+  </joint>
   <!-- BUFFERS -->
   <joint name="world_to_buffer" type="fixed">

File: mecademic_description/urdf/meca_500_r3_capsule.urdf.xacro (robot description, xacro)
@@ -538,4 +538,27 @@
     <limit effort="10.0" lower="-4.0" upper="4.0" velocity="8.72665"/>
   </joint>
+  <link name="ee_sphere">
+    <visual>
+      <origin xyz="0 0 0" rpy="0 0 0" />
+      <geometry>
+        <sphere radius="0.06" />
+      </geometry>
+    </visual>
+    <collision>
+      <origin xyz="0 0 0" rpy="0 0 0" />
+      <geometry>
+        <sphere radius="0.06" />
+      </geometry>
+    </collision>
+    <inertial>
+      <mass value="0.1"/>
+      <inertia ixx="0.01" ixy="0" ixz="0" iyy="0.01" iyz="0" izz="0.01"/>
+    </inertial>
+  </link>
+  <joint name="meca_axis_6_to_ee_sphere" type="fixed">
+    <origin xyz="0 0 0" rpy="0 0 0" />
+    <parent link="meca_axis_6_link_B" />
+    <child link="ee_sphere" />
+  </joint>
   <!-- BUFFERS -->
   <joint name="world_to_buffer" type="fixed">

Commit message: reduce ee_sphere collision radius to 0.05 m

File: mecademic_description/urdf/meca_500_r3.urdf.xacro (robot description, xacro)
@@ -458,11 +458,11 @@
       <origin xyz="0 0 0" rpy="0 0 0" />
       <geometry>
-        <sphere radius="0.06" />
-      </geometry>
-    </visual>
-    <collision>
-      <origin xyz="0 0 0" rpy="0 0 0" />
-      <geometry>
-        <sphere radius="0.06" />
+        <sphere radius="0.05" />
+      </geometry>
+    </visual>
+    <collision>
+      <origin xyz="0 0 0" rpy="0 0 0" />
+      <geometry>
+        <sphere radius="0.05" />
       </geometry>
     </collision>

File: mecademic_description/urdf/meca_500_r3_capsule.urdf.xacro (robot description, xacro)
@@ -542,11 +542,11 @@
       <origin xyz="0 0 0" rpy="0 0 0" />
       <geometry>
-        <sphere radius="0.06" />
-      </geometry>
-    </visual>
-    <collision>
-      <origin xyz="0 0 0" rpy="0 0 0" />
-      <geometry>
-        <sphere radius="0.06" />
+        <sphere radius="0.05" />
+      </geometry>
+    </visual>
+    <collision>
+      <origin xyz="0 0 0" rpy="0 0 0" />
+      <geometry>
+        <sphere radius="0.05" />
       </geometry>
     </collision>

Commit message: WIP: turn last link of 360 and joint limits accordingly

File: mecademic_description/urdf/meca_500_r3.urdf.xacro (robot description, xacro)
@@ -448,10 +448,11 @@
   </link>
   <joint name="meca_axis_6_joint_B" type="revolute">
-    <origin xyz="0.07 0 0" rpy="0 0 0" />
+    <origin xyz="0.07 0 0" rpy="3.141 0 0" />
     <parent link="meca_axis_5_link_B" />
     <child link="meca_axis_6_link_B" />
     <axis xyz="1 0 0" />
-    <limit effort="10.0" velocity="8.72665" lower="-4.0" upper="4.0" />
-  </joint>
+    <limit effort="10.0" velocity="8.72665" lower="-0.859" upper="7.141" />
+  </joint>
+  <!-- we turned last link by 360 because of cable problems. still to be confirmed -->
   <link name="ee_sphere">
     <visual>

File: mecademic_description/urdf/meca_500_r3_capsule.urdf.xacro (robot description, xacro)
@@ -532,9 +532,9 @@
   </link>
   <joint name="meca_axis_6_joint_B" type="revolute">
-    <origin xyz="0.07 0 0" rpy="0 0 0" />
+    <origin xyz="0.07 0 0" rpy="3.141 0 0" />
     <parent link="meca_axis_5_link_B" />
     <child link="meca_axis_6_link_B" />
     <axis xyz="1 0 0" />
-    <limit effort="10.0" lower="-4.0" upper="4.0" velocity="8.72665"/>
+    <limit effort="10.0" velocity="8.72665" lower="-0.859" upper="7.141" />
   </joint>
   <link name="ee_sphere">

Commit message: WIP: turn last link of meca_B of 360 and joint limits accordingly

File: mecademic_description/urdf/meca_500_r3.urdf.xacro (robot description, xacro)
@@ -628,10 +628,11 @@
   </link>
   <joint name="meca_axis_6_joint_B" type="revolute">
-    <origin xyz="0.07 0 0" rpy="0 0 0" />
+    <origin xyz="0.07 0 0" rpy="3.141 0 0" />
     <parent link="meca_axis_5_link_B" />
     <child link="meca_axis_6_link_B" />
     <axis xyz="1 0 0" />
-    <limit effort="10.0" velocity="8.72665" lower="-4.0" upper="4.0" />
-  </joint>
+    <limit effort="10.0" velocity="8.72665" lower="-0.859" upper="7.141" />
+  </joint>
+  <!-- we turned last link by 360 because of cable problems. still to be confirmed -->
   <!-- BUFFERS -->
   <joint name="world_to_buffer" type="fixed">

File: mecademic_description/urdf/meca_500_r3_capsule.urdf.xacro (robot description, xacro)
@@ -796,9 +796,9 @@
   </link>
   <joint name="meca_axis_6_joint_B" type="revolute">
-    <origin xyz="0.07 0 0" rpy="0 0 0" />
+    <origin xyz="0.07 0 0" rpy="3.141 0 0" />
     <parent link="meca_axis_5_link_B" />
     <child link="meca_axis_6_link_B" />
     <axis xyz="1 0 0" />
-    <limit effort="10.0" lower="-4.0" upper="4.0" velocity="8.72665"/>
+    <limit effort="10.0" velocity="8.72665" lower="-0.859" upper="7.141" />
   </joint>
   <!-- BUFFERS -->

Commit message: update urdf according to CAD

File: mecademic_description/urdf/meca_500_r3.urdf.xacro (robot description, xacro)
@@ -29,5 +29,5 @@
     <parent link="world"/>
     <child link="base_link_A"/>
-    <origin rpy="0 0 0" xyz="0.509 0.12 0.0"/>
+    <origin rpy="0 0 0" xyz="0.600 0.153 0.050"/>
   </joint>
   <gazebo>
@@ -146,5 +146,5 @@
     <parent link="L_1_A"/>
     <child link="meca_base_link_A"/>
-    <origin rpy="0 1.571 1.571" xyz="0.0 0 0.05"/>
+    <origin rpy="0 1.571 1.571" xyz="0.0 0.014 0.0744"/>
   </joint>
     <!-- Base link is the center of the robot's bottom plate -->
@@ -325,5 +325,5 @@
 <!-- 2nd ROBOT -->
   <joint name="world_to_base_B" type="fixed">
-      <origin xyz="0.456 0.572 0" rpy="0 0 -1.571"/>
+      <origin xyz="0.4521 0.9847 0.050" rpy="0 0 -1.571"/>
       <parent link="world"/>
       <child link="base_link_B"/>
@@ -349,34 +349,8 @@
     </inertial>
   </link>
-  <joint name="base_to_platform" type="fixed">
+  <joint name="fixed_rotary_table" type="fixed">
     <parent link="base_link_B"/>
-    <child link="platform"/>
-    <origin rpy="0.0 -0.0 0" xyz="0.0 0.0 0.0"/>
-  </joint>
-  <link name="platform">
-    <visual>
-      <geometry>
-        <box size="0.450 0.167 0.03"/>
-      </geometry>
-      <material name="blue">
-        <color rgba="0 0 .8 1"/>
-      </material>
-      <origin xyz="0 0 0.015" rpy="0 0 1.571" />
-    </visual>
-    <collision>
-      <origin xyz="0 0 0" rpy="1.571 0 0" />
-      <geometry>
-        <cylinder length="0.450" radius="0.15"/>
-      </geometry>
-    </collision>
-    <inertial>
-      <mass value="0.1"/>
-      <inertia ixx="1.0e-03" ixy="0.0" ixz="0.0" iyy="1.0e-03" iyz="0.0" izz="1.0e-03"/>
-    </inertial>
-  </link>
-  <joint name="fixed_rotary_table" type="fixed">
-    <parent link="platform"/>
     <child link="rotary_table_stator"/>
-    <origin rpy="0.0 -0.0 0.0" xyz="0.0 0.0 0.03"/>
+    <origin rpy="0.0 -0.0 0.0" xyz="0.0 0.0 0.0"/>
   </joint>
   <link name="rotary_table_stator">
@@ -457,5 +431,5 @@
     <parent link="L_1_B"/>
     <child link="meca_base_link_B"/>
-    <origin rpy="0 1.571 0" xyz="0.095 0.0 0.0645"/>
+    <origin rpy="0 1.571 0" xyz="0.0475 0.0 0.0575"/>
   </joint>
     <!-- Base link is the center of the robot's bottom plate -->
@@ -637,5 +611,5 @@
   <!-- BUFFERS -->
   <joint name="world_to_buffer" type="fixed">
-    <origin xyz="0.2 0.35 0.05" rpy="0 0 0"/>
+     <origin xyz="0 0.585 0.15" rpy="0 0 0"/>
     <parent link="world"/>
     <child link="buffer_base_link"/>
@@ -643,5 +617,5 @@
   <link name="buffer_base_link"/>
   <joint name="buffer_base_to_1" type="fixed">
-    <origin xyz="0 0 0" rpy="0 0 0"/>
+    <origin xyz="0.550 0 0" rpy="0 0 0"/>
     <parent link="buffer_base_link"/>
     <child link="buffer_1"/>
@@ -649,5 +623,5 @@
   <link name="buffer_1"/>
   <joint name="buffer_base_to_2" type="fixed">
-        <origin xyz="0.3 0.0 0" rpy="0 0 0"/>
+        <origin xyz="0.675 0.0 0" rpy="0 0 0"/>
         <parent link="buffer_base_link"/>
         <child link="buffer_2"/>
@@ -656,5 +630,5 @@
   <!-- CANDY MILL -->
   <joint name="world_to_mill" type="fixed">
-    <origin xyz="0.65 0.85 0.05" rpy="0 0 0"/>
+    <origin xyz="0.8154 1.0473 0.0" rpy="0 0 0"/>
     <parent link="world"/>
     <child link="mill_base_link"/>
@@ -662,5 +636,5 @@
   <link name="mill_base_link"/>
   <joint name="mill_base_to_stick" type="fixed">
-    <origin xyz="0.0 0 0.2" rpy="0 0 0"/>
+    <origin xyz="0.0 0 0.3068" rpy="0 0 0"/>
     <parent link="mill_base_link"/>
     <child link="mill_stick"/>
@@ -669,5 +643,5 @@
   <!-- SLIDERS -->
   <joint name="world_to_slider" type="fixed">
-    <origin xyz="0 0.3 0.05" rpy="0 0 0"/>
+    <origin xyz="0 0.585 0.0" rpy="0 0 0"/>
     <parent link="world"/>
     <child link="slider_base_link"/>
@@ -675,5 +649,5 @@
   <link name="slider_base_link"/>
   <joint name="slider_base_to_empty" type="fixed">
-    <origin xyz="0 0 0" rpy="0 0 0"/>
+    <origin xyz="0.397 0 0.194" rpy="0 0.1745 0"/>
     <parent link="slider_base_link"/>
     <child link="empty_container"/>
@@ -681,5 +655,5 @@
   <link name="empty_container"/>
   <joint name="sliders_base_to_lid" type="fixed">
-        <origin xyz="0 0.05 0" rpy="0 0 0"/>
+        <origin xyz="0.322 0 0.319" rpy="0 0.1745 0"/>
         <parent link="slider_base_link"/>
         <child link="lid"/>
@@ -687,5 +661,5 @@
   <link name="lid"/>
   <joint name="sliders_base_to_full" type="fixed">
-        <origin xyz="0.6 0 0" rpy="0 0 0"/>
+        <origin xyz="0.809 0 0.295" rpy="0 0.1745 0"/>
         <parent link="slider_base_link"/>
         <child link="full_container"/>
@@ -694,5 +668,5 @@
   <!-- FLOOR -->
   <joint name="world_to_floor" type="fixed">
-    <origin xyz="0 0 0" rpy="0 0 0"/>
+    <origin xyz="0 0 0.050" rpy="0 0 0"/>
     <parent link="world"/>
     <child link="floor_link"/>

File: mecademic_description/urdf/meca_500_r3_capsule.urdf.xacro (robot description, xacro)
@@ -29,5 +29,5 @@
     <parent link="world"/>
     <child link="base_link_A"/>
-    <origin rpy="0 0 0" xyz="0.509 0.12 0.0"/>
+    <origin rpy="0 0 0" xyz="0.600 0.153 0.050"/>
   </joint>
   <gazebo>
@@ -146,5 +146,5 @@
     <parent link="L_1_A"/>
     <child link="meca_base_link_A"/>
-    <origin rpy="0 1.571 1.571" xyz="0.0 0 0.05"/>
+    <origin rpy="0 1.571 1.571" xyz="0.0 0.014 0.0744"/>
   </joint>
     <!-- Base link is the center of the robot's bottom plate -->
@@ -409,5 +409,5 @@
 <!-- 2nd ROBOT -->
   <joint name="world_to_base_B" type="fixed">
-      <origin xyz="0.456 0.572 0" rpy="0 0 -1.571"/>
+      <origin xyz="0.4521 0.9847 0.050" rpy="0 0 -1.571"/>
       <parent link="world"/>
       <child link="base_link_B"/>
@@ -433,34 +433,8 @@
     </inertial>
   </link>
-  <joint name="base_to_platform" type="fixed">
+  <joint name="fixed_rotary_table" type="fixed">
     <parent link="base_link_B"/>
-    <child link="platform"/>
-    <origin rpy="0.0 -0.0 0" xyz="0.0 0.0 0.0"/>
-  </joint>
-  <link name="platform">
-    <visual>
-      <geometry>
-        <box size="0.450 0.167 0.03"/>
-      </geometry>
-      <material name="blue">
-        <color rgba="0 0 .8 1"/>
-      </material>
-      <origin xyz="0 0 0.015" rpy="0 0 1.571" />
-    </visual>
-    <collision>
-      <origin xyz="0 0 0" rpy="1.571 0 0" />
-      <geometry>
-        <cylinder length="0.450" radius="0.15"/>
-      </geometry>
-    </collision>
-    <inertial>
-      <mass value="0.1"/>
-      <inertia ixx="1.0e-03" ixy="0.0" ixz="0.0" iyy="1.0e-03" iyz="0.0" izz="1.0e-03"/>
-    </inertial>
-  </link>
-  <joint name="fixed_rotary_table" type="fixed">
-    <parent link="platform"/>
     <child link="rotary_table_stator"/>
-    <origin rpy="0.0 -0.0 0.0" xyz="0.0 0.0 0.03"/>
+    <origin rpy="0.0 -0.0 0.0" xyz="0.0 0.0 0.0"/>
   </joint>
   <link name="rotary_table_stator">
@@ -541,5 +515,5 @@
     <parent link="L_1_B"/>
     <child link="meca_base_link_B"/>
-    <origin rpy="0 1.571 0" xyz="0.095 0.0 0.0645"/>
+    <origin rpy="0 1.571 0" xyz="0.0475 0.0 0.0575"/>
   </joint>
     <!-- Base link is the center of the robot's bottom plate -->
@@ -804,5 +778,5 @@
   <!-- BUFFERS -->
   <joint name="world_to_buffer" type="fixed">
-    <origin xyz="0.2 0.35 0.05" rpy="0 0 0"/>
+     <origin xyz="0 0.585 0.15" rpy="0 0 0"/>
     <parent link="world"/>
     <child link="buffer_base_link"/>
@@ -810,5 +784,5 @@
   <link name="buffer_base_link"/>
   <joint name="buffer_base_to_1" type="fixed">
-    <origin xyz="0 0 0" rpy="0 0 0"/>
+    <origin xyz="0.550 0 0" rpy="0 0 0"/>
     <parent link="buffer_base_link"/>
     <child link="buffer_1"/>
@@ -816,5 +790,5 @@
   <link name="buffer_1"/>
   <joint name="buffer_base_to_2" type="fixed">
-        <origin xyz="0.3 0.0 0" rpy="0 0 0"/>
+        <origin xyz="0.675 0.0 0" rpy="0 0 0"/>
         <parent link="buffer_base_link"/>
         <child link="buffer_2"/>
@@ -823,5 +797,5 @@
   <!-- CANDY MILL -->
   <joint name="world_to_mill" type="fixed">
-    <origin xyz="0.65 0.85 0.05" rpy="0 0 0"/>
+    <origin xyz="0.8154 1.0473 0.0" rpy="0 0 0"/>
     <parent link="world"/>
     <child link="mill_base_link"/>
@@ -829,5 +803,5 @@
   <link name="mill_base_link"/>
   <joint name="mill_base_to_stick" type="fixed">
-    <origin xyz="0.0 0 0.2" rpy="0 0 0"/>
+    <origin xyz="0.0 0 0.3068" rpy="0 0 0"/>
     <parent link="mill_base_link"/>
     <child link="mill_stick"/>
@@ -836,5 +810,5 @@
   <!-- SLIDERS -->
   <joint name="world_to_slider" type="fixed">
-    <origin xyz="0 0.3 0.05" rpy="0 0 0"/>
+    <origin xyz="0 0.585 0.05" rpy="0 0 0"/>
     <parent link="world"/>
     <child link="slider_base_link"/>
@@ -842,5 +816,5 @@
   <link name="slider_base_link"/>
   <joint name="slider_base_to_empty" type="fixed">
-    <origin xyz="0 0 0" rpy="0 0 0"/>
+    <origin xyz="0.397 0 0.194" rpy="0 0.1745 0"/>
     <parent link="slider_base_link"/>
     <child link="empty_container"/>
@@ -848,5 +822,5 @@
   <link name="empty_container"/>
   <joint name="sliders_base_to_lid" type="fixed">
-        <origin xyz="0 0.05 0" rpy="0 0 0"/>
+        <origin xyz="0.322 0 0.319" rpy="0 0.1745 0"/>
         <parent link="slider_base_link"/>
         <child link="lid"/>
@@ -854,5 +828,5 @@
   <link name="lid"/>
   <joint name="sliders_base_to_full" type="fixed">
-        <origin xyz="0.6 0 0" rpy="0 0 0"/>
+       <origin xyz="0.809 0 0.295" rpy="0 0.1745 0"/>
         <parent link="slider_base_link"/>
         <child link="full_container"/>
@@ -861,5 +835,5 @@
   <!-- FLOOR -->
   <joint name="world_to_floor" type="fixed">
-    <origin xyz="0 0 0" rpy="0 0 0"/>
+    <origin xyz="0 0 0.050" rpy="0 0 0"/>
     <parent link="world"/>
     <child link="floor_link"/>

Commit message: add end effecctors links

File: mecademic_description/urdf/meca_500_r3.urdf.xacro (robot description, xacro)
@@ -323,4 +323,16 @@
     <limit effort="10.0" velocity="8.72665" lower="-4.0" upper="4.0" />
   </joint>
+  <!-- End Effector -->
+  <link name="ee_link_A">
+    <inertial>
+      <mass value="1"/>
+      <inertia ixx="0.01" ixy="0" ixz="0" iyy="0.01" iyz="0" izz="0.01"/>
+    </inertial>
+  </link>
+  <joint name="meca_to_ee_A_joint" type="fixed">
+    <origin xyz="0.015 0.0087 -0.0323" rpy="0 0 0" />
+    <parent link="meca_axis_6_link_A" />
+    <child link="ee_link_A" />
+  </joint>
 <!-- 2nd ROBOT -->
   <joint name="world_to_base_B" type="fixed">
@@ -609,4 +621,16 @@
   </joint>
   <!-- we turned last link by 360 because of cable problems. still to be confirmed -->
+  <!-- End Effector -->
+  <link name="ee_link_B">
+    <inertial>
+      <mass value="1"/>
+      <inertia ixx="0.01" ixy="0" ixz="0" iyy="0.01" iyz="0" izz="0.01"/>
+    </inertial>
+  </link>
+  <joint name="meca_to_ee_B_joint" type="fixed">
+    <origin xyz="0.0294 0 -0.01855" rpy="0 0 0" />
+    <parent link="meca_axis_6_link_B" />
+    <child link="ee_link_B" />
+  </joint>
   <!-- BUFFERS -->
   <joint name="world_to_buffer" type="fixed">

File: mecademic_description/urdf/meca_500_r3_capsule.urdf.xacro (robot description, xacro)
@@ -407,4 +407,16 @@
     <limit effort="10.0" lower="-4.0" upper="4.0" velocity="8.72665"/>
   </joint>
+  <!-- End Effector -->
+  <link name="ee_link_A">
+    <inertial>
+      <mass value="1"/>
+      <inertia ixx="0.01" ixy="0" ixz="0" iyy="0.01" iyz="0" izz="0.01"/>
+    </inertial>
+  </link>
+  <joint name="meca_to_ee_A_joint" type="fixed">
+    <origin xyz="0.015 0.0087 -0.0323" rpy="0 0 0" />
+    <parent link="meca_axis_6_link_A" />
+    <child link="ee_link_A" />
+  </joint>
 <!-- 2nd ROBOT -->
   <joint name="world_to_base_B" type="fixed">
@@ -776,4 +788,16 @@
     <limit effort="10.0" velocity="8.72665" lower="-0.859" upper="7.141" />
   </joint>
+  <!-- End Effector -->
+  <link name="ee_link_B">
+    <inertial>
+      <mass value="1"/>
+      <inertia ixx="0.01" ixy="0" ixz="0" iyy="0.01" iyz="0" izz="0.01"/>
+    </inertial>
+  </link>
+  <joint name="meca_to_ee_B_joint" type="fixed">
+    <origin xyz="0.0294 0 -0.01855" rpy="0 0 0" />
+    <parent link="meca_axis_6_link_B" />
+    <child link="ee_link_B" />
+  </joint>
   <!-- BUFFERS -->
   <joint name="world_to_buffer" type="fixed">
