Commit message: add gripper meshes

File: mecademic_description/urdf/meca_500_r3.urdf.xacro (robot description, xacro)
@@ -323,4 +323,28 @@
     <limit effort="10.0" velocity="8.72665" lower="-4.0" upper="4.0" />
   </joint>
+  <!-- gripper -->
+  <link name="vacuum_gripper">
+    <visual>
+      <origin xyz="0 0 0" rpy="0 0 0" />
+      <geometry>
+        <mesh filename="package://mecademic_description/meshes/pneumatic_tube_holder_mesh_v2.stl" scale="0.001 0.001 0.001"/>
+      </geometry>
+    </visual>
+    <collision>
+      <origin xyz="0 0 0" rpy="0 0 0" />
+      <geometry>
+        <mesh filename="package://mecademic_description/meshes/pneumatic_tube_holder_mesh_v2.stl" scale="0.001 0.001 0.001"/>
+      </geometry>
+    </collision>
+    <inertial>
+      <mass value="1"/>
+      <inertia ixx="0.01" ixy="0" ixz="0" iyy="0.01" iyz="0" izz="0.01"/>
+    </inertial>
+  </link>
+  <joint name="meca_to_gripper_A_joint" type="fixed">
+    <origin xyz="0 0 0" rpy="0 0 0" />
+    <parent link="meca_axis_6_link_A" />
+    <child link="vacuum_gripper" />
+  </joint>
   <!-- End Effector -->
   <link name="ee_link_A">
@@ -330,7 +354,7 @@
     </inertial>
   </link>
-  <joint name="meca_to_ee_A_joint" type="fixed">
+  <joint name="vacum_gripper_to_ee_A_joint" type="fixed">
     <origin xyz="0.015 0.0087 -0.0323" rpy="0 0 0" />
-    <parent link="meca_axis_6_link_A" />
+    <parent link="vacuum_gripper" />
     <child link="ee_link_A" />
   </joint>
@@ -621,4 +645,29 @@
   </joint>
   <!-- we turned last link by 360 because of cable problems. still to be confirmed -->
+  <!-- Gripper -->
+  <link name="two_finger_gripper">
+    <visual>
+      <origin xyz="0 0 0" rpy="0 0 0" />
+      <geometry>
+        <mesh filename="package://mecademic_description/meshes/gripper_finger_mesh_no_cable_metersv2.stl" />
+      </geometry>
+    </visual>
+    <collision>
+      <origin xyz="0 0 0" rpy="0 0 0" />
+      <geometry>
+        <mesh filename="package://mecademic_description/meshes/gripper_finger_mesh_no_cable_metersv2.stl" />
+      </geometry>
+    </collision>
+    <inertial>
+      <mass value="1"/>
+      <inertia ixx="0.01" ixy="0" ixz="0" iyy="0.01" iyz="0" izz="0.01"/>
+    </inertial>
+  </link>
+  <joint name="meca_to_gripper_B_joint" type="fixed">
+    <origin xyz="0 0 0" rpy=" 0 0 0" />
+    <parent link="meca_axis_6_link_B" />
+    <child link="two_finger_gripper" />
+  </joint>
+  <!-- we turned last link by 360 because of cable problems. still to be confirmed -->
   <!-- End Effector -->
   <link name="ee_link_B">
@@ -629,8 +678,13 @@
   </link>
   <joint name="meca_to_ee_B_joint" type="fixed">
+    <origin xyz="0.0379 0 0" rpy="0 0 0" />
+    <parent link="two_finger_gripper" />
+    <child link="ee_link_B" />
+  </joint>
+  <!-- <joint name="meca_to_ee_B_joint" type="fixed">
     <origin xyz="0.0294 0 -0.01855" rpy="0 0 0" />
-    <parent link="meca_axis_6_link_B" />
+    <parent link="two_finger_gripper" />
     <child link="ee_link_B" />
-  </joint>
+  </joint> -->
   <!-- BUFFERS -->
   <joint name="world_to_buffer" type="fixed">

File: mecademic_description/urdf/meca_500_r3_capsule.urdf.xacro (robot description, xacro)
@@ -407,4 +407,28 @@
     <limit effort="10.0" lower="-4.0" upper="4.0" velocity="8.72665"/>
   </joint>
+    <!-- gripper -->
+  <link name="vacuum_gripper">
+    <visual>
+      <origin xyz="0 0 0" rpy="0 0 0" />
+      <geometry>
+        <mesh filename="package://mecademic_description/meshes/pneumatic_tube_holder_mesh_v2.stl" scale="0.001 0.001 0.001"/>
+      </geometry>
+    </visual>
+    <collision>
+      <origin xyz="0 0 0" rpy="0 0 0" />
+      <geometry>
+        <mesh filename="package://mecademic_description/meshes/pneumatic_tube_holder_mesh_v2.stl" scale="0.001 0.001 0.001"/>
+      </geometry>
+    </collision>
+    <inertial>
+      <mass value="1"/>
+      <inertia ixx="0.01" ixy="0" ixz="0" iyy="0.01" iyz="0" izz="0.01"/>
+    </inertial>
+  </link>
+  <joint name="meca_to_gripper_A_joint" type="fixed">
+    <origin xyz="0 0 0" rpy="0 0 0" />
+    <parent link="meca_axis_6_link_A" />
+    <child link="vacuum_gripper" />
+  </joint>
   <!-- End Effector -->
   <link name="ee_link_A">
@@ -414,7 +438,7 @@
     </inertial>
   </link>
-  <joint name="meca_to_ee_A_joint" type="fixed">
+  <joint name="vacum_gripper_to_ee_A_joint" type="fixed">
     <origin xyz="0.015 0.0087 -0.0323" rpy="0 0 0" />
-    <parent link="meca_axis_6_link_A" />
+    <parent link="vacuum_gripper" />
     <child link="ee_link_A" />
   </joint>
@@ -788,4 +812,29 @@
     <limit effort="10.0" velocity="8.72665" lower="-0.859" upper="7.141" />
   </joint>
+  <!-- Gripper -->
+  <link name="two_finger_gripper">
+    <visual>
+      <origin xyz="0 0 0" rpy="0 0 0" />
+      <geometry>
+        <mesh filename="package://mecademic_description/meshes/gripper_finger_mesh_no_cable_metersv2.stl" />
+      </geometry>
+    </visual>
+    <collision>
+      <origin xyz="0 0 0" rpy="0 0 0" />
+      <geometry>
+        <mesh filename="package://mecademic_description/meshes/gripper_finger_mesh_no_cable_metersv2.stl" />
+      </geometry>
+    </collision>
+    <inertial>
+      <mass value="1"/>
+      <inertia ixx="0.01" ixy="0" ixz="0" iyy="0.01" iyz="0" izz="0.01"/>
+    </inertial>
+  </link>
+  <joint name="meca_to_gripper_B_joint" type="fixed">
+    <origin xyz="0 0 0" rpy=" 0 0 0" />
+    <parent link="meca_axis_6_link_B" />
+    <child link="two_finger_gripper" />
+  </joint>
+  <!-- we turned last link by 360 because of cable problems. still to be confirmed -->
   <!-- End Effector -->
   <link name="ee_link_B">
@@ -796,8 +845,13 @@
   </link>
   <joint name="meca_to_ee_B_joint" type="fixed">
+    <origin xyz="0.0379 0 0" rpy="0 0 0" />
+    <parent link="two_finger_gripper" />
+    <child link="ee_link_B" />
+  </joint>
+  <!-- <joint name="meca_to_ee_B_joint" type="fixed">
     <origin xyz="0.0294 0 -0.01855" rpy="0 0 0" />
-    <parent link="meca_axis_6_link_B" />
+    <parent link="two_finger_gripper" />
     <child link="ee_link_B" />
-  </joint>
+  </joint> -->
   <!-- BUFFERS -->
   <joint name="world_to_buffer" type="fixed">

Commit message: update urdf buffer and mill  frames

File: mecademic_description/urdf/meca_500_r3.urdf.xacro (robot description, xacro)
@@ -689,5 +689,5 @@
   <!-- BUFFERS -->
   <joint name="world_to_buffer" type="fixed">
-     <origin xyz="0 0.585 0.15" rpy="0 0 0"/>
+     <origin xyz="0 0.51 0.2" rpy="0 0 0"/>
     <parent link="world"/>
     <child link="buffer_base_link"/>
@@ -695,5 +695,5 @@
   <link name="buffer_base_link"/>
   <joint name="buffer_base_to_1" type="fixed">
-    <origin xyz="0.550 0 0" rpy="0 0 0"/>
+    <origin xyz="0.525 0 0" rpy="0 0 0"/>
     <parent link="buffer_base_link"/>
     <child link="buffer_1"/>
@@ -701,5 +701,5 @@
   <link name="buffer_1"/>
   <joint name="buffer_base_to_2" type="fixed">
-        <origin xyz="0.675 0.0 0" rpy="0 0 0"/>
+        <origin xyz="0.650 0.0 0" rpy="0 0 0"/>
         <parent link="buffer_base_link"/>
         <child link="buffer_2"/>
@@ -708,5 +708,5 @@
   <!-- CANDY MILL -->
   <joint name="world_to_mill" type="fixed">
-    <origin xyz="0.8154 1.0473 0.0" rpy="0 0 0"/>
+    <origin xyz="0.8154 0.8 0.0" rpy="0 0 0"/>
     <parent link="world"/>
     <child link="mill_base_link"/>
@@ -719,4 +719,10 @@
   </joint>
   <link name="mill_stick"/>
+  <joint name="mill_base_to_buffer" type="fixed">
+    <origin xyz="0.0 0 0.1" rpy="0 0 0"/>
+    <parent link="mill_base_link"/>
+    <child link="mill_buffer"/>
+  </joint>
+  <link name="mill_buffer"/>
   <!-- SLIDERS -->
   <joint name="world_to_slider" type="fixed">

File: mecademic_description/urdf/meca_500_r3_capsule.urdf.xacro (robot description, xacro)
@@ -896,5 +896,5 @@
   </joint>
   <joint name="world_to_buffer" type="fixed">
-    <origin rpy="0.0 0.0 0.0" xyz="0.0 0.585 0.15"/>
+     <origin xyz="0 0.51 0.2" rpy="0 0 0"/>
     <parent link="world"/>
     <child link="buffer_base_link"/>
@@ -902,5 +902,5 @@
   <link name="buffer_base_link"/>
   <joint name="buffer_base_to_1" type="fixed">
-    <origin rpy="0.0 0.0 0.0" xyz="0.55 0.0 0.0"/>
+    <origin xyz="0.525 0 0" rpy="0 0 0"/>
     <parent link="buffer_base_link"/>
     <child link="buffer_1"/>
@@ -908,11 +908,11 @@
   <link name="buffer_1"/>
   <joint name="buffer_base_to_2" type="fixed">
-    <origin rpy="0.0 0.0 0.0" xyz="0.675 0.0 0.0"/>
-    <parent link="buffer_base_link"/>
-    <child link="buffer_2"/>
-  </joint>
+        <origin xyz="0.650 0.0 0" rpy="0 0 0"/>
+        <parent link="buffer_base_link"/>
+        <child link="buffer_2"/>
+      </joint>
   <link name="buffer_2"/>
   <joint name="world_to_mill" type="fixed">
-    <origin rpy="0.0 0.0 0.0" xyz="0.8154 1.0473 0.0"/>
+    <origin xyz="0.8154 0.8 0.0" rpy="0 0 0"/>
     <parent link="world"/>
     <child link="mill_base_link"/>
@@ -925,4 +925,11 @@
   </joint>
   <link name="mill_stick"/>
+  <joint name="mill_base_to_buffer" type="fixed">
+    <origin xyz="0.0 0 0.1" rpy="0 0 0"/>
+    <parent link="mill_base_link"/>
+    <child link="mill_buffer"/>
+  </joint>
+  <link name="mill_buffer"/>
+  <!-- SLIDERS -->
   <joint name="world_to_slider" type="fixed">
     <origin rpy="0.0 0.0 0.0" xyz="0.0 0.585 0.0"/>

Commit message: remove floor collision

File: mecademic_description/urdf/meca_500_r3.urdf.xacro (robot description, xacro)
@@ -751,5 +751,5 @@
   <link name="full_container"/>
   <!-- FLOOR -->
-  <joint name="world_to_floor" type="fixed">
+  <!-- <joint name="world_to_floor" type="fixed">
     <origin xyz="0 0 0.050" rpy="0 0 0"/>
     <parent link="world"/>
@@ -772,4 +772,4 @@
       </geometry>
     </collision>
-  </link>
+  </link> -->
 </robot>

File: mecademic_description/urdf/meca_500_r3_capsule.urdf.xacro (robot description, xacro)
@@ -956,5 +956,5 @@
   </joint>
   <link name="full_container"/>
-  <joint name="world_to_floor" type="fixed">
+  <!-- <joint name="world_to_floor" type="fixed">
     <origin rpy="0.0 0.0 0.0" xyz="0.0 0.0 0.05"/>
     <parent link="world"/>
@@ -977,4 +977,4 @@
       </geometry>
     </collision>
-  </link>
+  </link> -->
 </robot>

Commit message: update postural (homing) and urdf (better inverse kinematics)
- reduced range and predictable motion of gripper cable

File: mecademic_description/urdf/meca_500_r3.urdf.xacro (robot description, xacro)
@@ -29,5 +29,5 @@
     <parent link="world"/>
     <child link="base_link_A"/>
-    <origin rpy="0 0 0" xyz="0.600 0.153 0.050"/>
+    <origin rpy="0 0 0" xyz="0.600 0.16 0.050"/>
   </joint>
   <gazebo>
@@ -689,5 +689,5 @@
   <!-- BUFFERS -->
   <joint name="world_to_buffer" type="fixed">
-     <origin xyz="0 0.51 0.2" rpy="0 0 0"/>
+     <origin xyz="0 0.585 0.2" rpy="0 0 0"/>
     <parent link="world"/>
     <child link="buffer_base_link"/>
@@ -720,5 +720,5 @@
   <link name="mill_stick"/>
   <joint name="mill_base_to_buffer" type="fixed">
-    <origin xyz="0.0 0 0.1" rpy="0 0 0"/>
+    <origin xyz="0.0 0 0.15" rpy="0 0 0"/>
     <parent link="mill_base_link"/>
     <child link="mill_buffer"/>

File: mecademic_description/urdf/meca_500_r3_capsule.urdf.xacro (robot description, xacro)
@@ -27,5 +27,5 @@
   <link name="world"/>
   <joint name="world_to_base_A" type="fixed">
-    <origin rpy="0.0 0.0 0.0" xyz="0.6 0.153 0.05"/>
+    <origin rpy="0.0 0.0 0.0" xyz="0.6 0.16 0.05"/>
     <parent link="world"/>
     <child link="base_link_A"/>
@@ -896,5 +896,5 @@
   </joint>
   <joint name="world_to_buffer" type="fixed">
-     <origin xyz="0 0.51 0.2" rpy="0 0 0"/>
+     <origin xyz="0 0.585 0.2" rpy="0 0 0"/>
     <parent link="world"/>
     <child link="buffer_base_link"/>
@@ -926,5 +926,5 @@
   <link name="mill_stick"/>
   <joint name="mill_base_to_buffer" type="fixed">
-    <origin xyz="0.0 0 0.1" rpy="0 0 0"/>
+    <origin xyz="0.0 0 0.15" rpy="0 0 0"/>
     <parent link="mill_base_link"/>
     <child link="mill_buffer"/>

Commit message: update urdf with linear drive from CAD

File: mecademic_description/urdf/meca_500_r3.urdf.xacro (robot description, xacro)
@@ -29,5 +29,5 @@
     <parent link="world"/>
     <child link="base_link_A"/>
-    <origin rpy="0 0 0" xyz="0.600 0.16 0.050"/>
+    <origin rpy="0 0 0" xyz="0.110 0.083 0.050"/>
   </joint>
   <gazebo>
@@ -54,21 +54,21 @@
     <parent link="base_link_A"/>
     <child link="gear_box"/>
-    <origin xyz="0.431 0.0 0.05" rpy="0 0 1.571" />
+    <origin xyz="0.927 0.07 0.08" rpy="0 0 1.571" />
   </joint>
  <link name="gear_box">
     <visual>
       <geometry>
-        <cylinder length="0.366" radius="0.12"/>
+        <cylinder length="0.405" radius="0.065"/>
       </geometry>
       <material name="blue">
         <color rgba="0 0 .8 1"/>
       </material>
-      <origin xyz="0.183 0 0" rpy="0 1.571 0" />
-    </visual>
-    <collision>
-      <origin xyz="0.183 0 0" rpy="0 1.571 0" />
-      <geometry>
-        <cylinder length="0.366" radius="0.12" />
-      </geometry>
+      <origin xyz="0.2025 0 0.0" rpy="0 1.571 0" />
+    </visual>
+    <collision>
+      <geometry>
+        <cylinder length="0.405" radius="0.065"/>
+      </geometry>
+      <origin xyz="0.2025 0 0.0" rpy="0 1.571 0" />
     </collision>
     <inertial>
@@ -81,20 +81,17 @@
     <parent link="base_link_A"/>
     <child link="linear_motor_stator"/>
-    <origin xyz="0.0 0.0 0.05" rpy="0 0 0" />
+    <origin xyz="0.0 0.0 0.0" rpy="0 0 0" />
   </joint>
   <link name="linear_motor_stator">
     <visual>
-      <geometry>
-        <box size="0.98 0.12 0.1"/>
-      </geometry>
-      <material name="blue">
-        <color rgba="0 0 .8 1"/>
-      </material>
-      <origin xyz="0 0 0" rpy="0 0 0" />
-    </visual>
-    <collision>
-      <origin xyz="0 0 0.05" rpy="0 1.571 0" />
-      <geometry>
-        <cylinder length="0.98" radius="0.12" />
+      <origin xyz="0 0 0" rpy="0 0 0" />
+      <geometry>
+        <mesh filename="package://mecademic_description/meshes/linear_guide_base_meters.stl" />
+      </geometry>
+    </visual>
+    <collision>
+      <origin xyz="0 0 0" rpy="0 0 0" />
+      <geometry>
+        <mesh filename="package://mecademic_description/meshes/linear_guide_base_meters.stl" />
       </geometry>
     </collision>
@@ -119,20 +116,17 @@
     <child link="L_1_A"/>
     <limit effort="100.0" lower="-0.002" upper="0.400" velocity="0.5"/>
-    <origin rpy="0 0 0" xyz="-0.26 0 0.09"/>
+    <origin rpy="0 0 0" xyz="0.262 0.06 0.102"/>
   </joint>
   <link name="L_1_A">
     <visual>
-      <geometry>
-        <box size="0.2 0.2 0.04"/>
-      </geometry>
-      <material name="blue">
-        <color rgba="0 0 .8 1"/>
-      </material>
-      <origin xyz="0 0 -0.02" rpy="0 0 0" />
-    </visual>
-    <collision>
-      <origin xyz="0 0 -0.02" rpy="0 0 0" />
-      <geometry>
-        <box size="0.2 0.2 0.04"/>
+      <origin xyz="0 0 0" rpy="0 0 0" />
+      <geometry>
+        <mesh filename="package://mecademic_description/meshes/linear_guide_mover_meters.stl" />
+      </geometry>
+    </visual>
+    <collision>
+      <origin xyz="0 0 0" rpy="0 0 0" />
+      <geometry>
+        <mesh filename="package://mecademic_description/meshes/linear_guide_mover_meters.stl" />
       </geometry>
     </collision>
@@ -143,8 +137,32 @@
     </inertial>
   </link>
-  <joint name="L_1_A_to_meca_base_link_A" type="fixed">
+  <joint name="L_1_A_to_stuff_on_top_A" type="fixed">
     <parent link="L_1_A"/>
+    <child link="stuff_on_top_A"/>
+    <origin rpy="0 0 0" xyz="0.0 0.0 0.0355"/>
+  </joint>
+  <link name="stuff_on_top_A">
+    <visual>
+      <origin xyz="0 0 0" rpy="0 0 0" />
+      <geometry>
+        <mesh filename="package://mecademic_description/meshes/pump_and_robot_mount_metres_lower_quality.stl" />
+      </geometry>
+    </visual>
+    <collision>
+      <origin xyz="0 0 0" rpy="0 0 0" />
+      <geometry>
+        <mesh filename="package://mecademic_description/meshes/pump_and_robot_mount_metres_lower_quality.stl" />
+      </geometry>
+    </collision>
+    <inertial>
+      <origin rpy="0 0 0" xyz="0.0 0.0 -0.024438213"/>
+      <mass value="0.42322395"/>
+      <inertia ixx="0.00063746146" ixy="1.1903424e-05" ixz="6.7230372e-07" iyy="0.00064218987" iyz="2.203073e-05" izz="0.001009674"/>
+    </inertial>
+  </link>
+  <joint name="stuff_on_top_A_to_meca_base_link_A" type="fixed">
+    <parent link="stuff_on_top_A"/>
     <child link="meca_base_link_A"/>
-    <origin rpy="0 1.571 1.571" xyz="0.0 0.014 0.0744"/>
+    <origin rpy="0 1.571 1.571" xyz="0.05 0.024 0.0705"/>
   </joint>
     <!-- Base link is the center of the robot's bottom plate -->
@@ -467,5 +485,5 @@
     <parent link="L_1_B"/>
     <child link="meca_base_link_B"/>
-    <origin rpy="0 1.571 0" xyz="0.0475 0.0 0.0575"/>
+    <origin rpy="0 1.571 0" xyz="0.0475 0.0 0.0645"/>
   </joint>
     <!-- Base link is the center of the robot's bottom plate -->
