Commit message: only rotary meca

File: mecademic_description/urdf/meca_500_r3.urdf.xacro (robot description, xacro)
@@ -25,338 +25,4 @@
   </material>
   <link name="world"/>
-<!-- 1st ROBOT -->
-  <joint name="world_to_base_A" type="fixed">
-    <parent link="world"/>
-    <child link="base_link_A"/>
-    <origin rpy="0 0 0" xyz="0.600 0.16 0.050"/>
-  </joint>
-  <gazebo>
-      <plugin filename="libxbot2_gz_joint_server.so" name="xbot2_gz_joint_server">
-          <pid>
-            <pid name="BL4104C_1" profile="medium_mot"/>
-            <pid name="meca_axis_1_joint_A" profile="small_mot"/>
-            <pid name="meca_axis_2_joint_A" profile="small_mot"/>
-            <pid name="meca_axis_3_joint_A" profile="small_mot"/>
-            <pid name="meca_axis_4_joint_A" profile="small_mot"/>
-            <pid name="meca_axis_5_joint_A" profile="small_mot"/>
-            <pid name="meca_axis_6_joint_A" profile="small_mot"/>
-          </pid>
-          <gain d="5" name="small_mot" p="100"/>
-      </plugin>
-    </gazebo>
-  <link name="base_link_A">
-    <inertial>
-      <mass value="0.1"/>
-      <inertia ixx="1.0e-03" ixy="0.0" ixz="0.0" iyy="1.0e-03" iyz="0.0" izz="1.0e-03"/>
-    </inertial>
-  </link>
-  <joint name="fixed_gear_box" type="fixed">
-    <parent link="base_link_A"/>
-    <child link="gear_box"/>
-    <origin xyz="0.431 0.0 0.05" rpy="0 0 1.571" />
-  </joint>
- <link name="gear_box">
-    <visual>
-      <geometry>
-        <cylinder length="0.366" radius="0.12"/>
-      </geometry>
-      <material name="blue">
-        <color rgba="0 0 .8 1"/>
-      </material>
-      <origin xyz="0.183 0 0" rpy="0 1.571 0" />
-    </visual>
-    <collision>
-      <origin xyz="0.183 0 0" rpy="0 1.571 0" />
-      <geometry>
-        <cylinder length="0.366" radius="0.12" />
-      </geometry>
-    </collision>
-    <inertial>
-      <origin rpy="0 0 0" xyz="0.0 0.0 0.10614489"/>
-      <mass value="2.0554934"/>
-      <inertia ixx="0.01068855" ixy="-1.14168e-05" ixz="2.71689e-06" iyy="0.010584907" iyz="8.76312e-05" izz="0.0032026258"/>
-    </inertial>
-  </link>
-  <joint name="fixed_linear_motor" type="fixed">
-    <parent link="base_link_A"/>
-    <child link="linear_motor_stator"/>
-    <origin xyz="0.0 0.0 0.05" rpy="0 0 0" />
-  </joint>
-  <link name="linear_motor_stator">
-    <visual>
-      <geometry>
-        <box size="0.98 0.12 0.1"/>
-      </geometry>
-      <material name="blue">
-        <color rgba="0 0 .8 1"/>
-      </material>
-      <origin xyz="0 0 0" rpy="0 0 0" />
-    </visual>
-    <collision>
-      <origin xyz="0 0 0.05" rpy="0 1.571 0" />
-      <geometry>
-        <cylinder length="0.98" radius="0.12" />
-      </geometry>
-    </collision>
-    <inertial>
-      <origin rpy="0 0 0" xyz="0.0 0.0 0.10614489"/>
-      <mass value="2.0554934"/>
-      <inertia ixx="0.01068855" ixy="-1.14168e-05" ixz="2.71689e-06" iyy="0.010584907" iyz="8.76312e-05" izz="0.0032026258"/>
-    </inertial>
-  </link>
-  <gazebo reference="linear_motor_stator">
-    <mu1>0.2</mu1>
-    <mu2>0.2</mu2>
-    <kp>1000000.0</kp>
-    <kd>1.0</kd>
-    <maxVel>0.0</maxVel>
-    <minDepth>0.0001</minDepth>
-    <material>Gazebo/Blue</material>
-  </gazebo>
-  <joint name="linear_motor" type="prismatic">
-    <axis xyz="1 0 0"/>
-    <parent link="linear_motor_stator"/>
-    <child link="L_1_A"/>
-    <limit effort="100.0" lower="-0.002" upper="0.400" velocity="0.5"/>
-    <origin rpy="0 0 0" xyz="-0.26 0 0.09"/>
-  </joint>
-  <link name="L_1_A">
-    <visual>
-      <geometry>
-        <box size="0.2 0.2 0.04"/>
-      </geometry>
-      <material name="blue">
-        <color rgba="0 0 .8 1"/>
-      </material>
-      <origin xyz="0 0 -0.02" rpy="0 0 0" />
-    </visual>
-    <collision>
-      <origin xyz="0 0 -0.02" rpy="0 0 0" />
-      <geometry>
-        <box size="0.2 0.2 0.04"/>
-      </geometry>
-    </collision>
-    <inertial>
-      <origin rpy="0 0 0" xyz="0.0 0.0 -0.024438213"/>
-      <mass value="0.42322395"/>
-      <inertia ixx="0.00063746146" ixy="1.1903424e-05" ixz="6.7230372e-07" iyy="0.00064218987" iyz="2.203073e-05" izz="0.001009674"/>
-    </inertial>
-  </link>
-  <joint name="L_1_A_to_meca_base_link_A" type="fixed">
-    <parent link="L_1_A"/>
-    <child link="meca_base_link_A"/>
-    <origin rpy="0 1.571 1.571" xyz="0.0 0.014 0.0744"/>
-  </joint>
-    <!-- Base link is the center of the robot's bottom plate -->
-  <link name="meca_base_link_A">
-    <visual>
-      <origin xyz="0 0 0" rpy="0 0 0" />
-      <geometry>
-        <mesh filename="package://mecademic_description/meshes/meca_500_r3_base.dae" />
-      </geometry>
-    </visual>
-    <collision>
-      <origin xyz="0 0 0" rpy="0 0 0" />
-      <geometry>
-        <mesh filename="package://mecademic_description/meshes/meca_500_r3_base_collision.stl" />
-      </geometry>
-    </collision>
-    <inertial>
-      <mass value="1"/>
-      <inertia ixx="0.01" ixy="0" ixz="0" iyy="0.01" iyz="0" izz="0.01"/>
-    </inertial>
-  </link>
-  <!-- Joint 1 -->
-  <link name="meca_axis_1_link_A">
-    <visual>
-      <origin xyz="0 0 0" rpy="0 0 0" />
-      <geometry>
-        <mesh filename="package://mecademic_description/meshes/meca_500_r3_j1.dae" />
-      </geometry>
-    </visual>
-    <collision>
-      <origin xyz="0 0 0" rpy="0 0 0" />
-      <geometry>
-        <mesh filename="package://mecademic_description/meshes/meca_500_r3_j1_collision.stl" />
-      </geometry>
-    </collision>
-    <inertial>
-      <mass value="1"/>
-      <inertia ixx="0.01" ixy="0" ixz="0" iyy="0.01" iyz="0" izz="0.01"/>
-    </inertial>
-  </link>
-  <joint name="meca_axis_1_joint_A" type="revolute">
-    <origin xyz="0.012498 0 0.091" rpy="0 0 0" />
-    <parent link="meca_base_link_A" />
-    <child link="meca_axis_1_link_A" />
-    <axis xyz="0 0 1" />
-    <limit effort="10.0" velocity="2.61799" lower="-3.05" upper="3.05" />
-  </joint>
-  <!-- Joint 2 -->
-  <link name="meca_axis_2_link_A">
-    <visual>
-      <origin xyz="0 0 0" rpy="0 0 0" />
-      <geometry>
-        <mesh filename="package://mecademic_description/meshes/meca_500_r3_j2.dae" />
-      </geometry>
-    </visual>
-    <collision>
-      <origin xyz="0 0 0" rpy="0 0 0" />
-      <geometry>
-        <mesh filename="package://mecademic_description/meshes/meca_500_r3_j2_collision.stl" />
-      </geometry>
-    </collision>
-    <inertial>
-      <mass value="1"/>
-      <inertia ixx="0.01" ixy="0" ixz="0" iyy="0.01" iyz="0" izz="0.01"/>
-    </inertial>
-  </link>
-  <joint name="meca_axis_2_joint_A" type="revolute">
-    <origin xyz="0 0 0.044" rpy="0 0 0" />
-    <parent link="meca_axis_1_link_A" />
-    <child link="meca_axis_2_link_A" />
-    <axis xyz="0 1 0" />
-    <limit effort="10.0" velocity="2.61799" lower="-1.22" upper="1.57" />
-  </joint>
-  <!-- Joint 3 -->
-  <link name="meca_axis_3_link_A">
-    <visual>
-      <origin xyz="0 0 0" rpy="0 0 0" />
-      <geometry>
-        <mesh filename="package://mecademic_description/meshes/meca_500_r3_j3.dae" />
-      </geometry>
-    </visual>
-    <collision>
-      <origin xyz="0 0 0" rpy="0 0 0" />
-      <geometry>
-        <mesh filename="package://mecademic_description/meshes/meca_500_r3_j3_collision.stl" />
-      </geometry>
-    </collision>
-    <inertial>
-      <mass value="1"/>
-      <inertia ixx="0.01" ixy="0" ixz="0" iyy="0.01" iyz="0" izz="0.01"/>
-    </inertial>
-  </link>
-  <joint name="meca_axis_3_joint_A" type="revolute">
-    <origin xyz="0 0 0.135" rpy="0 0 0" />
-    <parent link="meca_axis_2_link_A" />
-    <child link="meca_axis_3_link_A" />
-    <axis xyz="0 1 0" />
-    <limit effort="10.0" velocity="3.14159" lower="-2.35" upper="1.22" />
-  </joint>
-  <!-- Joint 4 -->
-  <link name="meca_axis_4_link_A">
-    <visual>
-      <origin xyz="0 0 0" rpy="0 0 0" />
-      <geometry>
-        <mesh filename="package://mecademic_description/meshes/meca_500_r3_j4.dae" />
-      </geometry>
-    </visual>
-    <collision>
-      <origin xyz="0 0 0" rpy="0 0 0" />
-      <geometry>
-        <mesh filename="package://mecademic_description/meshes/meca_500_r3_j4_collision.stl" />
-      </geometry>
-    </collision>
-    <inertial>
-      <mass value="1"/>
-      <inertia ixx="0.01" ixy="0" ixz="0" iyy="0.01" iyz="0" izz="0.01"/>
-    </inertial>
-  </link>
-  <joint name="meca_axis_4_joint_A" type="revolute">
-    <origin xyz="0 0 0.038" rpy="0 0 0" />
-    <parent link="meca_axis_3_link_A" />
-    <child link="meca_axis_4_link_A" />
-    <axis xyz="1 0 0" />
-    <limit effort="10.0" velocity="5.23599" lower="-2.96" upper="2.96" />
-  </joint>
-  <!-- Joint 5 -->
-  <link name="meca_axis_5_link_A">
-    <visual>
-      <origin xyz="0 0 0" rpy="0 0 0" />
-      <geometry>
-        <mesh filename="package://mecademic_description/meshes/meca_500_r3_j5.dae" />
-      </geometry>
-    </visual>
-    <collision>
-      <origin xyz="0 0 0" rpy="0 0 0" />
-      <geometry>
-        <mesh filename="package://mecademic_description/meshes/meca_500_r3_j5_collision.stl" />
-      </geometry>
-    </collision>
-    <inertial>
-      <mass value="1"/>
-      <inertia ixx="0.01" ixy="0" ixz="0" iyy="0.01" iyz="0" izz="0.01"/>
-    </inertial>
-  </link>
-  <joint name="meca_axis_5_joint_A" type="revolute">
-    <origin xyz="0.12 0 0" rpy="0 0 0" />
-    <parent link="meca_axis_4_link_A" />
-    <child link="meca_axis_5_link_A" />
-    <axis xyz="0 1 0" />
-    <limit effort="10.0" velocity="5.23599" lower="-2.00" upper="2.00" />
-  </joint>
-  <!-- Joint 6 -->
-  <link name="meca_axis_6_link_A">
-    <visual>
-      <origin xyz="0 0 0" rpy="0 0 0" />
-      <geometry>
-        <mesh filename="package://mecademic_description/meshes/meca_500_r3_j6.dae" />
-      </geometry>
-    </visual>
-    <collision>
-      <origin xyz="0 0 0" rpy="0 0 0" />
-      <geometry>
-        <mesh filename="package://mecademic_description/meshes/meca_500_r3_j6_collision.stl" />
-      </geometry>
-    </collision>
-    <inertial>
-      <mass value="1"/>
-      <inertia ixx="0.01" ixy="0" ixz="0" iyy="0.01" iyz="0" izz="0.01"/>
-    </inertial>
-  </link>
-  <joint name="meca_axis_6_joint_A" type="revolute">
-    <origin xyz="0.07 0 0" rpy="0 0 0" />
-    <parent link="meca_axis_5_link_A" />
-    <child link="meca_axis_6_link_A" />
-    <axis xyz="1 0 0" />
-    <limit effort="10.0" velocity="8.72665" lower="-4.0" upper="4.0" />
-  </joint>
-  <!-- gripper -->
-  <link name="vacuum_gripper">
-    <visual>
-      <origin xyz="0 0 0" rpy="0 0 0" />
-      <geometry>
-        <mesh filename="package://mecademic_description/meshes/pneumatic_tube_holder_mesh_v2.stl" scale="0.001 0.001 0.001"/>
-      </geometry>
-    </visual>
-    <collision>
-      <origin xyz="0 0 0" rpy="0 0 0" />
-      <geometry>
-        <mesh filename="package://mecademic_description/meshes/pneumatic_tube_holder_mesh_v2.stl" scale="0.001 0.001 0.001"/>
-      </geometry>
-    </collision>
-    <inertial>
-      <mass value="1"/>
-      <inertia ixx="0.01" ixy="0" ixz="0" iyy="0.01" iyz="0" izz="0.01"/>
-    </inertial>
-  </link>
-  <joint name="meca_to_gripper_A_joint" type="fixed">
-    <origin xyz="0 0 0" rpy="0 0 0" />
-    <parent link="meca_axis_6_link_A" />
-    <child link="vacuum_gripper" />
-  </joint>
-  <!-- End Effector -->
-  <link name="ee_link_A">
-    <inertial>
-      <mass value="1"/>
-      <inertia ixx="0.01" ixy="0" ixz="0" iyy="0.01" iyz="0" izz="0.01"/>
-    </inertial>
-  </link>
-  <joint name="vacum_gripper_to_ee_A_joint" type="fixed">
-    <origin xyz="0.015 0.0087 -0.0323" rpy="0 0 0" />
-    <parent link="vacuum_gripper" />
-    <child link="ee_link_A" />
-  </joint>
 <!-- 2nd ROBOT -->
   <joint name="world_to_base_B" type="fixed">
@@ -467,5 +133,5 @@
     <parent link="L_1_B"/>
     <child link="meca_base_link_B"/>
-    <origin rpy="0 1.571 0" xyz="0.0475 0.0 0.0575"/>
+    <origin rpy="0 1.571 0" xyz="0.0475 0.0 0.0645"/>
   </joint>
     <!-- Base link is the center of the robot's bottom plate -->
