Commit message: only rotary meca

File: mecademic_description/urdf/meca_500_r3_capsule.urdf.xacro (robot description, xacro)
@@ -26,448 +26,4 @@
   </material>
   <link name="world"/>
-  <joint name="world_to_base_A" type="fixed">
-    <origin rpy="0.0 0.0 0.0" xyz="0.6 0.16 0.05"/>
-    <parent link="world"/>
-    <child link="base_link_A"/>
-  </joint>
-  <gazebo>
-    <plugin filename="libxbot2_gz_joint_server.so" name="xbot2_gz_joint_server">
-      <pid>
-        <pid name="BL4104C_1" profile="medium_mot"/>
-        <pid name="meca_axis_1_joint_A" profile="small_mot"/>
-        <pid name="meca_axis_2_joint_A" profile="small_mot"/>
-        <pid name="meca_axis_3_joint_A" profile="small_mot"/>
-        <pid name="meca_axis_4_joint_A" profile="small_mot"/>
-        <pid name="meca_axis_5_joint_A" profile="small_mot"/>
-        <pid name="meca_axis_6_joint_A" profile="small_mot"/>
-      </pid>
-      <gain d="5" name="small_mot" p="100"/>
-    </plugin>
-  </gazebo>
-  <link name="base_link_A">
-    <inertial>
-      <mass value="0.1"/>
-      <inertia ixx="0.001" ixy="0.0" ixz="0.0" iyy="0.001" iyz="0.0" izz="0.001"/>
-    </inertial>
-  </link>
-  <joint name="fixed_gear_box" type="fixed">
-    <origin rpy="0.0 0.0 1.571" xyz="0.431 0.0 0.05"/>
-    <parent link="base_link_A"/>
-    <child link="gear_box"/>
-  </joint>
-  <link name="gear_box">
-    <inertial>
-      <origin rpy="0.0 0.0 0.0" xyz="0.0 0.0 0.10614489"/>
-      <mass value="2.0554934"/>
-      <inertia ixx="0.01068855" ixy="-1.14168e-05" ixz="2.71689e-06" iyy="0.010584907" iyz="8.76312e-05" izz="0.0032026258"/>
-    </inertial>
-    <visual>
-      <origin rpy="0.0 1.571 0.0" xyz="0.183 0.0 0.0"/>
-      <geometry>
-        <cylinder length="0.366" radius="0.12"/>
-      </geometry>
-      <material name="blue">
-        <color rgba="0.0 0.0 0.8 1.0"/>
-      </material>
-    </visual>
-    <collision>
-      <origin rpy="0.0 1.571 0.0" xyz="0.183 0.0 0.0"/>
-      <geometry>
-        <cylinder length="0.366" radius="0.12"/>
-      </geometry>
-    </collision>
-    <collision>
-      <origin rpy="0.0 1.571 0.0" xyz="0.000000 0.000000 0.000037"/>
-      <geometry>
-        <sphere radius="0.12"/>
-      </geometry>
-    </collision>
-    <collision>
-      <origin rpy="0.0 1.571 0.0" xyz="0.366000 0.000000 -0.000037"/>
-      <geometry>
-        <sphere radius="0.12"/>
-      </geometry>
-    </collision>
-  </link>
-  <joint name="fixed_linear_motor" type="fixed">
-    <origin rpy="0.0 0.0 0.0" xyz="0.0 0.0 0.05"/>
-    <parent link="base_link_A"/>
-    <child link="linear_motor_stator"/>
-  </joint>
-  <link name="linear_motor_stator">
-    <inertial>
-      <origin rpy="0.0 0.0 0.0" xyz="0.0 0.0 0.10614489"/>
-      <mass value="2.0554934"/>
-      <inertia ixx="0.01068855" ixy="-1.14168e-05" ixz="2.71689e-06" iyy="0.010584907" iyz="8.76312e-05" izz="0.0032026258"/>
-    </inertial>
-    <visual>
-      <origin rpy="0.0 0.0 0.0" xyz="0.0 0.0 0.0"/>
-      <geometry>
-        <box size="0.98 0.12 0.1"/>
-      </geometry>
-      <material name="blue">
-        <color rgba="0.0 0.0 0.8 1.0"/>
-      </material>
-    </visual>
-    <collision>
-      <origin rpy="0.0 1.571 0.0" xyz="0.0 0.0 0.05"/>
-      <geometry>
-        <cylinder length="0.98" radius="0.12"/>
-      </geometry>
-    </collision>
-    <collision>
-      <origin rpy="0.0 1.571 0.0" xyz="-0.490000 0.000000 0.050100"/>
-      <geometry>
-        <sphere radius="0.12"/>
-      </geometry>
-    </collision>
-    <collision>
-      <origin rpy="0.0 1.571 0.0" xyz="0.490000 0.000000 0.049900"/>
-      <geometry>
-        <sphere radius="0.12"/>
-      </geometry>
-    </collision>
-  </link>
-  <gazebo reference="linear_motor_stator">
-    <mu1>0.2</mu1>
-    <mu2>0.2</mu2>
-    <kp>1000000.0</kp>
-    <kd>1.0</kd>
-    <maxVel>0.0</maxVel>
-    <minDepth>0.0001</minDepth>
-    <material>Gazebo/Blue</material>
-  </gazebo>
-  <joint name="linear_motor" type="prismatic">
-    <origin rpy="0.0 0.0 0.0" xyz="-0.26 0.0 0.09"/>
-    <axis xyz="1.0 0.0 0.0"/>
-    <parent link="linear_motor_stator"/>
-    <child link="L_1_A"/>
-    <limit effort="100.0" lower="-0.002" upper="0.4" velocity="0.5"/>
-  </joint>
-  <link name="L_1_A">
-    <inertial>
-      <origin rpy="0.0 0.0 0.0" xyz="0.0 0.0 -0.024438213"/>
-      <mass value="0.42322395"/>
-      <inertia ixx="0.00063746146" ixy="1.1903424e-05" ixz="6.7230372e-07" iyy="0.00064218987" iyz="2.203073e-05" izz="0.001009674"/>
-    </inertial>
-    <visual>
-      <origin rpy="0.0 0.0 0.0" xyz="0.0 0.0 -0.02"/>
-      <geometry>
-        <box size="0.2 0.2 0.04"/>
-      </geometry>
-      <material name="blue">
-        <color rgba="0.0 0.0 0.8 1.0"/>
-      </material>
-    </visual>
-    <collision>
-      <origin rpy="0.0 0.0 0.0" xyz="0.0 0.0 -0.02"/>
-      <geometry>
-        <box size="0.2 0.2 0.04"/>
-      </geometry>
-    </collision>
-  </link>
-  <joint name="L_1_A_to_meca_base_link_A" type="fixed">
-    <origin rpy="0.0 1.571 1.571" xyz="0.0 0.014 0.0744"/>
-    <parent link="L_1_A"/>
-    <child link="meca_base_link_A"/>
-  </joint>
-  <link name="meca_base_link_A">
-    <inertial>
-      <mass value="1.0"/>
-      <inertia ixx="0.01" ixy="0.0" ixz="0.0" iyy="0.01" iyz="0.0" izz="0.01"/>
-    </inertial>
-    <visual>
-      <origin rpy="0.0 0.0 0.0" xyz="0.0 0.0 0.0"/>
-      <geometry>
-        <mesh filename="package://mecademic_description/meshes/meca_500_r3_base.dae"/>
-      </geometry>
-    </visual>
-    <collision>
-      <origin rpy="-0.00464229562531 1.241639409 -0.00331992768483" xyz="0.002912665 2.5933825e-05 0.03195115"/>
-      <geometry>
-        <cylinder length="0.0247681427348" radius="0.069277"/>
-      </geometry>
-    </collision>
-    <collision>
-      <origin rpy="-0.00464229562531 1.241639409 -0.00331992768483" xyz="-0.008807 0.000007 0.027948"/>
-      <geometry>
-        <sphere radius="0.069277"/>
-      </geometry>
-    </collision>
-    <collision>
-      <origin rpy="-0.00464229562531 1.241639409 -0.00331992768483" xyz="0.014632 0.000045 0.035954"/>
-      <geometry>
-        <sphere radius="0.069277"/>
-      </geometry>
-    </collision>
-  </link>
-  <link name="meca_axis_1_link_A">
-    <inertial>
-      <mass value="1.0"/>
-      <inertia ixx="0.01" ixy="0.0" ixz="0.0" iyy="0.01" iyz="0.0" izz="0.01"/>
-    </inertial>
-    <visual>
-      <origin rpy="0.0 0.0 0.0" xyz="0.0 0.0 0.0"/>
-      <geometry>
-        <mesh filename="package://mecademic_description/meshes/meca_500_r3_j1.dae"/>
-      </geometry>
-    </visual>
-    <collision>
-      <origin rpy="-1.5643390872 0.00108905813092 -0.00108204843032" xyz="1.404e-07 -0.00017605 0.03168225"/>
-      <geometry>
-        <cylinder length="0.0388249324419" radius="0.0530516"/>
-      </geometry>
-    </collision>
-    <collision>
-      <origin rpy="-1.5643390872 0.00108905813092 -0.00108204843032" xyz="-0.000021 -0.019588 0.031557"/>
-      <geometry>
-        <sphere radius="0.0530516"/>
-      </geometry>
-    </collision>
-    <collision>
-      <origin rpy="-1.5643390872 0.00108905813092 -0.00108204843032" xyz="0.000021 0.019236 0.031808"/>
-      <geometry>
-        <sphere radius="0.0530516"/>
-      </geometry>
-    </collision>
-  </link>
-  <joint name="meca_axis_1_joint_A" type="revolute">
-    <origin rpy="0.0 0.0 0.0" xyz="0.012498 0.0 0.091"/>
-    <axis xyz="0.0 0.0 1.0"/>
-    <parent link="meca_base_link_A"/>
-    <child link="meca_axis_1_link_A"/>
-    <limit effort="10.0" lower="-3.05" upper="3.05" velocity="2.61799"/>
-  </joint>
-  <link name="meca_axis_2_link_A">
-    <inertial>
-      <mass value="1.0"/>
-      <inertia ixx="0.01" ixy="0.0" ixz="0.0" iyy="0.01" iyz="0.0" izz="0.01"/>
-    </inertial>
-    <visual>
-      <origin rpy="0.0 0.0 0.0" xyz="0.0 0.0 0.0"/>
-      <geometry>
-        <mesh filename="package://mecademic_description/meshes/meca_500_r3_j2.dae"/>
-      </geometry>
-    </visual>
-    <collision>
-      <origin rpy="3.14150631803 -0.0666872950524 -3.13900434911" xyz="-0.007204205 2.561655e-06 0.07263715"/>
-      <geometry>
-        <cylinder length="0.121249210008" radius="0.0578403"/>
-      </geometry>
-    </collision>
-    <collision>
-      <origin rpy="3.14150631803 -0.0666872950524 -3.13900434911" xyz="-0.003164 0.000008 0.133127"/>
-      <geometry>
-        <sphere radius="0.0578403"/>
-      </geometry>
-    </collision>
-    <collision>
-      <origin rpy="3.14150631803 -0.0666872950524 -3.13900434911" xyz="-0.011244 -0.000003 0.012147"/>
-      <geometry>
-        <sphere radius="0.0578403"/>
-      </geometry>
-    </collision>
-  </link>
-  <joint name="meca_axis_2_joint_A" type="revolute">
-    <origin rpy="0.0 0.0 0.0" xyz="0.0 0.0 0.044"/>
-    <axis xyz="0.0 1.0 0.0"/>
-    <parent link="meca_axis_1_link_A"/>
-    <child link="meca_axis_2_link_A"/>
-    <limit effort="10.0" lower="-1.22" upper="1.57" velocity="2.61799"/>
-  </joint>
-  <link name="meca_axis_3_link_A">
-    <inertial>
-      <mass value="1.0"/>
-      <inertia ixx="0.01" ixy="0.0" ixz="0.0" iyy="0.01" iyz="0.0" izz="0.01"/>
-    </inertial>
-    <visual>
-      <origin rpy="0.0 0.0 0.0" xyz="0.0 0.0 0.0"/>
-      <geometry>
-        <mesh filename="package://mecademic_description/meshes/meca_500_r3_j3.dae"/>
-      </geometry>
-    </visual>
-    <collision>
-      <origin rpy="-0.0775632999618 0.486298597709 -0.0192491912301" xyz="0.009983498 -0.000990284 0.020095595"/>
-      <geometry>
-        <cylinder length="0.0408120816515" radius="0.0503272"/>
-      </geometry>
-    </collision>
-    <collision>
-      <origin rpy="-0.0775632999618 0.486298597709 -0.0192491912301" xyz="0.000447 -0.002388 0.002109"/>
-      <geometry>
-        <sphere radius="0.0503272"/>
-      </geometry>
-    </collision>
-    <collision>
-      <origin rpy="-0.0775632999618 0.486298597709 -0.0192491912301" xyz="0.019520 0.000408 0.038082"/>
-      <geometry>
-        <sphere radius="0.0503272"/>
-      </geometry>
-    </collision>
-  </link>
-  <joint name="meca_axis_3_joint_A" type="revolute">
-    <origin rpy="0.0 0.0 0.0" xyz="0.0 0.0 0.135"/>
-    <axis xyz="0.0 1.0 0.0"/>
-    <parent link="meca_axis_2_link_A"/>
-    <child link="meca_axis_3_link_A"/>
-    <limit effort="10.0" lower="-2.35" upper="1.22" velocity="3.14159"/>
-  </joint>
-  <link name="meca_axis_4_link_A">
-    <inertial>
-      <mass value="1.0"/>
-      <inertia ixx="0.01" ixy="0.0" ixz="0.0" iyy="0.01" iyz="0.0" izz="0.01"/>
-    </inertial>
-    <visual>
-      <origin rpy="0.0 0.0 0.0" xyz="0.0 0.0 0.0"/>
-      <geometry>
-        <mesh filename="package://mecademic_description/meshes/meca_500_r3_j4.dae"/>
-      </geometry>
-    </visual>
-    <collision>
-      <origin rpy="-1.61527511752 1.5509782436 -1.59546790677" xyz="0.1018437 -0.00037629375 0.0004856635"/>
-      <geometry>
-        <cylinder length="0.0362997282424" radius="0.0387182"/>
-      </geometry>
-    </collision>
-    <collision>
-      <origin rpy="-1.61527511752 1.5509782436 -1.59546790677" xyz="0.083697 -0.000736 0.000502"/>
-      <geometry>
-        <sphere radius="0.0387182"/>
-      </geometry>
-    </collision>
-    <collision>
-      <origin rpy="-1.61527511752 1.5509782436 -1.59546790677" xyz="0.119990 -0.000017 0.000470"/>
-      <geometry>
-        <sphere radius="0.0387182"/>
-      </geometry>
-    </collision>
-  </link>
-  <joint name="meca_axis_4_joint_A" type="revolute">
-    <origin rpy="0.0 0.0 0.0" xyz="0.0 0.0 0.038"/>
-    <axis xyz="1.0 0.0 0.0"/>
-    <parent link="meca_axis_3_link_A"/>
-    <child link="meca_axis_4_link_A"/>
-    <limit effort="10.0" lower="-2.96" upper="2.96" velocity="5.23599"/>
-  </joint>
-  <link name="meca_axis_5_link_A">
-    <inertial>
-      <mass value="1.0"/>
-      <inertia ixx="0.01" ixy="0.0" ixz="0.0" iyy="0.01" iyz="0.0" izz="0.01"/>
-    </inertial>
-    <visual>
-      <origin rpy="0.0 0.0 0.0" xyz="0.0 0.0 0.0"/>
-      <geometry>
-        <mesh filename="package://mecademic_description/meshes/meca_500_r3_j5.dae"/>
-      </geometry>
-    </visual>
-    <collision>
-      <origin rpy="-1.56738494938 1.42197043963 -1.41859762505" xyz="0.022533785 0.002385127 -0.000338951"/>
-      <geometry>
-        <cylinder length="0.0337980384654" radius="0.0373293"/>
-      </geometry>
-    </collision>
-    <collision>
-      <origin rpy="-1.56738494938 1.42197043963 -1.41859762505" xyz="0.005822 -0.000121 -0.000347"/>
-      <geometry>
-        <sphere radius="0.0373293"/>
-      </geometry>
-    </collision>
-    <collision>
-      <origin rpy="-1.56738494938 1.42197043963 -1.41859762505" xyz="0.039246 0.004891 -0.000330"/>
-      <geometry>
-        <sphere radius="0.0373293"/>
-      </geometry>
-    </collision>
-  </link>
-  <joint name="meca_axis_5_joint_A" type="revolute">
-    <origin rpy="0.0 0.0 0.0" xyz="0.12 0.0 0.0"/>
-    <axis xyz="0.0 1.0 0.0"/>
-    <parent link="meca_axis_4_link_A"/>
-    <child link="meca_axis_5_link_A"/>
-    <limit effort="10.0" lower="-2.0" upper="2.0" velocity="5.23599"/>
-  </joint>
-  <link name="meca_axis_6_link_A">
-    <inertial>
-      <mass value="1.0"/>
-      <inertia ixx="0.01" ixy="0.0" ixz="0.0" iyy="0.01" iyz="0.0" izz="0.01"/>
-    </inertial>
-    <visual>
-      <origin rpy="0.0 0.0 0.0" xyz="0.0 0.0 0.0"/>
-      <geometry>
-        <mesh filename="package://mecademic_description/meshes/meca_500_r3_j6.dae"/>
-      </geometry>
-    </visual>
-    <collision>
-      <origin rpy="3.14152943169 -0.0847389814668 -3.14010139052" xyz="-0.002858345 7.482995e-07 -1.9915e-05"/>
-      <geometry>
-        <cylinder length="0.00588946257883" radius="0.0134707"/>
-      </geometry>
-    </collision>
-    <collision>
-      <origin rpy="3.14152943169 -0.0847389814668 -3.14010139052" xyz="-0.002609 0.000001 0.002914"/>
-      <geometry>
-        <sphere radius="0.0134707"/>
-      </geometry>
-    </collision>
-    <collision>
-      <origin rpy="3.14152943169 -0.0847389814668 -3.14010139052" xyz="-0.003108 0.000001 -0.002954"/>
-      <geometry>
-        <sphere radius="0.0134707"/>
-      </geometry>
-    </collision>
-  </link>
-  <joint name="meca_axis_6_joint_A" type="revolute">
-    <origin rpy="0.0 0.0 0.0" xyz="0.07 0.0 0.0"/>
-    <axis xyz="1.0 0.0 0.0"/>
-    <parent link="meca_axis_5_link_A"/>
-    <child link="meca_axis_6_link_A"/>
-    <limit effort="10.0" lower="-4.0" upper="4.0" velocity="8.72665"/>
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
Commit message: update capsules for linear guide

File: mecademic_description/urdf/meca_500_r3.urdf.xacro (robot description, xacro)
@@ -146,11 +146,11 @@
       <origin xyz="0 0 0" rpy="0 0 0" />
       <geometry>
-        <mesh filename="package://mecademic_description/meshes/pump_and_robot_mount_metres_lower_quality.stl" />
-      </geometry>
-    </visual>
-    <collision>
-      <origin xyz="0 0 0" rpy="0 0 0" />
-      <geometry>
-        <mesh filename="package://mecademic_description/meshes/pump_and_robot_mount_metres_lower_quality.stl" />
+        <mesh filename="package://mecademic_description/meshes/pump_and_robot_mount_metres_even_lower_quality.stl" />
+      </geometry>
+    </visual>
+    <collision>
+      <origin xyz="0 0 0" rpy="0 0 0" />
+      <geometry>
+        <mesh filename="package://mecademic_description/meshes/pump_and_robot_mount_metres_even_lower_quality.stl" />
       </geometry>
     </collision>

File: mecademic_description/urdf/meca_500_r3_capsule.urdf.xacro (robot description, xacro)
@@ -27,5 +27,5 @@
   <link name="world"/>
   <joint name="world_to_base_A" type="fixed">
-    <origin rpy="0.0 0.0 0.0" xyz="0.6 0.16 0.05"/>
+    <origin rpy="0.0 0.0 0.0" xyz="0.11 0.083 0.05"/>
     <parent link="world"/>
     <child link="base_link_A"/>
@@ -52,5 +52,5 @@
   </link>
   <joint name="fixed_gear_box" type="fixed">
-    <origin rpy="0.0 0.0 1.571" xyz="0.431 0.0 0.05"/>
+    <origin rpy="0.0 0.0 1.571" xyz="0.927 0.07 0.08"/>
     <parent link="base_link_A"/>
     <child link="gear_box"/>
@@ -63,7 +63,7 @@
     </inertial>
     <visual>
-      <origin rpy="0.0 1.571 0.0" xyz="0.183 0.0 0.0"/>
-      <geometry>
-        <cylinder length="0.366" radius="0.12"/>
+      <origin rpy="0.0 1.571 0.0" xyz="0.2025 0.0 0.0"/>
+      <geometry>
+        <cylinder length="0.405" radius="0.065"/>
       </geometry>
       <material name="blue">
@@ -72,24 +72,24 @@
     </visual>
     <collision>
-      <origin rpy="0.0 1.571 0.0" xyz="0.183 0.0 0.0"/>
-      <geometry>
-        <cylinder length="0.366" radius="0.12"/>
-      </geometry>
-    </collision>
-    <collision>
-      <origin rpy="0.0 1.571 0.0" xyz="0.000000 0.000000 0.000037"/>
-      <geometry>
-        <sphere radius="0.12"/>
-      </geometry>
-    </collision>
-    <collision>
-      <origin rpy="0.0 1.571 0.0" xyz="0.366000 0.000000 -0.000037"/>
-      <geometry>
-        <sphere radius="0.12"/>
+      <origin rpy="0.0 1.571 0.0" xyz="0.2025 0.0 0.0"/>
+      <geometry>
+        <cylinder length="0.405" radius="0.065"/>
+      </geometry>
+    </collision>
+    <collision>
+      <origin rpy="0.0 1.571 0.0" xyz="0.000000 0.000000 0.000041"/>
+      <geometry>
+        <sphere radius="0.065"/>
+      </geometry>
+    </collision>
+    <collision>
+      <origin rpy="0.0 1.571 0.0" xyz="0.405000 0.000000 -0.000041"/>
+      <geometry>
+        <sphere radius="0.065"/>
       </geometry>
     </collision>
   </link>
   <joint name="fixed_linear_motor" type="fixed">
-    <origin rpy="0.0 0.0 0.0" xyz="0.0 0.0 0.05"/>
+    <origin rpy="0.0 0.0 0.0" xyz="0.0 0.0 0.0"/>
     <parent link="base_link_A"/>
     <child link="linear_motor_stator"/>
@@ -104,26 +104,23 @@
       <origin rpy="0.0 0.0 0.0" xyz="0.0 0.0 0.0"/>
       <geometry>
-        <box size="0.98 0.12 0.1"/>
-      </geometry>
-      <material name="blue">
-        <color rgba="0.0 0.0 0.8 1.0"/>
-      </material>
-    </visual>
-    <collision>
-      <origin rpy="0.0 1.571 0.0" xyz="0.0 0.0 0.05"/>
-      <geometry>
-        <cylinder length="0.98" radius="0.12"/>
-      </geometry>
-    </collision>
-    <collision>
-      <origin rpy="0.0 1.571 0.0" xyz="-0.490000 0.000000 0.050100"/>
-      <geometry>
-        <sphere radius="0.12"/>
-      </geometry>
-    </collision>
-    <collision>
-      <origin rpy="0.0 1.571 0.0" xyz="0.490000 0.000000 0.049900"/>
-      <geometry>
-        <sphere radius="0.12"/>
+        <mesh filename="package://mecademic_description/meshes/linear_guide_base_meters.stl"/>
+      </geometry>
+    </visual>
+    <collision>
+      <origin rpy="2.2937756802 1.5707939573 2.29377390347" xyz="0.49 0.05430915 0.05892555"/>
+      <geometry>
+        <cylinder length="0.956812000003" radius="0.081078"/>
+      </geometry>
+    </collision>
+    <collision>
+      <origin rpy="2.2937756802 1.5707939573 2.29377390347" xyz="0.011594 0.054310 0.058926"/>
+      <geometry>
+        <sphere radius="0.081078"/>
+      </geometry>
+    </collision>
+    <collision>
+      <origin rpy="2.2937756802 1.5707939573 2.29377390347" xyz="0.968406 0.054308 0.058925"/>
+      <geometry>
+        <sphere radius="0.081078"/>
       </geometry>
     </collision>
@@ -139,5 +136,5 @@
   </gazebo>
   <joint name="linear_motor" type="prismatic">
-    <origin rpy="0.0 0.0 0.0" xyz="-0.26 0.0 0.09"/>
+    <origin rpy="0.0 0.0 0.0" xyz="0.262 0.06 0.102"/>
     <axis xyz="1.0 0.0 0.0"/>
     <parent link="linear_motor_stator"/>
@@ -152,22 +149,67 @@
     </inertial>
     <visual>
-      <origin rpy="0.0 0.0 0.0" xyz="0.0 0.0 -0.02"/>
-      <geometry>
-        <box size="0.2 0.2 0.04"/>
-      </geometry>
-      <material name="blue">
-        <color rgba="0.0 0.0 0.8 1.0"/>
-      </material>
-    </visual>
-    <collision>
-      <origin rpy="0.0 0.0 0.0" xyz="0.0 0.0 -0.02"/>
-      <geometry>
-        <box size="0.2 0.2 0.04"/>
-      </geometry>
-    </collision>
-  </link>
-  <joint name="L_1_A_to_meca_base_link_A" type="fixed">
-    <origin rpy="0.0 1.571 1.571" xyz="0.0 0.014 0.0744"/>
+      <origin rpy="0.0 0.0 0.0" xyz="0.0 0.0 0.0"/>
+      <geometry>
+        <mesh filename="package://mecademic_description/meshes/linear_guide_mover_meters.stl"/>
+      </geometry>
+    </visual>
+    <collision>
+      <origin rpy="0.0 1.57079632679 1.60984711283e-14" xyz="0.0 1.35033e-10 0.0098086"/>
+      <geometry>
+        <cylinder length="0.1242354" radius="0.114543"/>
+      </geometry>
+    </collision>
+    <collision>
+      <origin rpy="0.0 1.57079632679 1.60984711283e-14" xyz="-0.062118 0.000000 0.009809"/>
+      <geometry>
+        <sphere radius="0.114543"/>
+      </geometry>
+    </collision>
+    <collision>
+      <origin rpy="0.0 1.57079632679 1.60984711283e-14" xyz="0.062118 0.000000 0.009809"/>
+      <geometry>
+        <sphere radius="0.114543"/>
+      </geometry>
+    </collision>
+  </link>
+  <joint name="L_1_A_to_stuff_on_top_A" type="fixed">
+    <origin rpy="0.0 0.0 0.0" xyz="0.0 0.0 0.0355"/>
     <parent link="L_1_A"/>
+    <child link="stuff_on_top_A"/>
+  </joint>
+  <link name="stuff_on_top_A">
+    <inertial>
+      <origin rpy="0.0 0.0 0.0" xyz="0.0 0.0 -0.024438213"/>
+      <mass value="0.42322395"/>
+      <inertia ixx="0.00063746146" ixy="1.1903424e-05" ixz="6.7230372e-07" iyy="0.00064218987" iyz="2.203073e-05" izz="0.001009674"/>
+    </inertial>
+    <visual>
+      <origin rpy="0.0 0.0 0.0" xyz="0.0 0.0 0.0"/>
+      <geometry>
+        <mesh filename="package://mecademic_description/meshes/pump_and_robot_mount_metres_even_lower_quality.stl"/>
+      </geometry>
+    </visual>
+    <collision>
+      <origin rpy="-1.62917422953 1.38891587263 -1.44663604517" xyz="-0.01940155 -0.01246106 0.07044685"/>
+      <geometry>
+        <cylinder length="0.0846839364147" radius="0.111533"/>
+      </geometry>
+    </collision>
+    <collision>
+      <origin rpy="-1.62917422953 1.38891587263 -1.44663604517" xyz="-0.061045 -0.020107 0.070894"/>
+      <geometry>
+        <sphere radius="0.111533"/>
+      </geometry>
+    </collision>
+    <collision>
+      <origin rpy="-1.62917422953 1.38891587263 -1.44663604517" xyz="0.022242 -0.004815 0.070000"/>
+      <geometry>
+        <sphere radius="0.111533"/>
+      </geometry>
+    </collision>
+  </link>
+  <joint name="stuff_on_top_A_to_meca_base_link_A" type="fixed">
+    <origin rpy="0.0 1.571 1.571" xyz="0.05 0.024 0.0705"/>
+    <parent link="stuff_on_top_A"/>
     <child link="meca_base_link_A"/>
   </joint>
@@ -593,5 +635,5 @@
   </link>
   <joint name="L_1_B_to_meca_base_link_B" type="fixed">
-    <origin rpy="0.0 1.571 0.0" xyz="0.0475 0.0 0.0575"/>
+    <origin rpy="0.0 1.571 0.0" xyz="0.0475 0.0 0.0645"/>
     <parent link="L_1_B"/>
     <child link="meca_base_link_B"/>
