Commit message: add buffer_and_slide_support mesh and collisions

File: mecademic_description/urdf/meca_500_r3.urdf.xacro (robot description, xacro)
@@ -711,5 +711,22 @@
     <child link="buffer_base_link"/>
   </joint>
-  <link name="buffer_base_link"/>
+  <link name="buffer_base_link">
+    <visual>
+      <origin xyz="0 0.065 -0.075" rpy="1.57 0 -1.57" />
+      <geometry>
+        <mesh filename="package://mecademic_description/meshes/buffer_and_slide_support_v17.stl" scale="0.001 0.001 0.001"/>
+      </geometry>
+    </visual>
+    <collision>
+      <origin xyz="0 0.065 -0.075" rpy="1.57 0 -1.57" />
+      <geometry>
+        <mesh filename="package://mecademic_description/meshes/buffer_and_slide_support_v17.stl" scale="0.001 0.001 0.001"/>
+      </geometry>
+    </collision>
+    <inertial>
+      <mass value="1"/>
+      <inertia ixx="0.01" ixy="0" ixz="0" iyy="0.01" iyz="0" izz="0.01"/>
+    </inertial>
+  </link>
   <joint name="buffer_base_to_1" type="fixed">
     <origin xyz="0.525 0 0" rpy="0 0 0"/>

File: mecademic_description/urdf/meca_500_r3_capsule.urdf.xacro (robot description, xacro)
@@ -942,5 +942,22 @@
     <child link="buffer_base_link"/>
   </joint>
-  <link name="buffer_base_link"/>
+  <link name="buffer_base_link">
+    <visual>
+      <origin xyz="0 0.065 -0.075" rpy="1.57 0 -1.57" />
+      <geometry>
+        <mesh filename="package://mecademic_description/meshes/buffer_and_slide_support_v17.stl" scale="0.001 0.001 0.001"/>
+      </geometry>
+    </visual>
+    <collision>
+      <origin xyz="0 0.065 -0.075" rpy="1.57 0 -1.57" />
+      <geometry>
+        <mesh filename="package://mecademic_description/meshes/buffer_and_slide_support_v17.stl" scale="0.001 0.001 0.001"/>
+      </geometry>
+    </collision>
+    <inertial>
+      <mass value="1"/>
+      <inertia ixx="0.01" ixy="0" ixz="0" iyy="0.01" iyz="0" izz="0.01"/>
+    </inertial>
+  </link>
   <joint name="buffer_base_to_1" type="fixed">
     <origin xyz="0.525 0 0" rpy="0 0 0"/>

Commit message: update transforms of buffers and sliders

File: mecademic_description/urdf/meca_500_r3.urdf.xacro (robot description, xacro)
@@ -707,5 +707,5 @@
   <!-- BUFFERS -->
   <joint name="world_to_buffer" type="fixed">
-     <origin xyz="0 0.585 0.2" rpy="0 0 0"/>
+     <origin xyz="0 0.650 0.075" rpy="0 0 0"/>
     <parent link="world"/>
     <child link="buffer_base_link"/>
@@ -713,5 +713,5 @@
   <link name="buffer_base_link">
     <visual>
-      <origin xyz="0 0.065 -0.075" rpy="1.57 0 -1.57" />
+      <origin xyz="0 0.0 0.0" rpy="1.57 0 -1.57" />
       <geometry>
         <mesh filename="package://mecademic_description/meshes/buffer_and_slide_support_v17.stl" scale="0.001 0.001 0.001"/>
@@ -719,5 +719,5 @@
     </visual>
     <collision>
-      <origin xyz="0 0.065 -0.075" rpy="1.57 0 -1.57" />
+      <origin xyz="0 0.0 0.0" rpy="1.57 0 -1.57" />
       <geometry>
         <mesh filename="package://mecademic_description/meshes/buffer_and_slide_support_v17.stl" scale="0.001 0.001 0.001"/>
@@ -730,5 +730,5 @@
   </link>
   <joint name="buffer_base_to_1" type="fixed">
-    <origin xyz="0.525 0 0" rpy="0 0 0"/>
+    <origin xyz="0.525 -0.065 0.03" rpy="0 0 0"/>
     <parent link="buffer_base_link"/>
     <child link="buffer_1"/>
@@ -736,5 +736,5 @@
   <link name="buffer_1"/>
   <joint name="buffer_base_to_2" type="fixed">
-        <origin xyz="0.650 0.0 0" rpy="0 0 0"/>
+        <origin xyz="0.650 -0.065 0.03" rpy="0 0 0"/>
         <parent link="buffer_base_link"/>
         <child link="buffer_2"/>
@@ -762,5 +762,5 @@
   <!-- SLIDERS -->
   <joint name="world_to_slider" type="fixed">
-    <origin xyz="0 0.585 0.0" rpy="0 0 0"/>
+    <origin xyz="0 0.650 0.0" rpy="0 0 0"/>
     <parent link="world"/>
     <child link="slider_base_link"/>
@@ -768,5 +768,5 @@
   <link name="slider_base_link"/>
   <joint name="slider_base_to_empty" type="fixed">
-    <origin xyz="0.397 0 0.194" rpy="0 0.1745 0"/>
+    <origin xyz="0.397 -0.065 0.194" rpy="0 0.1745 0"/>
     <parent link="slider_base_link"/>
     <child link="empty_container"/>
@@ -774,5 +774,5 @@
   <link name="empty_container"/>
   <joint name="sliders_base_to_lid" type="fixed">
-        <origin xyz="0.322 0 0.319" rpy="0 0.1745 0"/>
+        <origin xyz="0.322 -0.065 0.319" rpy="0 0.1745 0"/>
         <parent link="slider_base_link"/>
         <child link="lid"/>
@@ -780,5 +780,5 @@
   <link name="lid"/>
   <joint name="sliders_base_to_full" type="fixed">
-        <origin xyz="0.809 0 0.295" rpy="0 0.1745 0"/>
+        <origin xyz="0.809 -0.065 0.295" rpy="0 0.1745 0"/>
         <parent link="slider_base_link"/>
         <child link="full_container"/>

Commit message: move base_link_A

File: mecademic_description/urdf/meca_500_r3.urdf.xacro (robot description, xacro)
@@ -29,5 +29,5 @@
     <parent link="world"/>
     <child link="base_link_A"/>
-    <origin rpy="0 0 0" xyz="0.110 0.083 0.050"/>
+    <origin rpy="0 0 0" xyz="0.030 0.10 0.050"/>
   </joint>
   <gazebo>

File: mecademic_description/urdf/meca_500_r3_capsule.urdf.xacro (robot description, xacro)
@@ -27,5 +27,5 @@
   <link name="world"/>
   <joint name="world_to_base_A" type="fixed">
-    <origin rpy="0.0 0.0 0.0" xyz="0.11 0.083 0.05"/>
+    <origin rpy="0.0 0.0 0.0" xyz="0.03 0.10 0.05"/>
     <parent link="world"/>
     <child link="base_link_A"/>

Commit message: shift everything of 2 cm on y

File: mecademic_description/urdf/meca_500_r3.urdf.xacro (robot description, xacro)
@@ -29,5 +29,5 @@
     <parent link="world"/>
     <child link="base_link_A"/>
-    <origin rpy="0 0 0" xyz="0.030 0.10 0.050"/>
+    <origin rpy="0 0 0" xyz="0.030 0.083 0.050"/>
   </joint>
   <gazebo>
@@ -164,5 +164,5 @@
     <parent link="stuff_on_top_A"/>
     <child link="meca_base_link_A"/>
-    <origin rpy="0 1.571 1.571" xyz="0.05 0.024 0.0705"/>
+    <origin rpy="0 1.571 1.571" xyz="0.05 0.061 0.0705"/>
   </joint>
     <!-- Base link is the center of the robot's bottom plate -->
@@ -379,5 +379,5 @@
 <!-- 2nd ROBOT -->
   <joint name="world_to_base_B" type="fixed">
-      <origin xyz="0.4521 0.9847 0.050" rpy="0 0 -1.571"/>
+      <origin xyz="0.4521 1.0047 0.050" rpy="0 0 -1.571"/>
       <parent link="world"/>
       <child link="base_link_B"/>
@@ -707,5 +707,5 @@
   <!-- BUFFERS -->
   <joint name="world_to_buffer" type="fixed">
-     <origin xyz="0 0.650 0.075" rpy="0 0 0"/>
+     <origin xyz="0 0.670 0.075" rpy="0 0 0"/>
     <parent link="world"/>
     <child link="buffer_base_link"/>
@@ -743,5 +743,5 @@
   <!-- CANDY MILL -->
   <joint name="world_to_mill" type="fixed">
-    <origin xyz="0.8154 0.8 0.0" rpy="0 0 0"/>
+    <origin xyz="0.8154 0.82 0.0" rpy="0 0 0"/>
     <parent link="world"/>
     <child link="mill_base_link"/>
@@ -762,5 +762,5 @@
   <!-- SLIDERS -->
   <joint name="world_to_slider" type="fixed">
-    <origin xyz="0 0.650 0.0" rpy="0 0 0"/>
+    <origin xyz="0 0.670 0.0" rpy="0 0 0"/>
     <parent link="world"/>
     <child link="slider_base_link"/>

File: mecademic_description/urdf/meca_500_r3_capsule.urdf.xacro (robot description, xacro)
@@ -27,5 +27,5 @@
   <link name="world"/>
   <joint name="world_to_base_A" type="fixed">
-    <origin rpy="0.0 0.0 0.0" xyz="0.03 0.10 0.05"/>
+    <origin rpy="0.0 0.0 0.0" xyz="0.03 0.083 0.05"/>
     <parent link="world"/>
     <child link="base_link_A"/>
@@ -210,5 +210,5 @@
   </link>
   <joint name="stuff_on_top_A_to_meca_base_link_A" type="fixed">
-    <origin rpy="0.0 1.571 1.571" xyz="0.05 0.024 0.0705"/>
+    <origin rpy="0 1.571 1.571" xyz="0.05 0.061 0.0705"/>
     <parent link="stuff_on_top_A"/>
     <child link="meca_base_link_A"/>
@@ -513,5 +513,5 @@
   </joint>
   <joint name="world_to_base_B" type="fixed">
-    <origin rpy="0.0 0.0 -1.571" xyz="0.4521 0.9847 0.05"/>
+    <origin xyz="0.4521 1.0047 0.050" rpy="0 0 -1.571"/>
     <parent link="world"/>
     <child link="base_link_B"/>
@@ -938,5 +938,5 @@
   </joint>
   <joint name="world_to_buffer" type="fixed">
-    <origin xyz="0 0.650 0.075" rpy="0 0 0"/>
+   <origin xyz="0 0.670 0.075" rpy="0 0 0"/>
     <parent link="world"/>
     <child link="buffer_base_link"/>
@@ -973,5 +973,5 @@
   <link name="buffer_2"/>
   <joint name="world_to_mill" type="fixed">
-    <origin xyz="0.8154 0.8 0.0" rpy="0 0 0"/>
+    <origin xyz="0.8154 0.82 0.0" rpy="0 0 0"/>
     <parent link="world"/>
     <child link="mill_base_link"/>
@@ -992,5 +992,5 @@
   <!-- SLIDERS -->
   <joint name="world_to_slider" type="fixed">
-    <origin xyz="0 0.650 0.0" rpy="0 0 0"/>
+    <origin xyz="0 0.670 0.0" rpy="0 0 0"/>
     <parent link="world"/>
     <child link="slider_base_link"/>

Commit message: fix vacuum gripper tf

File: mecademic_description/urdf/meca_500_r3.urdf.xacro (robot description, xacro)
@@ -373,5 +373,5 @@
   </link>
   <joint name="vacum_gripper_to_ee_A_joint" type="fixed">
-    <origin xyz="0.015 0.0087 -0.0323" rpy="0 0 0" />
+    <origin xyz="0.015 0. -0.0323" rpy="0 0 0" />
     <parent link="vacuum_gripper" />
     <child link="ee_link_A" />

File: mecademic_description/urdf/meca_500_r3_capsule.urdf.xacro (robot description, xacro)
@@ -508,5 +508,5 @@
   </link>
   <joint name="vacum_gripper_to_ee_A_joint" type="fixed">
-    <origin rpy="0.0 0.0 0.0" xyz="0.015 0.0087 -0.0323"/>
+    <origin rpy="0.0 0.0 0.0" xyz="0.015 0.0 -0.0323"/>
     <parent link="vacuum_gripper"/>
     <child link="ee_link_A"/>

Commit message: update vacuum_gripper length

File: mecademic_description/urdf/meca_500_r3.urdf.xacro (robot description, xacro)
@@ -373,5 +373,5 @@
   </link>
   <joint name="vacum_gripper_to_ee_A_joint" type="fixed">
-    <origin xyz="0.015 0. -0.0323" rpy="0 0 0" />
+    <origin xyz="0.015 0. -0.0671" rpy="0 0 0" />
     <parent link="vacuum_gripper" />
     <child link="ee_link_A" />

File: mecademic_description/urdf/meca_500_r3_capsule.urdf.xacro (robot description, xacro)
@@ -508,5 +508,5 @@
   </link>
   <joint name="vacum_gripper_to_ee_A_joint" type="fixed">
-    <origin rpy="0.0 0.0 0.0" xyz="0.015 0.0 -0.0323"/>
+    <origin rpy="0.0 0.0 0.0" xyz="0.015 0.0 -0.0671"/>
     <parent link="vacuum_gripper"/>
     <child link="ee_link_A"/>

Commit message: increase linear motor upper joint limit 0.4 -> 0.45

File: mecademic_description/urdf/meca_500_r3.urdf.xacro (robot description, xacro)
@@ -115,5 +115,5 @@
     <parent link="linear_motor_stator"/>
     <child link="L_1_A"/>
-    <limit effort="100.0" lower="-0.002" upper="0.400" velocity="0.5"/>
+    <limit effort="100.0" lower="-0.002" upper="0.450" velocity="0.5"/>
     <origin rpy="0 0 0" xyz="0.262 0.06 0.102"/>
   </joint>

File: mecademic_description/urdf/meca_500_r3_capsule.urdf.xacro (robot description, xacro)
@@ -140,5 +140,5 @@
     <parent link="linear_motor_stator"/>
     <child link="L_1_A"/>
-    <limit effort="100.0" lower="-0.002" upper="0.4" velocity="0.5"/>
+    <limit effort="100.0" lower="-0.002" upper="0.450" velocity="0.5"/>
   </joint>
   <link name="L_1_A">

Commit message: update vacuum gripper mesh and capsule

File: mecademic_description/urdf/meca_500_r3.urdf.xacro (robot description, xacro)
@@ -346,11 +346,11 @@
       <origin xyz="0 0 0" rpy="0 0 0" />
       <geometry>
-        <mesh filename="package://mecademic_description/meshes/pneumatic_tube_holder_mesh_v2.stl" scale="0.001 0.001 0.001"/>
-      </geometry>
-    </visual>
-    <collision>
-      <origin xyz="0 0 0" rpy="0 0 0" />
-      <geometry>
-        <mesh filename="package://mecademic_description/meshes/pneumatic_tube_holder_mesh_v2.stl" scale="0.001 0.001 0.001"/>
+        <mesh filename="package://mecademic_description/meshes/for_mesh_pneumatic_tube_holder_new_v5.stl" scale="0.001 0.001 0.001"/>
+      </geometry>
+    </visual>
+    <collision>
+      <origin xyz="0 0 0" rpy="0 0 0" />
+      <geometry>
+        <mesh filename="package://mecademic_description/meshes/for_mesh_pneumatic_tube_holder_new_v5.stl" scale="0.001 0.001 0.001"/>
       </geometry>
     </collision>

File: mecademic_description/urdf/meca_500_r3_capsule.urdf.xacro (robot description, xacro)
@@ -140,5 +140,5 @@
     <parent link="linear_motor_stator"/>
     <child link="L_1_A"/>
-    <limit effort="100.0" lower="-0.002" upper="0.450" velocity="0.5"/>
+    <limit effort="100.0" lower="-0.002" upper="0.45" velocity="0.5"/>
   </joint>
   <link name="L_1_A">
@@ -210,5 +210,5 @@
   </link>
   <joint name="stuff_on_top_A_to_meca_base_link_A" type="fixed">
-    <origin rpy="0 1.571 1.571" xyz="0.05 0.061 0.0705"/>
+    <origin rpy="0.0 1.571 1.571" xyz="0.05 0.061 0.0705"/>
     <parent link="stuff_on_top_A"/>
     <child link="meca_base_link_A"/>
@@ -474,23 +474,23 @@
       <origin rpy="0.0 0.0 0.0" xyz="0.0 0.0 0.0"/>
       <geometry>
-        <mesh filename="package://mecademic_description/meshes/pneumatic_tube_holder_mesh_v2.stl" scale="0.001 0.001 0.001"/>
-      </geometry>
-    </visual>
-    <collision>
-      <origin rpy="4.35637496773e-05 -0.0111409793996 -2.42673928992e-07" xyz="0.0127944 8.22252e-07 -0.00216735"/>
-      <geometry>
-        <cylinder length="0.052940785559" radius="0.0217467"/>
-      </geometry>
-    </collision>
-    <collision>
-      <origin rpy="4.35637496773e-05 -0.0111409793996 -2.42673928992e-07" xyz="0.013089 0.000002 -0.028636"/>
-      <geometry>
-        <sphere radius="0.0217467"/>
-      </geometry>
-    </collision>
-    <collision>
-      <origin rpy="4.35637496773e-05 -0.0111409793996 -2.42673928992e-07" xyz="0.012500 -0.000000 0.024301"/>
-      <geometry>
-        <sphere radius="0.0217467"/>
+        <mesh filename="package://mecademic_description/meshes/for_mesh_pneumatic_tube_holder_new_v5.stl" scale="0.001 0.001 0.001"/>
+      </geometry>
+    </visual>
+    <collision>
+      <origin rpy="0.000369675884525 -0.00595860855088 -1.10138021455e-06" xyz="0.01273105 -7.811225e-05 -0.03211868"/>
+      <geometry>
+        <cylinder length="0.0836945315022" radius="0.0220478"/>
+      </geometry>
+    </collision>
+    <collision>
+      <origin rpy="0.000369675884525 -0.00595860855088 -1.10138021455e-06" xyz="0.012980 -0.000063 -0.073965"/>
+      <geometry>
+        <sphere radius="0.0220478"/>
+      </geometry>
+    </collision>
+    <collision>
+      <origin rpy="0.000369675884525 -0.00595860855088 -1.10138021455e-06" xyz="0.012482 -0.000094 0.009728"/>
+      <geometry>
+        <sphere radius="0.0220478"/>
       </geometry>
     </collision>
@@ -513,5 +513,5 @@
   </joint>
   <joint name="world_to_base_B" type="fixed">
-    <origin xyz="0.4521 1.0047 0.050" rpy="0 0 -1.571"/>
+    <origin rpy="0.0 0.0 -1.571" xyz="0.4521 1.0047 0.05"/>
     <parent link="world"/>
     <child link="base_link_B"/>
@@ -938,11 +938,15 @@
   </joint>
   <joint name="world_to_buffer" type="fixed">
-   <origin xyz="0 0.670 0.075" rpy="0 0 0"/>
+    <origin rpy="0.0 0.0 0.0" xyz="0.0 0.67 0.075"/>
     <parent link="world"/>
     <child link="buffer_base_link"/>
   </joint>
   <link name="buffer_base_link">
-    <visual>
-      <origin xyz="0 0.0 0.0" rpy="1.57 0 -1.57" />
+    <inertial>
+      <mass value="1.0"/>
+      <inertia ixx="0.01" ixy="0.0" ixz="0.0" iyy="0.01" iyz="0.0" izz="0.01"/>
+    </inertial>
+    <visual>
+      <origin rpy="1.57 0.0 -1.57" xyz="0.0 0.0 0.0"/>
       <geometry>
         <mesh filename="package://mecademic_description/meshes/buffer_and_slide_support_v17.stl" scale="0.001 0.001 0.001"/>
@@ -961,5 +965,5 @@
   </link>
   <joint name="buffer_base_to_1" type="fixed">
-    <origin xyz="0.525 -0.065 0.03" rpy="0 0 0"/>
+    <origin rpy="0.0 0.0 0.0" xyz="0.525 -0.065 0.03"/>
     <parent link="buffer_base_link"/>
     <child link="buffer_1"/>
@@ -967,5 +971,5 @@
   <link name="buffer_1"/>
   <joint name="buffer_base_to_2" type="fixed">
-        <origin xyz="0.650 -0.065 0.03" rpy="0 0 0"/>
+    <origin rpy="0.0 0.0 0.0" xyz="0.65 -0.065 0.03"/>
         <parent link="buffer_base_link"/>
         <child link="buffer_2"/>
@@ -973,5 +977,5 @@
   <link name="buffer_2"/>
   <joint name="world_to_mill" type="fixed">
-    <origin xyz="0.8154 0.82 0.0" rpy="0 0 0"/>
+    <origin rpy="0.0 0.0 0.0" xyz="0.8154 0.82 0.0"/>
     <parent link="world"/>
     <child link="mill_base_link"/>
@@ -985,12 +989,11 @@
   <link name="mill_stick"/>
   <joint name="mill_base_to_buffer" type="fixed">
-    <origin xyz="0.0 0 0.15" rpy="0 0 0"/>
+    <origin rpy="0.0 0.0 0.0" xyz="0.0 0.0 0.15"/>
     <parent link="mill_base_link"/>
     <child link="mill_buffer"/>
   </joint>
   <link name="mill_buffer"/>
-  <!-- SLIDERS -->
   <joint name="world_to_slider" type="fixed">
-    <origin xyz="0 0.670 0.0" rpy="0 0 0"/>
+    <origin rpy="0.0 0.0 0.0" xyz="0.0 0.67 0.0"/>
     <parent link="world"/>
     <child link="slider_base_link"/>
@@ -998,5 +1001,5 @@
   <link name="slider_base_link"/>
   <joint name="slider_base_to_empty" type="fixed">
-    <origin xyz="0.397 -0.065 0.194" rpy="0 0.1745 0"/>
+    <origin rpy="0.0 0.1745 0.0" xyz="0.397 -0.065 0.194"/>
     <parent link="slider_base_link"/>
     <child link="empty_container"/>
@@ -1004,5 +1007,5 @@
   <link name="empty_container"/>
   <joint name="sliders_base_to_lid" type="fixed">
-    <origin xyz="0.322 -0.065 0.319" rpy="0 0.1745 0"/>
+    <origin rpy="0.0 0.1745 0.0" xyz="0.322 -0.065 0.319"/>
     <parent link="slider_base_link"/>
     <child link="lid"/>
@@ -1010,30 +1013,8 @@
   <link name="lid"/>
   <joint name="sliders_base_to_full" type="fixed">
-    <origin xyz="0.809 -0.065 0.295" rpy="0 0.1745 0"/>
+    <origin rpy="0.0 0.1745 0.0" xyz="0.809 -0.065 0.295"/>
     <parent link="slider_base_link"/>
     <child link="full_container"/>
   </joint>
   <link name="full_container"/>
-  <!-- <joint name="world_to_floor" type="fixed">
-    <origin rpy="0.0 0.0 0.0" xyz="0.0 0.0 0.05"/>
-    <parent link="world"/>
-    <child link="floor_link"/>
-  </joint>
-  <link name="floor_link">
-    <visual>
-      <origin rpy="0.0 0.0 0.0" xyz="0.0 0.0 0.0"/>
-      <geometry>
-        <box size="2.0 2.0 0.0"/>
-      </geometry>
-      <material name="grey">
-        <color rgba="0.232 0.232 0.232 1.0"/>
-      </material>
-    </visual>
-    <collision>
-      <origin rpy="0.0 0.0 0.0" xyz="0.0 0.0 0.0"/>
-      <geometry>
-        <box size="2.0 2.0 0.0"/>
-      </geometry>
-    </collision>
-  </link> -->
 </robot>

Commit message: fix rotary table radius (removed proximity sensor margin)

File: mecademic_description/urdf/meca_500_r3.urdf.xacro (robot description, xacro)
@@ -420,5 +420,5 @@
       <origin rpy="0.0 0.0 0.0" xyz="0.0 0.0 0.105"/>
       <geometry>
-        <cylinder length="0.21" radius="0.16"/>
+        <cylinder length="0.21" radius="0.135"/>
       </geometry>
     </collision>

File: mecademic_description/urdf/meca_500_r3_capsule.urdf.xacro (robot description, xacro)
@@ -558,5 +558,5 @@
       <origin rpy="0.0 0.0 0.0" xyz="0.0 0.0 0.105"/>
       <geometry>
-        <cylinder length="0.21" radius="0.145"/>
+        <cylinder length="0.21" radius="0.135"/>
       </geometry>
     </collision>
@@ -564,5 +564,5 @@
       <origin rpy="0.0 0.0 0.0" xyz="0.000000 0.000000 0.000000"/>
       <geometry>
-        <sphere radius="0.145"/>
+        <sphere radius="0.135"/>
       </geometry>
     </collision>
@@ -570,5 +570,5 @@
       <origin rpy="0.0 0.0 0.0" xyz="0.000000 0.000000 0.210000"/>
       <geometry>
-        <sphere radius="0.145"/>
+        <sphere radius="0.135"/>
       </geometry>
     </collision>

Commit message: new mesh for the sliders

File: mecademic_description/urdf/meca_500_r3.urdf.xacro (robot description, xacro)
@@ -713,13 +713,13 @@
   <link name="buffer_base_link">
     <visual>
-      <origin xyz="0 0.0 0.0" rpy="1.57 0 -1.57" />
-      <geometry>
-        <mesh filename="package://mecademic_description/meshes/buffer_and_slide_support_v17.stl" scale="0.001 0.001 0.001"/>
-      </geometry>
-    </visual>
-    <collision>
-      <origin xyz="0 0.0 0.0" rpy="1.57 0 -1.57" />
-      <geometry>
-        <mesh filename="package://mecademic_description/meshes/buffer_and_slide_support_v17.stl" scale="0.001 0.001 0.001"/>
+      <origin xyz="0 0.0 0.0" rpy="0 0 0" />
+      <geometry>
+        <mesh filename="package://mecademic_description/meshes/for_mesh_buffer_and_input_slide_support_new_v21.stl" scale="1 1 1"/>
+      </geometry>
+    </visual>
+    <collision>
+      <origin xyz="0 0.0 0.0" rpy="0 0 0" />
+      <geometry>
+        <mesh filename="package://mecademic_description/meshes/for_mesh_buffer_and_input_slide_support_new_v21.stl" scale="1 1 1"/>
       </geometry>
     </collision>

File: mecademic_description/urdf/meca_500_r3_capsule.urdf.xacro (robot description, xacro)
@@ -948,13 +948,13 @@
     </inertial>
     <visual>
-      <origin rpy="1.57 0.0 -1.57" xyz="0.0 0.0 0.0"/>
-      <geometry>
-        <mesh filename="package://mecademic_description/meshes/buffer_and_slide_support_v17.stl" scale="0.001 0.001 0.001"/>
-      </geometry>
-    </visual>
-    <collision>
-      <origin xyz="0 0.0 0.0" rpy="1.57 0 -1.57" />
-      <geometry>
-        <mesh filename="package://mecademic_description/meshes/buffer_and_slide_support_v17.stl" scale="0.001 0.001 0.001"/>
+      <origin rpy="0 0.0 0" xyz="0.0 0.0 0.0"/>
+      <geometry>
+        <mesh filename="package://mecademic_description/meshes/for_mesh_buffer_and_input_slide_support_new_v21.stl" scale="1 1 1"/>
+      </geometry>
+    </visual>
+    <collision>
+      <origin xyz="0 0.0 0.0" rpy="0 0 0" />
+      <geometry>
+        <mesh filename="package://mecademic_description/meshes/for_mesh_buffer_and_input_slide_support_new_v21.stl" scale="1 1 1"/>
       </geometry>
     </collision>

Commit message: fix buffer base link height

File: mecademic_description/urdf/meca_500_r3.urdf.xacro (robot description, xacro)
@@ -707,5 +707,5 @@
   <!-- BUFFERS -->
   <joint name="world_to_buffer" type="fixed">
-     <origin xyz="0 0.670 0.075" rpy="0 0 0"/>
+     <origin xyz="0 0.670 0.080" rpy="0 0 0"/>
     <parent link="world"/>
     <child link="buffer_base_link"/>

File: mecademic_description/urdf/meca_500_r3_capsule.urdf.xacro (robot description, xacro)
@@ -938,5 +938,5 @@
   </joint>
   <joint name="world_to_buffer" type="fixed">
-    <origin rpy="0.0 0.0 0.0" xyz="0.0 0.67 0.075"/>
+    <origin rpy="0.0 0.0 0.0" xyz="0.0 0.67 0.080"/>
     <parent link="world"/>
     <child link="buffer_base_link"/>
