Commit message: update the frames of the objects on the sliders

File: mecademic_description/urdf/meca_500_r3.urdf.xacro (robot description, xacro)
@@ -768,5 +768,5 @@
   <link name="slider_base_link"/>
   <joint name="slider_base_to_empty" type="fixed">
-    <origin xyz="0.397 -0.065 0.194" rpy="0 0.1745 0"/>
+    <origin xyz="0.354 -0.065 0.165" rpy="0 0.349 0"/>
     <parent link="slider_base_link"/>
     <child link="empty_container"/>
@@ -774,5 +774,5 @@
   <link name="empty_container"/>
   <joint name="sliders_base_to_lid" type="fixed">
-        <origin xyz="0.322 -0.065 0.319" rpy="0 0.1745 0"/>
+        <origin xyz="0.303 -0.065 0.310" rpy="0 0.349 0"/>
         <parent link="slider_base_link"/>
         <child link="lid"/>
@@ -780,5 +780,5 @@
   <link name="lid"/>
   <joint name="sliders_base_to_full" type="fixed">
-        <origin xyz="0.809 -0.065 0.295" rpy="0 0.1745 0"/>
+        <origin xyz="0.822 -0.065 0.287" rpy="0 0.349 0"/>
         <parent link="slider_base_link"/>
         <child link="full_container"/>

File: mecademic_description/urdf/meca_500_r3_capsule.urdf.xacro (robot description, xacro)
@@ -999,7 +999,12 @@
     <child link="slider_base_link"/>
   </joint>
+  <joint name="world_to_slider" type="fixed">
+    <origin xyz="0 0.670 0.0" rpy="0 0 0"/>
+    <parent link="world"/>
+    <child link="slider_base_link"/>
+  </joint>
   <link name="slider_base_link"/>
   <joint name="slider_base_to_empty" type="fixed">
-    <origin rpy="0.0 0.1745 0.0" xyz="0.397 -0.065 0.194"/>
+    <origin xyz="0.354 -0.065 0.165" rpy="0 0.349 0"/>
     <parent link="slider_base_link"/>
     <child link="empty_container"/>
@@ -1007,14 +1012,14 @@
   <link name="empty_container"/>
   <joint name="sliders_base_to_lid" type="fixed">
-    <origin rpy="0.0 0.1745 0.0" xyz="0.322 -0.065 0.319"/>
-    <parent link="slider_base_link"/>
-    <child link="lid"/>
-  </joint>
+        <origin xyz="0.303 -0.065 0.310" rpy="0 0.349 0"/>
+        <parent link="slider_base_link"/>
+        <child link="lid"/>
+      </joint>
   <link name="lid"/>
   <joint name="sliders_base_to_full" type="fixed">
-    <origin rpy="0.0 0.1745 0.0" xyz="0.809 -0.065 0.295"/>
-    <parent link="slider_base_link"/>
-    <child link="full_container"/>
-  </joint>
+        <origin xyz="0.822 -0.065 0.287" rpy="0 0.349 0"/>
+        <parent link="slider_base_link"/>
+        <child link="full_container"/>
+      </joint>
   <link name="full_container"/>
 </robot>

Commit message: update buffer mesh and slider frames

File: mecademic_description/urdf/meca_500_r3.urdf.xacro (robot description, xacro)
@@ -715,5 +715,5 @@
       <origin xyz="0 0.0 0.0" rpy="0 0 0" />
       <geometry>
-        <mesh filename="package://mecademic_description/meshes/for_mesh_buffer_and_input_slide_support_new_v21.stl" scale="1 1 1"/>
+        <mesh filename="package://mecademic_description/meshes/for_mesh_buffer_and_input_slide_support_new_v6.stl" scale="1 1 1"/>
       </geometry>
     </visual>
@@ -721,5 +721,5 @@
       <origin xyz="0 0.0 0.0" rpy="0 0 0" />
       <geometry>
-        <mesh filename="package://mecademic_description/meshes/for_mesh_buffer_and_input_slide_support_new_v21.stl" scale="1 1 1"/>
+        <mesh filename="package://mecademic_description/meshes/for_mesh_buffer_and_input_slide_support_new_v6.stl" scale="1 1 1"/>
       </geometry>
     </collision>
@@ -768,5 +768,5 @@
   <link name="slider_base_link"/>
   <joint name="slider_base_to_empty" type="fixed">
-    <origin xyz="0.354 -0.065 0.165" rpy="0 0.349 0"/>
+    <origin xyz="0.364 -0.065 0.160" rpy="0 0.349 0"/>
     <parent link="slider_base_link"/>
     <child link="empty_container"/>
@@ -774,5 +774,5 @@
   <link name="empty_container"/>
   <joint name="sliders_base_to_lid" type="fixed">
-        <origin xyz="0.303 -0.065 0.310" rpy="0 0.349 0"/>
+        <origin xyz="0.276 -0.065 0.293" rpy="0 0.349 0"/>
         <parent link="slider_base_link"/>
         <child link="lid"/>

File: mecademic_description/urdf/meca_500_r3_capsule.urdf.xacro (robot description, xacro)
@@ -950,5 +950,5 @@
       <origin rpy="0 0.0 0" xyz="0.0 0.0 0.0"/>
       <geometry>
-        <mesh filename="package://mecademic_description/meshes/for_mesh_buffer_and_input_slide_support_new_v21.stl" scale="1 1 1"/>
+        <mesh filename="package://mecademic_description/meshes/for_mesh_buffer_and_input_slide_support_new_v6.stl" scale="1 1 1"/>
       </geometry>
     </visual>
@@ -956,5 +956,5 @@
       <origin xyz="0 0.0 0.0" rpy="0 0 0" />
       <geometry>
-        <mesh filename="package://mecademic_description/meshes/for_mesh_buffer_and_input_slide_support_new_v21.stl" scale="1 1 1"/>
+        <mesh filename="package://mecademic_description/meshes/for_mesh_buffer_and_input_slide_support_new_v6.stl" scale="1 1 1"/>
       </geometry>
     </collision>
@@ -995,9 +995,4 @@
   <link name="mill_buffer"/>
   <joint name="world_to_slider" type="fixed">
-    <origin rpy="0.0 0.0 0.0" xyz="0.0 0.67 0.0"/>
-    <parent link="world"/>
-    <child link="slider_base_link"/>
-  </joint>
-  <joint name="world_to_slider" type="fixed">
     <origin xyz="0 0.670 0.0" rpy="0 0 0"/>
     <parent link="world"/>
@@ -1006,5 +1001,5 @@
   <link name="slider_base_link"/>
   <joint name="slider_base_to_empty" type="fixed">
-    <origin xyz="0.354 -0.065 0.165" rpy="0 0.349 0"/>
+    <origin xyz="0.364 -0.065 0.160" rpy="0 0.349 0"/>
     <parent link="slider_base_link"/>
     <child link="empty_container"/>
@@ -1012,5 +1007,5 @@
   <link name="empty_container"/>
   <joint name="sliders_base_to_lid" type="fixed">
-        <origin xyz="0.303 -0.065 0.310" rpy="0 0.349 0"/>
+        <origin xyz="0.276 -0.065 0.293" rpy="0 0.349 0"/>
         <parent link="slider_base_link"/>
         <child link="lid"/>

Commit message: fix slider frames orientation

File: mecademic_description/urdf/meca_500_r3.urdf.xacro (robot description, xacro)
@@ -768,5 +768,5 @@
   <link name="slider_base_link"/>
   <joint name="slider_base_to_empty" type="fixed">
-    <origin xyz="0.364 -0.065 0.160" rpy="0 0.349 0"/>
+    <origin xyz="0.364 -0.065 0.160" rpy="0 0.314 0"/>
     <parent link="slider_base_link"/>
     <child link="empty_container"/>
@@ -774,5 +774,5 @@
   <link name="empty_container"/>
   <joint name="sliders_base_to_lid" type="fixed">
-        <origin xyz="0.276 -0.065 0.293" rpy="0 0.349 0"/>
+        <origin xyz="0.276 -0.065 0.293" rpy="0 0.314 0"/>
         <parent link="slider_base_link"/>
         <child link="lid"/>
@@ -780,5 +780,5 @@
   <link name="lid"/>
   <joint name="sliders_base_to_full" type="fixed">
-        <origin xyz="0.822 -0.065 0.287" rpy="0 0.349 0"/>
+        <origin xyz="0.822 -0.065 0.287" rpy="0 0.314 0"/>
         <parent link="slider_base_link"/>
         <child link="full_container"/>

File: mecademic_description/urdf/meca_500_r3_capsule.urdf.xacro (robot description, xacro)
@@ -1001,5 +1001,5 @@
   <link name="slider_base_link"/>
   <joint name="slider_base_to_empty" type="fixed">
-    <origin xyz="0.364 -0.065 0.160" rpy="0 0.349 0"/>
+    <origin xyz="0.364 -0.065 0.160" rpy="0 0.314 0"/>
     <parent link="slider_base_link"/>
     <child link="empty_container"/>
@@ -1007,5 +1007,5 @@
   <link name="empty_container"/>
   <joint name="sliders_base_to_lid" type="fixed">
-        <origin xyz="0.276 -0.065 0.293" rpy="0 0.349 0"/>
+        <origin xyz="0.276 -0.065 0.293" rpy="0 0.314 0"/>
         <parent link="slider_base_link"/>
         <child link="lid"/>
@@ -1013,5 +1013,5 @@
   <link name="lid"/>
   <joint name="sliders_base_to_full" type="fixed">
-        <origin xyz="0.822 -0.065 0.287" rpy="0 0.349 0"/>
+        <origin xyz="0.822 -0.065 0.287" rpy="0 0.314 0"/>
         <parent link="slider_base_link"/>
         <child link="full_container"/>

Commit message: update slider mesh and frames

File: mecademic_description/urdf/meca_500_r3.urdf.xacro (robot description, xacro)
@@ -715,5 +715,5 @@
       <origin xyz="0 0.0 0.0" rpy="0 0 0" />
       <geometry>
-        <mesh filename="package://mecademic_description/meshes/for_mesh_buffer_and_input_slide_support_new_v6.stl" scale="1 1 1"/>
+        <mesh filename="package://mecademic_description/meshes/for_mesh_buffer_and_input_slide_support_new_v11.stl" scale="1 1 1"/>
       </geometry>
     </visual>
@@ -721,5 +721,5 @@
       <origin xyz="0 0.0 0.0" rpy="0 0 0" />
       <geometry>
-        <mesh filename="package://mecademic_description/meshes/for_mesh_buffer_and_input_slide_support_new_v6.stl" scale="1 1 1"/>
+        <mesh filename="package://mecademic_description/meshes/for_mesh_buffer_and_input_slide_support_new_v11.stl" scale="1 1 1"/>
       </geometry>
     </collision>
@@ -774,5 +774,5 @@
   <link name="empty_container"/>
   <joint name="sliders_base_to_lid" type="fixed">
-        <origin xyz="0.276 -0.065 0.293" rpy="0 0.314 0"/>
+        <origin xyz="0.282 -0.065 0.313" rpy="0 0.314 0"/>
         <parent link="slider_base_link"/>
         <child link="lid"/>
@@ -780,5 +780,5 @@
   <link name="lid"/>
   <joint name="sliders_base_to_full" type="fixed">
-        <origin xyz="0.822 -0.065 0.287" rpy="0 0.314 0"/>
+        <origin xyz="0.815 -0.065 0.310" rpy="0 0.314 0"/>
         <parent link="slider_base_link"/>
         <child link="full_container"/>

File: mecademic_description/urdf/meca_500_r3_capsule.urdf.xacro (robot description, xacro)
@@ -950,5 +950,5 @@
       <origin rpy="0 0.0 0" xyz="0.0 0.0 0.0"/>
       <geometry>
-        <mesh filename="package://mecademic_description/meshes/for_mesh_buffer_and_input_slide_support_new_v6.stl" scale="1 1 1"/>
+        <mesh filename="package://mecademic_description/meshes/for_mesh_buffer_and_input_slide_support_new_v11.stl" scale="1 1 1"/>
       </geometry>
     </visual>
@@ -956,5 +956,5 @@
       <origin xyz="0 0.0 0.0" rpy="0 0 0" />
       <geometry>
-        <mesh filename="package://mecademic_description/meshes/for_mesh_buffer_and_input_slide_support_new_v6.stl" scale="1 1 1"/>
+        <mesh filename="package://mecademic_description/meshes/for_mesh_buffer_and_input_slide_support_new_v11.stl" scale="1 1 1"/>
       </geometry>
     </collision>
@@ -1007,5 +1007,5 @@
   <link name="empty_container"/>
   <joint name="sliders_base_to_lid" type="fixed">
-        <origin xyz="0.276 -0.065 0.293" rpy="0 0.314 0"/>
+       <origin xyz="0.282 -0.065 0.313" rpy="0 0.314 0"/>
         <parent link="slider_base_link"/>
         <child link="lid"/>
@@ -1013,5 +1013,5 @@
   <link name="lid"/>
   <joint name="sliders_base_to_full" type="fixed">
-        <origin xyz="0.822 -0.065 0.287" rpy="0 0.314 0"/>
+        <origin xyz="0.815 -0.065 0.310" rpy="0 0.314 0"/>
         <parent link="slider_base_link"/>
         <child link="full_container"/>

Commit message: remove some collisions objects

File: mecademic_description/urdf/meca_500_r3.urdf.xacro (robot description, xacro)
@@ -51,5 +51,5 @@
     </inertial>
   </link>
-  <joint name="fixed_gear_box" type="fixed">
+  <!-- <joint name="fixed_gear_box" type="fixed">
     <parent link="base_link_A"/>
     <child link="gear_box"/>
@@ -77,5 +77,5 @@
       <inertia ixx="0.01068855" ixy="-1.14168e-05" ixz="2.71689e-06" iyy="0.010584907" iyz="8.76312e-05" izz="0.0032026258"/>
     </inertial>
-  </link>
+  </link> -->
   <joint name="fixed_linear_motor" type="fixed">
     <parent link="base_link_A"/>
@@ -706,5 +706,5 @@
   </joint> -->
   <!-- BUFFERS -->
-  <joint name="world_to_buffer" type="fixed">
+  <!-- <joint name="world_to_buffer" type="fixed">
      <origin xyz="0 0.670 0.080" rpy="0 0 0"/>
     <parent link="world"/>
@@ -740,7 +740,7 @@
         <child link="buffer_2"/>
       </joint>
-  <link name="buffer_2"/>
+  <link name="buffer_2"/> -->
   <!-- CANDY MILL -->
-  <joint name="world_to_mill" type="fixed">
+  <!-- <joint name="world_to_mill" type="fixed">
     <origin xyz="0.8154 0.82 0.0" rpy="0 0 0"/>
     <parent link="world"/>
@@ -759,7 +759,7 @@
     <child link="mill_buffer"/>
   </joint>
-  <link name="mill_buffer"/>
+  <link name="mill_buffer"/> -->
   <!-- SLIDERS -->
-  <joint name="world_to_slider" type="fixed">
+  <!-- <joint name="world_to_slider" type="fixed">
     <origin xyz="0 0.670 0.0" rpy="0 0 0"/>
     <parent link="world"/>
@@ -784,5 +784,5 @@
         <child link="full_container"/>
       </joint>
-  <link name="full_container"/>
+  <link name="full_container"/> -->
   <!-- FLOOR -->
   <!-- <joint name="world_to_floor" type="fixed">

File: mecademic_description/urdf/meca_500_r3_capsule.urdf.xacro (robot description, xacro)
@@ -51,5 +51,5 @@
     </inertial>
   </link>
-  <joint name="fixed_gear_box" type="fixed">
+  <!-- <joint name="fixed_gear_box" type="fixed">
     <origin rpy="0.0 0.0 1.571" xyz="0.927 0.07 0.08"/>
     <parent link="base_link_A"/>
@@ -89,5 +89,5 @@
       </geometry>
     </collision>
-  </link>
+  </link> -->
   <joint name="fixed_linear_motor" type="fixed">
     <origin rpy="0.0 0.0 0.0" xyz="0.0 0.0 0.0"/>
@@ -107,5 +107,5 @@
       </geometry>
     </visual>
-    <collision>
+    <!-- <collision>
       <origin rpy="2.2937756802 1.5707939573 2.29377390347" xyz="0.49 0.05430915 0.05892555"/>
       <geometry>
@@ -124,5 +124,5 @@
         <sphere radius="0.081078"/>
       </geometry>
-    </collision>
+    </collision> -->
   </link>
   <gazebo reference="linear_motor_stator">
@@ -154,5 +154,5 @@
       </geometry>
     </visual>
-    <collision>
+    <!-- <collision>
       <origin rpy="0.0 1.57079632679 1.60984711283e-14" xyz="0.0 1.35033e-10 0.0098086"/>
       <geometry>
@@ -171,5 +171,5 @@
         <sphere radius="0.114543"/>
       </geometry>
-    </collision>
+    </collision> -->
   </link>
   <joint name="L_1_A_to_stuff_on_top_A" type="fixed">
@@ -190,5 +190,5 @@
       </geometry>
     </visual>
-    <collision>
+    <!-- <collision>
       <origin rpy="-1.62917422953 1.38891587263 -1.44663604517" xyz="-0.01940155 -0.01246106 0.07044685"/>
       <geometry>
@@ -207,5 +207,5 @@
         <sphere radius="0.111533"/>
       </geometry>
-    </collision>
+    </collision> -->
   </link>
   <joint name="stuff_on_top_A_to_meca_base_link_A" type="fixed">
@@ -513,5 +513,5 @@
   </joint>
   <joint name="world_to_base_B" type="fixed">
-    <origin rpy="0.0 0.0 -1.571" xyz="0.4521 1.0047 0.05"/>
+    <origin rpy="0.0 0.0 -1.571" xyz="0.5 0.8 0.05"/>
     <parent link="world"/>
     <child link="base_link_B"/>
@@ -555,5 +555,5 @@
       <material name="grey"/>
     </visual>
-    <collision>
+    <!-- <collision>
       <origin rpy="0.0 0.0 0.0" xyz="0.0 0.0 0.105"/>
       <geometry>
@@ -572,5 +572,5 @@
         <sphere radius="0.135"/>
       </geometry>
-    </collision>
+    </collision> -->
   </link>
   <gazebo reference="rotary_table_stator">
@@ -603,5 +603,5 @@
       <material name="grey"/>
     </visual>
-    <collision>
+    <!-- <collision>
       <origin rpy="0.0 0.0 0.0" xyz="0.0 0.0 0.002"/>
       <geometry>
@@ -620,5 +620,5 @@
         <sphere radius="0.063"/>
       </geometry>
-    </collision>
+    </collision> -->
   </link>
   <joint name="fixed_L_1_B_rotor_fast" type="fixed">
@@ -937,5 +937,5 @@
     <child link="ee_link_B"/>
   </joint>
-  <joint name="world_to_buffer" type="fixed">
+  <!-- <joint name="world_to_buffer" type="fixed">
     <origin rpy="0.0 0.0 0.0" xyz="0.0 0.67 0.080"/>
     <parent link="world"/>
@@ -1017,4 +1017,4 @@
         <child link="full_container"/>
       </joint>
-  <link name="full_container"/>
+  <link name="full_container"/> -->
 </robot>
